File: LTC6811_ESP32.kicad_sch (KiCad schematic)
At the start: 17 parts, among them J11 CAN, J12 USB, J18 OLED, J3 + 12V -, Q1 BSS138

Commit message: Add files via upload
Parts:
- removed J11: CAN, Connectors_Molex:Molex_KK-6410-05_05x2.54mm_Straight, symbol BMS-Master-rescue:Conn_01x05-Connector_Generic-BMS-Master-rescue
- removed LOGO1: Logo_Open_Hardware_Small, ENNOID:ENNOID-LOGO, symbol Graphic:Logo_Open_Hardware_Small
- added J31: CAN, Connector_PinHeader_2.54mm:PinHeader_1x04_P2.54mm_Vertical, symbol Connector_Generic:Conn_01x04
- added LOGO2: teTra, Symbol:teTra-LOGO, symbol Fiber_Optic:logo
- J2: renamed from J18; footprint Connectors_Molex:Molex_KK-6410-05_05x2.54mm_Straight -> Connector_PinHeader_2.54mm:PinHeader_1x05_P2.54mm_Vertical
- J4: renamed from J12; footprint Connector_USB:USB_Micro-B_Molex-105133-0001 -> Connector_USB:Micro_USB_B-2013499-1; Link (none) -> https://www.digikey.jp/en/products/detail/te-connectivity-a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; MPN 47346-0001 -> 2013499-1
- Q1: footprint TO_SOT_Packages_SMD:SOT-23 -> Package_TO_SOT_SMD:SOT-23
- renumbered J3 to J1, R3 to R2, R2 to R3, R9 to R4, R4 to R5, R42 to R6, R46 to R7, R50 to R8
Connections:
- net CAN/5V_CAN: now also J31.1 (Pin_1)
- net CAN/CANH: now also J31.2 (Pin_2)
- net CAN/CANL: now also J31.3 (Pin_3)
- net CAN/CAN_GND: now also J31.4 (Pin_4)
Other:
- sheet CAN ports: added none; removed EnableRequest, Enable_CAN
- sheet MCU ports: added none; removed PowerEnable
- sheet PowerSupply ports: added BAT+; removed 12V, EnableFromExt, PowerEnable
- sheet USB ports: added none; removed EnableRequest
- company: ENNOID -> teTra

Commit message: Add files via upload
Parts:
- removed D1: POWER, LED_SMD:LED_0603_1608Metric, symbol BMS-Master-rescue:LED-Device-BMS-Master-rescue
- removed D2: STATUS, LED_SMD:LED_0603_1608Metric, symbol BMS-Master-rescue:LED-Device-BMS-Master-rescue
- removed J1: + 12V -, ENNOID:Pin_1x02-XL, symbol BMS-Master-rescue:Conn_01x02-Connector_Generic-BMS-Master-rescue
- added D1, D2: LED Red, LED_SMD:LED_0603_1608Metric, symbol Device:LED
- added R104: 0R, Resistor_SMD:R_0805_2012Metric, symbol Device:R_Small
- J2: value OLED -> OLED /NC; Link (none) -> https://www.digikey.jp/en/products/detail/molex/0705430004/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
- J31: value CAN -> CAN /NC
- R1, R2: value 470 -> 470R
- R5: value 1.5k -> 1.5K
- R6, R7, R8: value 4.75k -> 4.75K
Connections:
- net GND: now also D1.1 (K), D2.1 (K), R104.1
- net at R2.1: now also D2.2 (A)
- net at R1.1: now also D1.2 (A)
- new net GND_PACK: R104.2
Other:
- moved on the sheet: R7

Commit message: Add files via upload
Parts:
- BZ1: Link (none) -> https://www.digikey.jp/en/products/detail/pui-audio-inc/AI-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
- LOGO2: value teTra -> teTra /NC
- Q1: Link (none) -> https://www.digikey.jp/en/products/detail/anbon-semiconduct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
- R1, R2, R5: Link (none) -> https://www.digikey.jp/en/products/detail/yageo/RC0603JR-07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
- R104: Link https://www.digikey.jp/en/products/detail/koa-speer-electronics-inc/RK73Z2ATTD/10235990?s=N4IgTCBcDaIEoGkDsBmAWmAggFWwERAF0BfIA -> https://www.digikey.jp/en/products/detail/koa-speer-electronics-inc/RK73Z2ATTD/10235990
- R3, R4: Link (none) -> https://www.digikey.jp/en/products/detail/yageo/RC0603JR-07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; MPN (none) -> RC0603JR-070RL
- R6, R7, R8: value 4.75K -> 4.7K; Link (none) -> https://www.digikey.jp/en/products/detail/yageo/RC0603JR-07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
Changed lines of the file:
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@@
       (effects (font (size 1.27 1.27)) hide)
     )
-    (property "Datasheet" "~" (at 179.705 182.88 0)
+    (property "Datasheet" "https://www.yageo.com/upload/media/product/app/datasheet/rchip/pyu-rc_group_51_rohs_l.pdf" (at 179.705 182.88 0)
       (effects (font (size 1.27 1.27)) hide)
     )
@@
       (effects (font (size 1.27 1.27)) hide)
     )
+    (property "Description" "470 Ohms ±5% 0.1W, 1/10W Chip Resistor 0603 (1608 Metric) Moisture Resistant Thick Film" (at 179.705 182.88 0)
+      (effects (font (size 1.27 1.27)) hide)
+    )
+    (property "Link" "https://www.digikey.jp/en/products/detail/yageo/RC0603JR-07470RL/726791?s=N4IgTCBcDaIEoGEAMA2JBmAUnAtEg7ACz5JwAyIAugL5A" (at 179.705 182.88 0)
+      (effects (font (size 1.27 1.27)) hide)
+    )
     (pin "1")
     (pin "2")
@@
       (effects (font (size 1.27 1.27)) hide)
     )
-    (property "Datasheet" "~" (at 103.505 181.61 0)
+    (property "Datasheet" "https://www.yageo.com/upload/media/product/app/datasheet/rchip/pyu-rc_group_51_rohs_l.pdf" (at 103.505 181.61 0)
       (effects (font (size 1.27 1.27)) hide)
     )
@@
       (effects (font (size 1.27 1.27)) hide)
     )
+    (property "Description" "470 Ohms ±5% 0.1W, 1/10W Chip Resistor 0603 (1608 Metric) Moisture Resistant Thick Film" (at 103.505 181.61 0)
+      (effects (font (size 1.27 1.27)) hide)
+    )
+    (property "Link" "https://www.digikey.jp/en/products/detail/yageo/RC0603JR-07470RL/726791?s=N4IgTCBcDaIEoGEAMA2JBmAUnAtEg7ACz5JwAyIAugL5A" (at 103.505 181.61 0)
+      (effects (font (size 1.27 1.27)) hide)
+    )
     (pin "1")
     (pin "2")
@@
       (effects (font (size 1.27 1.27)) hide)
     )
-    (property "Datasheet" "~" (at 243.205 190.5 0)
+    (property "Datasheet" "https://www.yageo.com/upload/media/product/productsearch/datasheet/rchip/PYu-RC_Group_51_RoHS_L_12.pdf" (at 243.205 190.5 0)
       (effects (font (size 1.27 1.27)) hide)
     )
     (property "MPN" "RC0603JR-071K5L" (at 243.205 190.5 0)
+      (effects (font (size 1.27 1.27)) hide)
+    )
+    (property "Description" "1.5 kOhms ±5% 0.1W, 1/10W Chip Resistor 0603 (1608 Metric) Moisture Resistant Thick Film" (at 243.205 190.5 0)
+      (effects (font (size 1.27 1.27)) hide)
+    )
+    (property "Link" "https://www.digikey.jp/en/products/detail/yageo/RC0603JR-071K5L/726689?s=N4IgTCBcDaIEoGEAMA2JBmAUnAtEg7AIwDSArADIgC6AvkA" (at 243.205 190.5 0)
       (effects (font (size 1.27 1.27)) hide)
     )
@@
       (effects (font (size 1.27 1.27)) hide)
     )
-    (property "Datasheet" "~" (at 271.78 177.8 90)
+    (property "Datasheet" "https://www.puiaudio.com/media/SpecSheet/AI-1027-TWT-5V-2-R.pdf" (at 271.78 177.8 90)
       (effects (font (size 1.27 1.27)) hide)
     )
     (property "MPN" "AI-1027-TWT-5V-2-R " (at 272.415 180.34 0)
+      (effects (font (size 1.27 1.27)) hide)
+    )
+    (property "Description" "Buzzers Indicator, Internally Driven Electromechanical/Magnetic 5 V 30mA 2.73kHz 82dB @ 5V, 10cm Through Hole PC Pins" (at 272.415 180.34 0)
+      (effects (font (size 1.27 1.27)) hide)
+    )
+    (property "Link" "https://www.digikey.jp/en/products/detail/pui-audio-inc/AI-1027-TWT-5V-2-R/5011389?s=N4IgTCBcDaIIIEkC0BGADGA7EgKgdRyQFYA1JMJAJQAIQBdAXyA" (at 272.415 180.34 0)
       (effects (font (size 1.27 1.27)) hide)
     )
@@
       (effects (font (size 1.27 1.27) italic) (justify left) hide)
     )
-    (property "Datasheet" "https://www.fairchildsemi.com/datasheets/BS/BSS138.pdf" (at 267.335 190.5 0)
+    (property "Datasheet" "https://mm.digikey.com/Volume0/opasdata/d220001/medias/docus/3037/BSS138.pdf" (at 267.335 190.5 0)
       (effects (font (size 1.27 1.27)) (justify left) hide)
     )
     (property "MPN" "BSS138" (at 267.335 190.5 0)
+      (effects (font (size 1.27 1.27)) hide)
+    )
+    (property "Description" "N-Channel 50 V 220mA (Ta) 350mW (Ta) Surface Mount SOT-23" (at 267.335 190.5 0)
+      (effects (font (size 1.27 1.27)) hide)
+    )
+    (property "Link" "https://www.digikey.jp/en/products/detail/anbon-semiconductor-int-l-limited/BSS138/16708474" (at 267.335 190.5 0)
       (effects (font (size 1.27 1.27)) hide)
     )
@@
       (effects (font (size 1.27 1.27)))
     )
-    (property "Value" "4.75K" (at 264.795 146.05 90)
+    (property "Value" "4.7K" (at 264.795 146.05 90)
       (effects (font (size 1.27 1.27)))
     )
@@
       (effects (font (size 1.27 1.27)) hide)
     )
-    (property "Datasheet" "~" (at 267.335 146.05 0)
+    (property "Datasheet" "https://www.yageo.com/upload/media/product/productsearch/datasheet/rchip/PYu-RC_Group_51_RoHS_L_12.pdf" (at 267.335 146.05 0)
       (effects (font (size 1.27 1.27)) hide)
     )
@@
       (effects (font (size 1.27 1.27)) hide)
     )
+    (property "Description" "4.7 kOhms ±5% 0.1W, 1/10W Chip Resistor 0603 (1608 Metric) Moisture Resistant Thick Film" (at 267.335 146.05 0)
+      (effects (font (size 1.27 1.27)) hide)
+    )
+    (property "Link" "https://www.digikey.jp/en/products/detail/yageo/RC0603JR-074K7L/726785?s=N4IgTCBcDaIEoGEAMA2JBmAUnAtEg7ACwDS%2BAMiALoC%2BQA" (at 267.335 146.05 0)
+      (effects (font (size 1.27 1.27)) hide)
+    )
     (pin "1")
     (pin "2")
@@
       (effects (font (size 1.27 1.27)))
     )
-    (property "Value" "4.75K" (at 254.635 146.05 90)
+    (property "Value" "4.7K" (at 254.635 146.05 90)
       (effects (font (size 1.27 1.27)))
     )
@@
       (effects (font (size 1.27 1.27)) hide)
     )
-    (property "Datasheet" "~" (at 257.175 146.05 0)
+    (property "Datasheet" "https://www.yageo.com/upload/media/product/productsearch/datasheet/rchip/PYu-RC_Group_51_RoHS_L_12.pdf" (at 257.175 146.05 0)
       (effects (font (size 1.27 1.27)) hide)
     )
@@
       (effects (font (size 1.27 1.27)) hide)
     )
+    (property "Description" "4.7 kOhms ±5% 0.1W, 1/10W Chip Resistor 0603 (1608 Metric) Moisture Resistant Thick Film" (at 257.175 146.05 0)
+      (effects (font (size 1.27 1.27)) hide)
+    )
+    (property "Link" "https://www.digikey.jp/en/products/detail/yageo/RC0603JR-074K7L/726785?s=N4IgTCBcDaIEoGEAMA2JBmAUnAtEg7ACwDS%2BAMiALoC%2BQA" (at 257.175 146.05 0)
+      (effects (font (size 1.27 1.27)) hide)
+    )
     (pin "1")
     (pin "2")
@@
       (effects (font (size 1.27 1.27)))
     )
-    (property "Value" "4.75K" (at 258.445 163.83 90)
+    (property "Value" "4.7K" (at 258.445 163.83 90)
       (effects (font (size 1.27 1.27)))
     )
@@
       (effects (font (size 1.27 1.27)) hide)
     )
-    (property "Datasheet" "~" (at 260.985 163.83 0)
+    (property "Datasheet" "https://www.yageo.com/upload/media/product/productsearch/datasheet/rchip/PYu-RC_Group_51_RoHS_L_12.pdf" (at 260.985 163.83 0)
       (effects (font (size 1.27 1.27)) hide)
     )
     (property "MPN" "RC0603JR-074K7L" (at 260.985 163.83 0)
+      (effects (font (size 1.27 1.27)) hide)
+    )
+    (property "Description" "4.7 kOhms ±5% 0.1W, 1/10W Chip Resistor 0603 (1608 Metric) Moisture Resistant Thick Film" (at 260.985 163.83 0)
+      (effects (font (size 1.27 1.27)) hide)
+    )
+    (property "Link" "https://www.digikey.jp/en/products/detail/yageo/RC0603JR-074K7L/726785?s=N4IgTCBcDaIEoGEAMA2JBmAUnAtEg7ACwDS%2BAMiALoC%2BQA" (at 260.985 163.83 0)
       (effects (font (size 1.27 1.27)) hide)
     )
@@
       (effects (font (size 1.27 1.27)) hide)
     )
-    (property "Datasheet" "~" (at 234.315 125.73 0)
-      (effects (font (size 1.27 1.27)) hide)
-    )
-    (property "MPN" "" (at 234.315 125.73 0)
+    (property "Datasheet" "https://www.yageo.com/upload/media/product/productsearch/datasheet/rchip/PYu-RC_Group_51_RoHS_L_12.pdf" (at 234.315 125.73 0)
+      (effects (font (size 1.27 1.27)) hide)
+    )
+    (property "MPN" "RC0603JR-070RL" (at 234.315 125.73 0)
+      (effects (font (size 1.27 1.27)) hide)
+    )
+    (property "Description" "0 Ohms Jumper Chip Resistor 0603 (1608 Metric) Moisture Resistant Thick Film" (at 234.315 125.73 0)
+      (effects (font (size 1.27 1.27)) hide)
+    )
+    (property "Link" "https://www.digikey.jp/en/products/detail/yageo/RC0603JR-070RL/726675?s=N4IgTCBcDaIEoGEAMA2JBmAUnAtEg7EnADIgC6AvkA" (at 234.315 125.73 0)
       (effects (font (size 1.27 1.27)) hide)
     )
@@
       (effects (font (size 1.27 1.27)) hide)
     )
-    (property "Datasheet" "~" (at 234.315 123.19 0)
-      (effects (font (size 1.27 1.27)) hide)
-    )
-    (property "MPN" "" (at 234.315 123.19 0)
+    (property "Datasheet" "https://www.yageo.com/upload/media/product/productsearch/datasheet/rchip/PYu-RC_Group_51_RoHS_L_12.pdf" (at 234.315 123.19 0)
+      (effects (font (size 1.27 1.27)) hide)
+    )
+    (property "MPN" "RC0603JR-070RL" (at 234.315 123.19 0)
+      (effects (font (size 1.27 1.27)) hide)
+    )
+    (property "Description" "0 Ohms Jumper Chip Resistor 0603 (1608 Metric) Moisture Resistant Thick Film" (at 234.315 123.19 0)
+      (effects (font (size 1.27 1.27)) hide)
+    )
+    (property "Link" "https://www.digikey.jp/en/products/detail/yageo/RC0603JR-070RL/726675?s=N4IgTCBcDaIEoGEAMA2JBmAUnAtEg7EnADIgC6AvkA" (at 234.315 123.19 0)
       (effects (font (size 1.27 1.27)) hide)
     )
@@
       (effects (font (size 1.27 1.27)) hide)
     )
-    (property "Link" "https://www.digikey.jp/en/products/detail/koa-speer-electronics-inc/RK73Z2ATTD/10235990?s=N4IgTCBcDaIEoGkDsBmAWmAggFWwERAF0BfIA" (at 305.435 196.85 0)
+    (property "Link" "https://www.digikey.jp/en/products/detail/koa-speer-electronics-inc/RK73Z2ATTD/10235990" (at 305.435 196.85 0)
       (effects (font (size 1.27 1.27)) hide)
     )
@@
       (effects (font (size 1.27 1.27)) hide)
     )
-    (property "Value" "teTra" (at 330.454 253.111 0)
+    (property "Value" "teTra /NC" (at 330.454 253.111 0)
       (effects (font (size 1.27 1.27)) hide)
     )
@@
   )
   (sheet_instances
-    (path "/" (page "16"))
+    (path "/" (page "1"))
   )
 )

Commit message: Add files via upload
Parts:
- removed R104: 0R, Resistor_SMD:R_0805_2012Metric, symbol Device:R_Small
Changed lines of the file:
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@@
-    (stroke (width 0) (type default))
-  )
-  (wire (pts (xy 311.785 196.85) (xy 307.975 196.85))
     (stroke (width 0) (type default))
   )
@@
     (stroke (width 0) (type default))
   )
-  (wire (pts (xy 299.72 196.85) (xy 299.72 198.12))
-    (stroke (width 0) (type default))
-  )
   (wire (pts (xy 103.505 195.58) (xy 103.505 198.12))
     (stroke (width 0) (type default))
@@
     (stroke (width 0.508) (type default))
   )
-  (wire (pts (xy 311.785 198.12) (xy 311.785 196.85))
-    (stroke (width 0) (type default))
-  )
   (wire (pts (xy 179.705 196.85) (xy 179.705 199.39))
     (stroke (width 0) (type default))
@@
   )
   (wire (pts (xy 252.095 190.5) (xy 262.255 190.5))
-    (stroke (width 0) (type default))
-  )
-  (wire (pts (xy 302.895 196.85) (xy 299.72 196.85))
     (stroke (width 0) (type default))
   )
@@
     )
   )
-  (symbol (lib_id "power:GNDA") (at 109.22 128.27 0) (unit 1)
-    (in_bom yes) (on_board yes) (dnp no)
-    (property "Reference" "#PWR04" (at 109.22 134.62 0)
-      (effects (font (size 1.27 1.27)) hide)
-    )
-    (property "Value" "GNDA" (at 109.347 132.6642 0)
-      (effects (font (size 1.27 1.27)))
-    )
-    (property "Footprint" "" (at 109.22 128.27 0)
-      (effects (font (size 1.27 1.27)) hide)
-    )
-    (property "Datasheet" "" (at 109.22 128.27 0)
-      (effects (font (size 1.27 1.27)) hide)
-    )
-    (pin "1")
-    (instances
-      (project "LTC6811_ESP32"
-        (path "/6a86ff6f-b159-4c4c-8a40-e732cc82e010"
-          (reference "#PWR04") (unit 1)
-        )
-      )
-    )
-  )
-  (symbol (lib_id "power:GND_PACK") (at 299.72 198.12 0) (unit 1)
-    (in_bom yes) (on_board yes) (dnp no) (fields_autoplaced)
-    (property "Reference" "#PWR079" (at 299.72 204.47 0)
-      (effects (font (size 1.27 1.27)) hide)
-    )
-    (property "Value" "GND_PACK" (at 299.72 202.565 0)
-      (effects (font (size 1.27 1.27)))
-    )
-    (property "Footprint" "" (at 299.72 198.12 0)
-      (effects (font (size 1.27 1.27)) hide)
-    )
-    (property "Datasheet" "" (at 299.72 198.12 0)
-      (effects (font (size 1.27 1.27)) hide)
-    )
-    (pin "1")
-    (instances
-      (project "LTC6811_ESP32"
-        (path "/6a86ff6f-b159-4c4c-8a40-e732cc82e010/0999518d-09c3-4a69-bd78-ff81b3ce8dd2"
-          (reference "#PWR079") (unit 1)
-        )
-        (path "/6a86ff6f-b159-4c4c-8a40-e732cc82e010"
-          (reference "#PWR098") (unit 1)
-        )
-      )
-    )
-  )
   (symbol (lib_id "BMS-Master-rescue:R-Device-BMS-Master-rescue") (at 234.315 125.73 90) (unit 1)
     (in_bom yes) (on_board yes) (dnp no)
@@
         (path "/6a86ff6f-b159-4c4c-8a40-e732cc82e010"
           (reference "R4") (unit 1)
-        )
-      )
-    )
-  )
-  (symbol (lib_id "BMS-Master-rescue:GND-power-BMS-Master-rescue") (at 311.785 198.12 0) (unit 1)
-    (in_bom yes) (on_board yes) (dnp no)
-    (property "Reference" "#PWR05" (at 311.785 204.47 0)
-      (effects (font (size 1.27 1.27)) hide)
-    )
-    (property "Value" "GND" (at 311.912 202.5142 0)
-      (effects (font (size 1.27 1.27)))
-    )
-    (property "Footprint" "" (at 311.785 198.12 0)
-      (effects (font (size 1.27 1.27)) hide)
-    )
-    (property "Datasheet" "" (at 311.785 198.12 0)
-      (effects (font (size 1.27 1.27)) hide)
-    )
-    (pin "1")
-    (instances
-      (project "LTC6811_ESP32"
-        (path "/6a86ff6f-b159-4c4c-8a40-e732cc82e010"
-          (reference "#PWR05") (unit 1)
         )
       )
@@
     )
   )
+  (symbol (lib_id "BMS-Master-rescue:GND-power-BMS-Master-rescue") (at 109.22 128.27 0) (unit 1)
+    (in_bom yes) (on_board yes) (dnp no)
+    (property "Reference" "#PWR04" (at 109.22 134.62 0)
+      (effects (font (size 1.27 1.27)) hide)
+    )
+    (property "Value" "GND" (at 109.347 132.6642 0)
+      (effects (font (size 1.27 1.27)))
+    )
+    (property "Footprint" "" (at 109.22 128.27 0)
+      (effects (font (size 1.27 1.27)) hide)
+    )
+    (property "Datasheet" "" (at 109.22 128.27 0)
+      (effects (font (size 1.27 1.27)) hide)
+    )
+    (pin "1")
+    (instances
+      (project "LTC6811_ESP32"
+        (path "/6a86ff6f-b159-4c4c-8a40-e732cc82e010"
+          (reference "#PWR04") (unit 1)
+        )
+      )
+    )
+  )
   (symbol (lib_id "Device:LED") (at 179.705 193.04 270) (unit 1)
     (in_bom yes) (on_board yes) (dnp no)
@@
         )
       )
-    )
-  )
-  (symbol (lib_id "Device:R_Small") (at 305.435 196.85 270) (unit 1)
-    (in_bom yes) (on_board yes) (dnp no)
-    (property "Reference" "R104" (at 303.53 194.945 90)
-      (effects (font (size 1.27 1.27)) (justify left))
-    )
-    (property "Value" "0R" (at 307.975 195.58 90)
-      (effects (font (size 1.27 1.27) (color 255 19 38 1)) (justify left) hide)
-    )
-    (property "Footprint" "Resistor_SMD:R_0805_2012Metric" (at 305.435 196.85 0)
-      (effects (font (size 1.27 1.27)) hide)
-    )
-    (property "Datasheet" "https://www.koaspeer.com/pdfs/RK73Z.pdf" (at 305.435 196.85 0)
-      (effects (font (size 1.27 1.27)) hide)
-    )
-    (property "Description" "0 Ohms Jumper Chip Resistor 0805 (2012 Metric) Automotive AEC-Q200, Moisture Resistant Metal Element" (at 305.435 196.85 0)
-      (effects (font (size 1.27 1.27)) hide)
-    )
-    (property "Link" "https://www.digikey.jp/en/products/detail/koa-speer-electronics-inc/RK73Z2ATTD/10235990" (at 305.435 196.85 0)
-      (effects (font (size 1.27 1.27)) hide)
-    )
-    (property "MPN" "RK73Z2ATTD" (at 305.435 196.85 0)
-      (effects (font (size 1.27 1.27)) hide)
-    )
-    (pin "1")
-    (pin "2")
-    (instances
-      (project "LTC6811_ESP32"
-        (path "/6a86ff6f-b159-4c4c-8a40-e732cc82e010"
-          (reference "R104") (unit 1)
-        )
-      )
-      (project "L9963E+ESP32_V1.0"
-        (path "/e9bba7f0-c10d-45df-9f8e-74901087917a"
-          (reference "R50") (unit 1)
-        )
-      )
