File: CAN.kicad_sch (KiCad schematic)
At the start: 8 parts, among them U8 ISO1050DUBR, U9 SFH617A-2X009T

Commit message: Add files via upload
Parts:
- removed R116: 2.2k, Resistor_SMD:R_0603_1608Metric, symbol BMS-Master-rescue:R-Device-BMS-Master-rescue
- removed U9: SFH617A-2X009T, Housings_DIP:SMDIP-4_W9.53mm_Clearance8mm, symbol Isolator:SFH617A-2X017T
- D8: renamed from D4; footprint TO_SOT_Packages_SMD:SOT-23 -> Package_TO_SOT_SMD:SOT-23
- U11: renamed from U8; footprint ENNOID:ISO1050 -> Package_SO:SOP-8_6.62x9.15mm_P2.54mm
- renumbered C43 to C42, C44 to C43, C46 to C44, C47 to C45
Other:
- company: (none) -> teTra
- moved on the sheet: C42, C43, C44, C45, D8, U11

Commit message: Add files via upload
Parts:
- C42, C44: value 1u -> 1uF 25V; Link (none) -> https://www.digikey.jp/en/products/detail/nextgen-component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; MPN GRM188R71E105KA12D -> 0603B105K250XD
- C43: value 100n -> 100nF 100V; Link (none) -> https://www.digikey.jp/en/products/detail/samsung-electro-m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; MPN GRM188R71E104KA01D -> CL10B104KC8NNNC
- C45: value 100n -> 100nF 50V; Link (none) -> https://www.digikey.jp/en/products/detail/nextgen-component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; MPN GRM188R71E104KA01D -> 0603B104K500XD
- D8: value SZNUP2105L -> ESD24VS2U; Link (none) -> https://www.digikey.jp/en/products/detail/infineon-technolo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; MPN SZNUP2105LT1G -> ESD24VS2UE6327HTSA1
Changed lines of the file:
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@@
       (effects (font (size 1.27 1.27)) (justify left))
     )
-    (property "Value" "100n" (at 51.816 54.483 0)
+    (property "Value" "100nF 100V" (at 51.816 54.483 0)
       (effects (font (size 1.27 1.27)) (justify left))
     )
@@
       (effects (font (size 1.27 1.27)) hide)
     )
-    (property "Datasheet" "~" (at 48.895 53.34 0)
-      (effects (font (size 1.27 1.27)) hide)
-    )
-    (property "MPN" "GRM188R71E104KA01D" (at 48.895 53.34 0)
+    (property "Datasheet" "https://www.digikey.jp/en/products/detail/samsung-electro-mechanics/CL10B104KC8NNNC/5961291?s=N4IgTCBcDaIMIBkCMAGAQqgLAaTgDgDki4AdEkAXQF8g" (at 48.895 53.34 0)
+      (effects (font (size 1.27 1.27)) hide)
+    )
+    (property "MPN" "CL10B104KC8NNNC" (at 48.895 53.34 0)
+      (effects (font (size 1.27 1.27)) hide)
+    )
+    (property "Description" "0.1 µF ±10% 100V Ceramic Capacitor X7R 0603 (1608 Metric)" (at 48.895 53.34 0)
+      (effects (font (size 1.27 1.27)) hide)
+    )
+    (property "Link" "https://www.digikey.jp/en/products/detail/samsung-electro-mechanics/CL10B104KC8NNNC/5961291?s=N4IgTCBcDaIMIBkCMAGAQqgLAaTgDgDki4QBdAXyA" (at 48.895 53.34 0)
       (effects (font (size 1.27 1.27)) hide)
     )
@@
       (effects (font (size 1.27 1.27)) (justify left))
     )
-    (property "Value" "1u" (at 40.386 54.483 0)
+    (property "Value" "1uF 25V" (at 40.386 54.483 0)
       (effects (font (size 1.27 1.27)) (justify left))
     )
@@
       (effects (font (size 1.27 1.27)) hide)
     )
-    (property "Datasheet" "~" (at 37.465 53.34 0)
-      (effects (font (size 1.27 1.27)) hide)
-    )
-    (property "MPN" "GRM188R71E105KA12D" (at 37.465 53.34 0)
+    (property "Datasheet" "https://mm.digikey.com/Volume0/opasdata/d220001/medias/docus/4562/0603B105K250XD.pdf" (at 37.465 53.34 0)
+      (effects (font (size 1.27 1.27)) hide)
+    )
+    (property "MPN" "0603B105K250XD" (at 37.465 53.34 0)
+      (effects (font (size 1.27 1.27)) hide)
+    )
+    (property "Description" "1 µF ±10% 25V Ceramic Capacitor X7R 0603 (1608 Metric)" (at 37.465 53.34 0)
+      (effects (font (size 1.27 1.27)) hide)
+    )
+    (property "Link" "https://www.digikey.jp/en/products/detail/nextgen-components/0603B105K250XD/14670931" (at 37.465 53.34 0)
       (effects (font (size 1.27 1.27)) hide)
     )
@@
       (effects (font (size 1.27 1.27)))
     )
-    (property "Value" "100n" (at 134.8994 40.64 90)
+    (property "Value" "100nF 50V" (at 134.8994 40.64 90)
       (effects (font (size 1.27 1.27)))
     )
@@
       (effects (font (size 1.27 1.27)) hide)
     )
-    (property "Datasheet" "~" (at 130.81 40.64 0)
-      (effects (font (size 1.27 1.27)) hide)
-    )
-    (property "MPN" "GRM188R71E104KA01D" (at 130.81 40.64 0)
+    (property "Datasheet" "https://mm.digikey.com/Volume0/opasdata/d220001/medias/docus/4564/0603B104K500XD.pdf" (at 130.81 40.64 0)
+      (effects (font (size 1.27 1.27)) hide)
+    )
+    (property "MPN" "0603B104K500XD" (at 130.81 40.64 0)
+      (effects (font (size 1.27 1.27)) hide)
+    )
+    (property "Description" "0.1 µF ±10% 50V Ceramic Capacitor X7R 0603 (1608 Metric)" (at 130.81 40.64 0)
+      (effects (font (size 1.27 1.27)) hide)
+    )
+    (property "Link" "https://www.digikey.jp/en/products/detail/nextgen-components/0603B104K500XD/15761336" (at 130.81 40.64 0)
       (effects (font (size 1.27 1.27)) hide)
     )
@@
       (effects (font (size 1.27 1.27)) (justify left))
     )
-    (property "Value" "1u" (at 124.841 41.783 0)
+    (property "Value" "1uF 25V" (at 124.841 41.783 0)
       (effects (font (size 1.27 1.27)) (justify left))
     )
@@
       (effects (font (size 1.27 1.27)) hide)
     )
-    (property "Datasheet" "~" (at 121.92 40.64 0)
-      (effects (font (size 1.27 1.27)) hide)
-    )
-    (property "MPN" "GRM188R71E105KA12D" (at 121.92 40.64 0)
+    (property "Datasheet" "https://mm.digikey.com/Volume0/opasdata/d220001/medias/docus/4562/0603B105K250XD.pdf" (at 121.92 40.64 0)
+      (effects (font (size 1.27 1.27)) hide)
+    )
+    (property "MPN" "0603B105K250XD" (at 121.92 40.64 0)
+      (effects (font (size 1.27 1.27)) hide)
+    )
+    (property "Description" "1 µF ±10% 25V Ceramic Capacitor X7R 0603 (1608 Metric)" (at 121.92 40.64 0)
+      (effects (font (size 1.27 1.27)) hide)
+    )
+    (property "Link" "https://www.digikey.jp/en/products/detail/nextgen-components/0603B105K250XD/14670931" (at 121.92 40.64 0)
       (effects (font (size 1.27 1.27)) hide)
     )
@@
       (effects (font (size 1.27 1.27)) (justify left))
     )
-    (property "Value" "SZNUP2105L" (at 136.652 64.643 0)
+    (property "Value" "ESD24VS2U" (at 136.652 64.643 0)
       (effects (font (size 1.27 1.27)) (justify left))
     )
@@
       (effects (font (size 1.27 1.27)) (justify left) hide)
     )
-    (property "Datasheet" "http://www.onsemi.com/pub_link/Collateral/NUP2105L-D.PDF" (at 134.62 60.325 0)
-      (effects (font (size 1.27 1.27)) hide)
-    )
-    (property "MPN" "SZNUP2105LT1G" (at 131.445 63.5 0)
-      (effects (font (size 1.27 1.27)) hide)
-    )
+    (property "Datasheet" "https://www.infineon.com/dgdl/Infineon-ESD24VS2U-DS-v01_01-en.pdf?fileId=db3a3043340fff53013413a2249d2ff3" (at 134.62 60.325 0)
+      (effects (font (size 1.27 1.27)) hide)
+    )
+    (property "MPN" "ESD24VS2UE6327HTSA1" (at 131.445 63.5 0)
+      (effects (font (size 1.27 1.27)) hide)
+    )
+    (property "Description" "41V Clamp 5A (8/20µs) Ipp Tvs Diode Surface Mount PG-SOT23" (at 131.445 63.5 0)
+      (effects (font (size 1.27 1.27)) hide)
+    )
+    (property "Link" "https://www.digikey.jp/en/products/detail/infineon-technologies/ESD24VS2UE6327HTSA1/1785650" (at 131.445 63.5 0)
+      (effects (font (size 1.27 1.27)) hide)
+    )

Commit message: Add files via upload
Parts:
- U11: Link (none) -> https://www.digikey.jp/en/products/detail/texas-instruments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
Changed lines of the file:
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@@
       (effects (font (size 1.27 1.27)) hide)
     )
-    (property "Datasheet" "" (at 93.345 62.23 0)
+    (property "Datasheet" "https://www.ti.com/general/docs/suppproductinfo.tsp?distId=10&gotoUrl=https%3A%2F%2Fwww.ti.com%2Flit%2Fgpn%2Fiso1050" (at 93.345 62.23 0)
       (effects (font (size 1.27 1.27)) hide)
     )
@@
       (effects (font (size 1.27 1.27)) hide)
     )
+    (property "Description" "1/1 Transceiver, Isolated Half CANbus 8-SOP" (at 95.885 53.34 0)
+      (effects (font (size 1.27 1.27)) hide)
+    )
+    (property "Link" "https://www.digikey.jp/en/products/detail/texas-instruments/ISO1050DUBR/2094633?s=N4IgTCBcDaIJIGUDyBGADAVjQEQKoCEAlEAXQF8g" (at 95.885 53.34 0)
+      (effects (font (size 1.27 1.27)) hide)
+    )
