File: MCU.kicad_sch (KiCad schematic)
At the start: 30 parts, among them J17 DEBUG, J29 JTAG, J31 UART, Q27 BSS138, U13 ESP32-DevKitC V4, U17 STM32F303CCTx, U2 LTC6820, Y1 8MHz

Commit message: Add files via upload
Parts:
- removed C76, C77: 18p, Capacitor_SMD:C_0603_1608Metric, symbol BMS-Master-rescue:C-Device-BMS-Master-rescue
- removed C78, C81, C82, C83, C84: 100n, Capacitor_SMD:C_0603_1608Metric, symbol BMS-Master-rescue:C-Device-BMS-Master-rescue
- removed J17: DEBUG, Connector_Molex:Molex_PicoBlade_53398-0571_1x05-1MP_P1.25mm_Vertical, symbol BMS-Master-rescue:Conn_01x05-Connector_Generic-BMS-Master-rescue
- removed Q27: BSS138, TO_SOT_Packages_SMD:SOT-23, symbol BMS-Master-rescue:BSS138-Transistor_FET-BMS-Master-rescue
- removed R168: 10k, Resistor_SMD:R_0603_1608Metric, symbol BMS-Master-rescue:R-Device-BMS-Master-rescue
- removed R170: 100k, Resistor_SMD:R_0603_1608Metric, symbol BMS-Master-rescue:R-Device-BMS-Master-rescue
- removed U17: STM32F303CCTx, Housings_QFP:LQFP-48_7x7mm_Pitch0.5mm, symbol BMS-Master-rescue:STM32F303CCTx-MCU_ST_STM32-BMS-Master-rescue
- removed Y1: 8MHz, Crystals:Crystal_SMD_Abracon_ABM3-2pin_5.0x3.2mm, symbol BMS-Master-rescue:Crystal-Device-BMS-Master-rescue
- added J1: Boot Option, Connector_PinHeader_2.54mm:PinHeader_1x02_P2.54mm_Vertical, symbol Connector_Generic:Conn_01x02
Connections:
- net GND: now also J1.2 (Pin_2)
- net Boot: now reaches U13.25 (IO0)
- net Boot: now also J1.1 (Pin_1)
- no-connect marks 7 -> 4
Other:
- note removed: "DEBUG"
- moved on the sheet: C18, C19, C20, C6, C7, C8, J29, J31, R16, R36, R37, R5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

Commit message: Add files via upload
Parts:
- J5: renamed from J31; Link (none) -> https://www.digikey.jp/en/products/detail/samtec-inc/TSW-10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; MPN (none) -> TSW-104-07-G-S; 型号 TSW-104-07-G-S -> (none); 购买链接 https://www.digikey.jp/en/products/detail/samtec-inc/TSW-10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 -> (none)
- J6: renamed from J29; Link (none) -> https://www.digikey.jp/en/products/detail/samtec-inc/TSW-10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; MPN (none) -> TSW-104-07-G-S; 型号 TSW-104-07-G-S -> (none); 购买链接 https://www.digikey.jp/en/products/detail/samtec-inc/TSW-10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 -> (none)
- U8: renamed from U13; footprint RF_Module:ESP32-DevKitC V4 -> RF_Module:ESP32-DevKitc V4_DIP-38_27.9mm×48.2mm
- U9: renamed from U2; footprint Housings_SSOP:MSOP-16_3x4mm_Pitch0.5mm -> Package_SO:MSOP-16_3x4mm_P0.5mm
- renumbered C19 to C32, C18 to C33, C6 to C34, C7 to C35, C20 to C36, C8 to C37, J1 to J7, R16 to R43, R5 to R44, R6 to R45, R7 to R46, R36 to R47, R37 to R48
Connections:
- net PowerEnable: no longer names the net of U8.11 (IO27)
Other:
- company: (none) -> teTra

Commit message: Add files via upload
Parts:
- C32, C33: value 100nF -> 100nF 50V; footprint Capacitor_SMD:C_0603_1608Metric_Pad1.08x0.95mm_HandSolder -> Capacitor_SMD:C_0603_1608Metric; Link (none) -> https://www.digikey.jp/en/products/detail/nextgen-component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; MPN (none) -> 0603B104K500XD
- C34, C35: value 10n -> 10nF 100V; Link (none) -> https://www.digikey.jp/en/products/detail/murata-electronic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; MPN GRM188R71H103KA01D -> GCM188R72A103KA37D
- C36: value 1u -> 1uF 25V; Link (none) -> https://www.digikey.jp/en/products/detail/nextgen-component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; MPN GRM188R71E105KA12D -> 0603B105K250XD
- C37: value 100n -> 100nF 100V; Link (none) -> https://www.digikey.jp/en/products/detail/samsung-electro-m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; MPN GRM188R71E104KA01D -> CL10B104KC8NNNC; Voltage 25V -> (none)
- J5: value UART -> UART /NC
- J6: value JTAG -> JTAG /NC
- J7: value Boot Option -> Boot Option /C
- R44: value 806 -> 806R
- R47: value 1.2k -> 1.2K
- R48: value 2k -> 2K
Connections:
- net MISO: now also U8.31 (IO19); no longer U8.37 (IO23)
- net MOSI: now also U8.37 (IO23); no longer U8.31 (IO19)

Commit message: Add files via upload
Parts:
- J7: value Boot Option /C -> Boot Option /NC
- R43: footprint Resistor_SMD:R_0603_1608Metric_Pad0.98x0.95mm_HandSolder -> Resistor_SMD:R_0603_1608Metric; Link (none) -> https://www.digikey.jp/en/products/detail/stackpole-electro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; MPN (none) -> RMCF0603FT10K0
- R44, R48: Link (none) -> https://www.digikey.jp/en/products/detail/yageo/RC0603FR-07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
- R45, R46: value 51 -> 51R; Link (none) -> https://www.digikey.jp/en/products/detail/yageo/RC0603JR-07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
- R47: Link (none) -> https://www.digikey.jp/en/products/detail/yageo/RC0603JR-07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
- TR2: Link (none) -> https://www.digikey.jp/en/products/detail/pulse-electronics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
- U8: Link (none) -> https://www.digikey.jp/en/products/detail/espressif-systems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; MPN (none) -> ESP32-DEVKITC-32E
- U9: Link (none) -> https://www.digikey.jp/en/products/detail/analog-devices-in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
Changed lines of the file:
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@@
     )
   )
-  (text "12位ADC最小测量电压为0.8mV" (at 74.295 188.595 0)
+  (text "12位ADC最小测量电压为0.8mV" (at 69.215 184.15 0)
     (effects (font (size 1.27 1.27)) (justify left bottom))
   )
@@
       (effects (font (size 1.27 1.27)))
     )
-    (property "Value" "51" (at 97.5614 50.165 90)
+    (property "Value" "51R" (at 97.5614 50.165 90)
       (effects (font (size 1.27 1.27)))
     )
@@
       (effects (font (size 1.27 1.27)) hide)
     )
-    (property "Datasheet" "~" (at 94.615 50.165 0)
+    (property "Datasheet" "https://www.yageo.com/upload/media/product/productsearch/datasheet/rchip/PYu-RC_Group_51_RoHS_L_12.pdf" (at 94.615 50.165 0)
       (effects (font (size 1.27 1.27)) hide)
     )
@@
       (effects (font (size 1.27 1.27)) hide)
     )
+    (property "Description" "51 Ohms ±5% 0.1W, 1/10W Chip Resistor 0603 (1608 Metric) Moisture Resistant Thick Film" (at 94.615 50.165 0)
+      (effects (font (size 1.27 1.27)) hide)
+    )
+    (property "Link" "https://www.digikey.jp/en/products/detail/yageo/RC0603JR-0751RL/726803?s=N4IgTCBcDaIEoGEAMA2JBmAUnAtEg7AKwCMcAMiALoC%2BQA" (at 94.615 50.165 0)
+      (effects (font (size 1.27 1.27)) hide)
+    )
     (pin "1")
     (pin "2")
@@
       (effects (font (size 1.27 1.27)))
     )
-    (property "Value" "51" (at 97.5614 60.325 90)
+    (property "Value" "51R" (at 97.5614 60.325 90)
       (effects (font (size 1.27 1.27)))
     )
@@
       (effects (font (size 1.27 1.27)) hide)
     )
-    (property "Datasheet" "~" (at 94.615 60.325 0)
+    (property "Datasheet" "https://www.yageo.com/upload/media/product/productsearch/datasheet/rchip/PYu-RC_Group_51_RoHS_L_12.pdf" (at 94.615 60.325 0)
       (effects (font (size 1.27 1.27)) hide)
     )
     (property "MPN" "RC0603JR-0751RL" (at 94.615 60.325 0)
+      (effects (font (size 1.27 1.27)) hide)
+    )
+    (property "Description" "51 Ohms ±5% 0.1W, 1/10W Chip Resistor 0603 (1608 Metric) Moisture Resistant Thick Film" (at 94.615 60.325 0)
+      (effects (font (size 1.27 1.27)) hide)
+    )
+    (property "Link" "https://www.digikey.jp/en/products/detail/yageo/RC0603JR-0751RL/726803?s=N4IgTCBcDaIEoGEAMA2JBmAUnAtEg7AKwCMcAMiALoC%2BQA" (at 94.615 60.325 0)
       (effects (font (size 1.27 1.27)) hide)
     )
@@
       (effects (font (size 1.27 1.27)) hide)
     )
-    (property "Link" "" (at 45.085 60.325 0)
+    (property "Link" "https://www.digikey.jp/en/products/detail/pulse-electronics/HM2108NL/7914611" (at 45.085 60.325 0)
       (effects (font (size 1.27 1.27)) hide)
     )
@@
       (effects (font (size 1.27 1.27)) hide)
     )
-    (property "Datasheet" "~" (at 102.235 67.945 0)
+    (property "Datasheet" "https://www.yageo.com/upload/media/product/productsearch/datasheet/rchip/PYu-RC_Group_51_RoHS_L_12.pdf" (at 102.235 67.945 0)
       (effects (font (size 1.27 1.27)) hide)
     )
@@
       (effects (font (size 1.27 1.27)) hide)
     )
+    (property "Description" "1.2 kOhms ±5% 0.1W, 1/10W Chip Resistor 0603 (1608 Metric) Moisture Resistant Thick Film" (at 102.235 67.945 0)
+      (effects (font (size 1.27 1.27)) hide)
+    )
+    (property "Link" "https://www.digikey.jp/en/products/detail/yageo/RC0603JR-071K2L/726683?s=N4IgTCBcDaIEoGEAMA2JBmAUnAtEg7AIwDSYAMiALoC%2BQA" (at 102.235 67.945 0)
+      (effects (font (size 1.27 1.27)) hide)
+    )
     (pin "1")
     (pin "2")
@@
       (effects (font (size 1.27 1.27)) hide)
     )
-    (property "Datasheet" "~" (at 88.265 67.945 0)
+    (property "Datasheet" "https://www.yageo.com/upload/media/product/app/datasheet/rchip/pyu-rc_group_51_rohs_l.pdf" (at 88.265 67.945 0)
       (effects (font (size 1.27 1.27)) hide)
     )
     (property "MPN" "RC0603FR-07806RL" (at 88.265 67.945 0)
+      (effects (font (size 1.27 1.27)) hide)
+    )
+    (property "Description" "806 Ohms ±1% 0.1W, 1/10W Chip Resistor 0603 (1608 Metric) Moisture Resistant Thick Film" (at 88.265 67.945 0)
+      (effects (font (size 1.27 1.27)) hide)
+    )
+    (property "Link" "https://www.digikey.jp/en/products/detail/yageo/RC0603FR-07806RL/727397?s=N4IgTCBcDaIEoGEAMA2JBmAYnAtEg7ABypwAyIAugL5A" (at 88.265 67.945 0)
       (effects (font (size 1.27 1.27)) hide)
     )
@@
       (effects (font (size 1.27 1.27)) hide)
     )
-    (property "Datasheet" "" (at 127.635 81.915 0)
+    (property "Datasheet" "https://www.analog.com/media/en/technical-documentation/data-sheets/LTC6820.pdf" (at 127.635 81.915 0)
       (effects (font (size 1.27 1.27)) hide)
     )
     (property "MPN" "LTC6820IMS#PBF " (at 127.635 69.215 0)
+      (effects (font (size 1.27 1.27)) hide)
+    )
+    (property "Description" "Isolated Communications Interface Interface 16-MSOP" (at 127.635 69.215 0)
+      (effects (font (size 1.27 1.27)) hide)
+    )
+    (property "Link" "https://www.digikey.jp/en/products/detail/analog-devices-inc/LTC6820IMS-PBF/3838555?s=N4IgTCBcDaIDIBUDCA2AHGADASQLIGUBiABQCEAxAAhAF0BfIA" (at 127.635 69.215 0)
       (effects (font (size 1.27 1.27)) hide)
     )
@@
       (effects (font (size 1.27 1.27)) hide)
     )
-    (property "Datasheet" "~" (at 160.655 69.215 0)
+    (property "Datasheet" "https://www.yageo.com/upload/media/product/app/datasheet/rchip/pyu-rc_group_51_rohs_l.pdf" (at 160.655 69.215 0)
       (effects (font (size 1.27 1.27)) hide)
     )
     (property "MPN" "RC0603FR-072KL" (at 160.655 69.215 0)
+      (effects (font (size 1.27 1.27)) hide)
+    )
+    (property "Description" "2 kOhms ±1% 0.1W, 1/10W Chip Resistor 0603 (1608 Metric) Moisture Resistant Thick Film" (at 160.655 69.215 0)
+      (effects (font (size 1.27 1.27)) hide)
+    )
+    (property "Link" "https://www.digikey.jp/en/products/detail/yageo/RC0603FR-072KL/727009?s=N4IgTCBcDaIEoGEAMA2JBmAYnAtEg7GANIAyIAugL5A" (at 160.655 69.215 0)
       (effects (font (size 1.27 1.27)) hide)
     )
@@
       (effects (font (size 1.27 1.27)) (justify left))
     )
-    (property "Footprint" "Resistor_SMD:R_0603_1608Metric_Pad0.98x0.95mm_HandSolder" (at 34.925 132.715 0)
-      (effects (font (size 1.27 1.27)) hide)
-    )
-    (property "Datasheet" "~" (at 34.925 132.715 0)
+    (property "Footprint" "Resistor_SMD:R_0603_1608Metric" (at 34.925 132.715 0)
+      (effects (font (size 1.27 1.27)) hide)
+    )
+    (property "Datasheet" "https://www.seielect.com/catalog/sei-rmcf_rmcp.pdf" (at 34.925 132.715 0)
+      (effects (font (size 1.27 1.27)) hide)
+    )
+    (property "Description" "10 kOhms ±1% 0.1W, 1/10W Chip Resistor 0603 (1608 Metric) Automotive AEC-Q200 Thick Film" (at 34.925 132.715 0)
+      (effects (font (size 1.27 1.27)) hide)
+    )
+    (property "Link" "https://www.digikey.jp/en/products/detail/stackpole-electronics-inc/RMCF0603FT10K0/1761235?s=N4IgTCBcDaIEoFkDCAxADANjQZhQFQEY0BpNEAXQF8g" (at 34.925 132.715 0)
+      (effects (font (size 1.27 1.27)) hide)
+    )
+    (property "MPN" "RMCF0603FT10K0" (at 34.925 132.715 0)
       (effects (font (size 1.27 1.27)) hide)
     )
@@
       (effects (font (size 1.27 1.27) italic) hide)
     )
-    (property "Datasheet" "https://mm.digikey.com/Volume0/opasdata/d220001/medias/docus/3656/ESP32-S3-WROOM-1_1U_v0.5.1_Preliminary.pdf" (at 80.645 121.666 0)
+    (property "Datasheet" "https://mm.digikey.com/Volume0/opasdata/d220001/medias/docus/754/ESP32-DevKitC_GSG_Ver1.4_2017.pdf" (at 80.645 121.666 0)
       (effects (font (size 1.27 1.27) italic) hide)
+    )
+    (property "Description" "- ESP32-WROOM-32E Transceiver; 802.11 b/g/n (Wi-Fi, WiFi, WLAN), Bluetooth® Smart Ready 4.x Dual Mode 2.4GHz Evaluation Board" (at 80.645 152.4 0)
+      (effects (font (size 1.27 1.27)) hide)
+    )
+    (property "Link" "https://www.digikey.jp/en/products/detail/espressif-systems/ESP32-DEVKITC-32E/12091810" (at 80.645 152.4 0)
+      (effects (font (size 1.27 1.27)) hide)
+    )
+    (property "MPN" "ESP32-DEVKITC-32E" (at 80.645 152.4 0)
+      (effects (font (size 1.27 1.27)) hide)
     )
     (pin "23")
@@
       (effects (font (size 1.27 1.27)) (justify left))
     )
-    (property "Value" "Boot Option /C" (at 143.51 181.61 0)
+    (property "Value" "Boot Option /NC" (at 143.51 181.61 0)
       (effects (font (size 1.27 1.27)) (justify left) hide)
     )
