File: PowerMonitor.kicad_sch (KiCad schematic)
At the start: 61 parts, among them U1 AMC1301 or AMC1302, U12 AMC1301, U15 OPA2197IDR, U16 ISL28022, U3 TPS76350, U4 SN6501DBV

Commit message: Add files via upload
Parts:
- removed R119, R122, R125: 470K, Resistor_SMD:R_1206_3216Metric, symbol BMS-Master-rescue:R-Device-BMS-Master-rescue
- added R17, R20, R21: 470kΩ ±0.1% 250mW, Resistor_SMD:R_0805_2012Metric, symbol BMS-Master-rescue:R-Device-BMS-Master-rescue
- R129: value 1k -> 1kΩ ±0.1% 250mW; footprint Resistor_SMD:R_0603_1608Metric -> Resistor_SMD:R_0805_2012Metric; Link (none) -> https://www.digikey.jp/en/products/detail/panasonic-electro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; MPN MCR03EZPFX1001 -> ERJ-PB6B1001V
- R19: value 470K -> 470kΩ ±0.1% 250mW; footprint Resistor_SMD:R_1206_3216Metric -> Resistor_SMD:R_0805_2012Metric; Link (none) -> https://www.digikey.jp/en/products/detail/panasonic-electro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; MPN RC1206FR-07470KL -> ERJ-PB6B4703V
Connections:
- net at R19.2: now also R17.1
- net at R129.1, R22.1: now also R21.2
- new net: R17.2, R20.1
- new net: R20.2, R21.1
Other:
- moved on the sheet: C1, C10, C11, C12, C13, C14, C15, C16, C2, C3, C4, C49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

Commit message: Add files via upload
Parts:
- added unit 2 of U5
- D4: renamed from D14; footprint Diodes_SMD:D_SOD-123 -> Diode_SMD:D_SOD-123
- D5: renamed from D15; footprint Diodes_SMD:D_SOD-123 -> Diode_SMD:D_SOD-123
- U2: renamed from U1; footprint Housings_SOIC:SSO-8_6.8x5.9mm_Pitch1.27mm_Clearance8mm -> Package_SO:SSO-8_6.8x5.9mm_P1.27mm_Clearance8mm
- U3: renamed from U12; footprint Housings_SOIC:SSO-8_6.8x5.9mm_Pitch1.27mm_Clearance8mm -> Package_SO:SSO-8_6.8x5.9mm_P1.27mm_Clearance8mm; Link (none) -> https://www.digikey.jp/en/products/detail/texas-instruments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
- U5: renamed from U15; footprint Housings_SOIC:SOIC-8_3.9x4.9mm_Pitch1.27mm -> PCM_4ms_Package_SOIC:SOIC-8_3.9x4.9mm_Pitch1.27mm
- U6: renamed from U16; footprint Housings_SSOP:MSOP-10_3x3mm_Pitch0.5mm -> PCM_4ms_Package_SSOP:MSOP-10_3x3mm_P0.5mm; Link (none) -> https://www.digikey.jp/en/products/detail/renesas-electroni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
- renumbered D5 to D3, R26 to R10, R17 to R11, R20 to R12, R29 to R13, R21 to R14, R129 to R15, R30 to R16, R31 to R17, R132 to R18, R22 to R19, R35 to R20, R38 to R21, R142 to R22, R143 to R23, R39 to R24, R40 to R25, R148 to R26, R149 to R27, R155 to R28, R156 to R29, R14 to R30, R15 to R31, R13 to R32, R160 to R33, R164 to R34, R166 to R35, R167 to R36, R19 to R9, U3 to U1
Connections:
- no-connect marks 3 -> 6
Other:
- company: (none) -> teTra

Commit message: Add files via upload
Parts:
- removed C16: 1u, Capacitor_SMD:C_0603_1608Metric, symbol BMS-Master-rescue:C-Device
- removed C75: 100n, Capacitor_SMD:C_0603_1608Metric, symbol BMS-Master-rescue:C-Device
- removed D3: POWER, LED_SMD:LED_0603_1608Metric, symbol BMS-Master-rescue:LED-Device-BMS-Master-rescue
- removed unit 3 of U5
- added D3: LED Red, LED_SMD:LED_0603_1608Metric, symbol Device:LED
- C1, C2: value 10u -> 10uF 25V; Link (none) -> https://www.digikey.jp/en/products/detail/samsung-electro-m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
- C10, C68: value 220p -> 220pF 50V; Link (none) -> https://www.digikey.jp/en/products/detail/murata-electronic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; MPN GRM1555C1H221JA01D -> GCM1885C1H221JA16D
- C11, C13, C14, C3, C4, C52, C58, C72, C73: value 100n -> 100nF 100V; Link (none) -> https://www.digikey.jp/en/products/detail/samsung-electro-m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; MPN GRM188R71E104KA01D -> CL10B104KC8NNNC
- C12, C49: value 330p -> 330pF 100V; Link (none) -> https://search.murata.co.jp/Ceramy/image/img/A01X/G101/ENG/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; MPN CL10B331KB8NNNC -> GRM188R72A331KA01D
- C15, C62: value 2.2u -> 2.2uF 16V; Link (none) -> https://www.digikey.jp/en/products/detail/kemet/C0603C225K4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; MPN GRM188R61A225KE34D -> C0603C225K4PAC7867; Voltage 50V -> (none)
- C5: value 10u -> 10uF 25V; footprint Capacitor_SMD:C_0603_1608Metric -> Capacitor_SMD:C_0805_2012Metric; Link (none) -> https://www.digikey.jp/en/products/detail/samsung-electro-m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; MPN CL10A106MQ8NNNC -> CL21A106KAYNNNE
- C65, C9: value 2.2n -> 2.2nF 16V; Link (none) -> https://www.digikey.jp/en/products/detail/kemet/C0603C222K4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; MPN GRM1885C1H222JA01D -> C0603C222K4RECAUTO
- C67: value 100nF -> 100nF 100V
- D4, D5: Link (none) -> https://www.digikey.jp/en/products/detail/micro-commercial-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; MPN MBR0502L -> MBR0520-TP
- R10: value 470 -> 470R
- R11, R12, R14, R9: value 470kΩ ±0.1% 250mW -> 470KΩ ±0.1% 250mW
- R15: value 1kΩ ±0.1% 250mW -> 1KΩ ±0.1% 250mW
- R16, R17, R18, R24, R25, R26, R27, R32: value 1k -> 1K
- R19: value 10 -> 10R
- R20, R21, R22, R23: value 100 -> 100R
- R28, R29: value 5.6k -> 5.6K
- R30, R31: value 3.3k -> 3.3K
- R35, R36: value 4.75k -> 4.75K
Connections:
- net GNDA: now also D3.1 (K)
- net at R10.1: now also D3.2 (A)

Commit message: Add files via upload
Parts:
- added BAT-1, BAT1: BAT-, Battery:Battery_6mm×10mm_Cell_half_2, symbol Connector_Generic:Conn_01x01
- R10, R19, R28, R29: Link (none) -> https://www.digikey.jp/en/products/detail/yageo/RC0603JR-07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
- R13: value 0.1MR 1% 2W 4020 -> 0.1MR 1% 15W; Link https://www.mouser.jp/ProductDetail/ROHM-Semiconductor/PSR5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 -> https://www.digikey.jp/en/products/detail/rohm-semiconducto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
- R15: Link https://www.digikey.jp/en/products/detail/panasonic-electronic-components/ERJ-PB6B1001V/6213377?s=N4IgTCBcDaIKICUBSAFAQgNjQRgAy%2BwDUQBdAXyA -> https://www.digikey.jp/en/products/detail/panasonic-electronic-components/ERJ-PB6B1001V/6213377?s=N4IgTCBcDaIKICUBSBaACgIQGwYIwAZ9cA1EAXQF8g
- R16, R17, R18, R24, R25, R26, R27, R32: Link (none) -> https://www.digikey.jp/en/products/detail/vishay-dale/CRCW0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; MPN MCR03EZPFX1001 -> CRCW06031K00FKEA
- R20, R21, R22, R23, R30, R31, R33, R34: Link (none) -> https://www.digikey.jp/en/products/detail/yageo/RC0603FR-07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
- R35, R36: value 4.75K -> 4.7K; Link (none) -> https://www.digikey.jp/en/products/detail/yageo/RC0603JR-07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
- TR1: Link (none) -> https://www.digikey.jp/en/products/detail/w%C3%BCrth-elektr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
- U1, U2, U4, U5: Link (none) -> https://www.digikey.jp/en/products/detail/texas-instruments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
- U5: footprint Housings_SOIC:SOIC-8_3.9x4.9mm_Pitch1.27mm -> PCM_4ms_Package_SOIC:SOIC-8_3.9x4.9mm_Pitch1.27mm; Link (none) -> https://www.digikey.jp/en/products/detail/texas-instruments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
Connections:
- net BAT-: now also BAT-1.1 (Pin_1)
- net GND_PACK: now also BAT1.1 (Pin_1)

Commit message: Add files via upload
Connections:
- net BAT- is gone; now on net GND: BAT-1.1 (Pin_1), R13.2, R17.1
- net GNDA is gone; now on net GND_PACK: C1.2, C13.2, C2.2, C3.2, C52.2, D3.1 (K), R15.2, R18.2, TR1.2, U1.2 (GND), U2.4 (GND2), U3.4 (GND2)
- net Vbat: now also U5.7; no longer U5.1
- net at R29.2, R33.1: now also U5.5 (+); no longer U5.3 (+)
- net at R28.2, R34.1: now also U5.6 (-); no longer U5.2 (-)
Other:
- moved on the sheet: BAT-1, BAT1

Commit message: Add files via upload
Parts:
- R17: footprint Resistor_SMD:R_0603_1608Metric -> Resistor_SMD:R_2010_5025Metric; Link https://www.digikey.jp/en/products/detail/vishay-dale/CRCW0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 -> https://www.digikey.jp/en/products/detail/yageo/RC2010JK-07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; MPN CRCW06031K00FKEA -> RC2010JK-071KL
Changed lines of the file:
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@@
       (effects (font (size 1.27 1.27)))
     )
-    (property "Footprint" "Resistor_SMD:R_0603_1608Metric" (at 123.19 189.103 90)
+    (property "Footprint" "Resistor_SMD:R_2010_5025Metric" (at 123.19 189.103 90)
       (effects (font (size 1.27 1.27)) hide)
     )
-    (property "Datasheet" "https://www.vishay.com/docs/20035/dcrcwe3.pdf" (at 123.19 187.325 0)
+    (property "Datasheet" "https://www.yageo.com/upload/media/product/productsearch/datasheet/rchip/PYu-RC_Group_51_RoHS_L_12.pdf" (at 123.19 187.325 0)
       (effects (font (size 1.27 1.27)) hide)
     )
-    (property "MPN" "CRCW06031K00FKEA" (at 123.19 187.325 0)
+    (property "MPN" "RC2010JK-071KL" (at 123.19 187.325 0)
       (effects (font (size 1.27 1.27)) hide)
     )
-    (property "Description" "1 kOhms ±1% 0.1W, 1/10W Chip Resistor 0603 (1608 Metric) Automotive AEC-Q200 Thick Film" (at 123.19 187.325 0)
+    (property "Description" "1 kOhms ±5% 0.75W, 3/4W Chip Resistor 2010 (5025 Metric) Moisture Resistant Thick Film" (at 123.19 187.325 0)
       (effects (font (size 1.27 1.27)) hide)
     )
-    (property "Link" "https://www.digikey.jp/en/products/detail/vishay-dale/CRCW06031K00FKEA/1179809" (at 123.19 187.325 0)
+    (property "Link" "https://www.digikey.jp/en/products/detail/yageo/RC2010JK-071KL/5921660" (at 123.19 187.325 0)
       (effects (font (size 1.27 1.27)) hide)
     )
