File: USB.kicad_sch (KiCad schematic)
At the start: 12 parts, among them J14 SERIAL, Q26 BSS138, U7 CP2104

Commit message: Add files via upload
Parts:
- removed Q26: BSS138, TO_SOT_Packages_SMD:SOT-23, symbol Transistor_FET:BSS138
- D7: renamed from D3; footprint TO_SOT_Packages_SMD:SOT-23 -> Package_TO_SOT_SMD:SOT-23
- J8: renamed from J14; footprint Connectors_Molex:Molex_KK-6410-05_05x2.54mm_Straight -> Connector_PinHeader_2.54mm:PinHeader_1x05_P2.54mm_Vertical
- U10: renamed from U7; footprint Housings_DFN_QFN:QFN-24-1EP_4x4mm_Pitch0.5mm -> Package_DFN_QFN:HVQFN-24-1EP_4x4mm_P0.5mm_EP2.6x2.6mm; Link (none) -> https://www.digikey.jp/en/products/detail/silicon-labs/CP21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
- renumbered R111 to R49, R112 to R50, R113 to R51, R114 to R52
Other:
- company: (none) -> teTra
- moved on the sheet: C39, C40, C41, C42, D7, J8, R49, R50, R51, R52, U10

Commit message: Add files via upload
Parts:
- removed D7: SP0502BAHT, Package_TO_SOT_SMD:SOT-23, symbol Power_Protection:SP0502BAHT
- added D8: ESD24VS2U, Package_TO_SOT_SMD:SOT-23, symbol Power_Protection:SZNUP2105L
- C39, C40, C42: value 2.2u -> 2.2uF 16V; Link (none) -> https://www.digikey.jp/en/products/detail/kemet/C0603C225K4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; MPN GRM188R61A225KE34D -> C0603C225K4PAC7867; Voltage 50V -> (none)
- C41: value 100n -> 100nF 100V; Link (none) -> https://www.digikey.jp/en/products/detail/samsung-electro-m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; MPN GRM188R71E104KA01D -> CL10B104KC8NNNC
- J8: value SERIAL -> SERIAL /NC
- R49, R50: value 240 -> 240R
- R51, R52: value 10k -> 10K
Connections:
- net D+: now also D8.2 (K)
- net D-: now also D8.1 (K)
- net GND: now also D8.3 (A)
Changed lines of the file:
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@@
       (effects (font (size 1.27 1.27)))
     )
-    (property "Value" "240" (at 64.77 55.245 90)
+    (property "Value" "240R" (at 64.77 55.245 90)
       (effects (font (size 1.27 1.27)))
     )
@@
       (effects (font (size 1.27 1.27)))
     )
-    (property "Value" "240" (at 64.77 57.785 90)
+    (property "Value" "240R" (at 64.77 57.785 90)
       (effects (font (size 1.27 1.27)))
     )
@@
     )
   )
-  (symbol (lib_id "Power_Protection:SP0502BAHT") (at 143.51 73.025 0) (unit 1)
-    (in_bom yes) (on_board yes) (dnp no)
-    (property "Reference" "D7" (at 148.717 71.8566 0)
-      (effects (font (size 1.27 1.27)) (justify left))
-    )
-    (property "Value" "SP0502BAHT" (at 148.717 74.168 0)
-      (effects (font (size 1.27 1.27)) (justify left))
-    )
-    (property "Footprint" "Package_TO_SOT_SMD:SOT-23" (at 149.225 74.295 0)
-      (effects (font (size 1.27 1.27)) (justify left) hide)
-    )
-    (property "Datasheet" "http://www.littelfuse.com/~/media/files/littelfuse/technical%20resources/documents/data%20sheets/sp05xxba.pdf" (at 146.685 69.85 0)
-      (effects (font (size 1.27 1.27)) hide)
-    )
-    (property "MPN" "SP0502BAHTG" (at 143.51 73.025 0)
-      (effects (font (size 1.27 1.27)) hide)
-    )
-    (pin "3")
-    (pin "1")
-    (pin "2")
-    (instances
-      (project "LTC6811_ESP32"
-        (path "/6a86ff6f-b159-4c4c-8a40-e732cc82e010/00000000-0000-0000-0000-00005c246ca0"
-          (reference "D7") (unit 1)
-        )
-      )
-    )
-  )
   (symbol (lib_id "power:GND") (at 143.51 80.645 0) (unit 1)
     (in_bom yes) (on_board yes) (dnp no)
@@
       (effects (font (size 1.27 1.27)))
     )
-    (property "Value" "10k" (at 78.74 73.025 90)
+    (property "Value" "10K" (at 78.74 73.025 90)
       (effects (font (size 1.27 1.27)))
     )
@@
       (effects (font (size 1.27 1.27)) (justify left))
     )
-    (property "Value" "2.2u" (at 129.921 85.598 0)
+    (property "Value" "2.2uF 16V" (at 129.921 85.598 0)
       (effects (font (size 1.27 1.27)) (justify left))
     )
@@
       (effects (font (size 1.27 1.27)) hide)
     )
-    (property "Datasheet" "~" (at 127 84.455 0)
-      (effects (font (size 1.27 1.27)) hide)
-    )
-    (property "MPN" "GRM188R61A225KE34D" (at 127 84.455 0)
-      (effects (font (size 1.27 1.27)) hide)
-    )
-    (property "Voltage" "50V" (at 127 84.455 0)
+    (property "Datasheet" "https://connect.kemet.com:7667/gateway/IntelliData-ComponentDocumentation/1.0/download/datasheet/C0603C225K4PACTU" (at 127 84.455 0)
+      (effects (font (size 1.27 1.27)) hide)
+    )
+    (property "MPN" "C0603C225K4PAC7867" (at 127 84.455 0)
+      (effects (font (size 1.27 1.27)) hide)
+    )
+    (property "Description" "2.2 µF ±10% 16V Ceramic Capacitor X5R 0603 (1608 Metric)" (at 127 84.455 0)
+      (effects (font (size 1.27 1.27)) hide)
+    )
+    (property "Link" "https://www.digikey.jp/en/products/detail/kemet/C0603C225K4PAC7867/2200308" (at 127 84.455 0)
       (effects (font (size 1.27 1.27)) hide)
     )
@@
       (effects (font (size 1.27 1.27)) (justify left))
     )
-    (property "Value" "2.2u" (at 82.931 36.703 0)
+    (property "Value" "2.2uF 16V" (at 82.931 36.703 0)
       (effects (font (size 1.27 1.27)) (justify left))
     )
@@
       (effects (font (size 1.27 1.27)) hide)
     )
-    (property "Datasheet" "~" (at 80.01 35.56 0)
-      (effects (font (size 1.27 1.27)) hide)
-    )
-    (property "MPN" "GRM188R61A225KE34D" (at 80.01 35.56 0)
-      (effects (font (size 1.27 1.27)) hide)
-    )
-    (property "Voltage" "50V" (at 80.01 35.56 0)
+    (property "Datasheet" "https://connect.kemet.com:7667/gateway/IntelliData-ComponentDocumentation/1.0/download/datasheet/C0603C225K4PACTU" (at 80.01 35.56 0)
+      (effects (font (size 1.27 1.27)) hide)
+    )
+    (property "MPN" "C0603C225K4PAC7867" (at 80.01 35.56 0)
+      (effects (font (size 1.27 1.27)) hide)
+    )
+    (property "Description" "2.2 µF ±10% 16V Ceramic Capacitor X5R 0603 (1608 Metric)" (at 80.01 35.56 0)
+      (effects (font (size 1.27 1.27)) hide)
+    )
+    (property "Link" "https://www.digikey.jp/en/products/detail/kemet/C0603C225K4PAC7867/2200308" (at 80.01 35.56 0)
       (effects (font (size 1.27 1.27)) hide)
     )
@@
       (effects (font (size 1.27 1.27)) (justify left))
     )
-    (property "Value" "2.2u" (at 146.431 43.688 0)
+    (property "Value" "2.2uF 16V" (at 146.431 43.688 0)
       (effects (font (size 1.27 1.27)) (justify left))
     )
@@
       (effects (font (size 1.27 1.27)) hide)
     )
-    (property "Datasheet" "~" (at 143.51 42.545 0)
-      (effects (font (size 1.27 1.27)) hide)
-    )
-    (property "MPN" "GRM188R61A225KE34D" (at 143.51 42.545 0)
-      (effects (font (size 1.27 1.27)) hide)
-    )
-    (property "Voltage" "50V" (at 143.51 42.545 0)
+    (property "Datasheet" "https://connect.kemet.com:7667/gateway/IntelliData-ComponentDocumentation/1.0/download/datasheet/C0603C225K4PACTU" (at 143.51 42.545 0)
+      (effects (font (size 1.27 1.27)) hide)
+    )
+    (property "MPN" "C0603C225K4PAC7867" (at 143.51 42.545 0)
+      (effects (font (size 1.27 1.27)) hide)
+    )
+    (property "Description" "2.2 µF ±10% 16V Ceramic Capacitor X5R 0603 (1608 Metric)" (at 143.51 42.545 0)
+      (effects (font (size 1.27 1.27)) hide)
+    )
+    (property "Link" "https://www.digikey.jp/en/products/detail/kemet/C0603C225K4PAC7867/2200308" (at 143.51 42.545 0)
       (effects (font (size 1.27 1.27)) hide)
     )
@@
       (effects (font (size 1.27 1.27)) (justify left))
     )
-    (property "Value" "100n" (at 136.271 43.688 0)
+    (property "Value" "100nF 100V" (at 136.271 43.688 0)
       (effects (font (size 1.27 1.27)) (justify left))
     )
@@
       (effects (font (size 1.27 1.27)) hide)
     )
-    (property "Datasheet" "~" (at 133.35 42.545 0)
-      (effects (font (size 1.27 1.27)) hide)
-    )
-    (property "MPN" "GRM188R71E104KA01D" (at 133.35 42.545 0)
+    (property "Datasheet" "https://www.digikey.jp/en/products/detail/samsung-electro-mechanics/CL10B104KC8NNNC/5961291?s=N4IgTCBcDaIMIBkCMAGAQqgLAaTgDgDki4AdEkAXQF8g" (at 133.35 42.545 0)
+      (effects (font (size 1.27 1.27)) hide)
+    )
+    (property "MPN" "CL10B104KC8NNNC" (at 133.35 42.545 0)
+      (effects (font (size 1.27 1.27)) hide)
+    )
+    (property "Description" "0.1 µF ±10% 100V Ceramic Capacitor X7R 0603 (1608 Metric)" (at 133.35 42.545 0)
+      (effects (font (size 1.27 1.27)) hide)
+    )
+    (property "Link" "https://www.digikey.jp/en/products/detail/samsung-electro-mechanics/CL10B104KC8NNNC/5961291?s=N4IgTCBcDaIMIBkCMAGAQqgLAaTgDgDki4QBdAXyA" (at 133.35 42.545 0)
       (effects (font (size 1.27 1.27)) hide)
     )
@@
       (effects (font (size 1.27 1.27)))
     )
-    (property "Value" "10k" (at 161.29 43.815 0)
+    (property "Value" "10K" (at 161.29 43.815 0)
       (effects (font (size 1.27 1.27)))
     )
@@
       (effects (font (size 1.27 1.27)) (justify left))
     )
-    (property "Value" "SERIAL" (at 56.642 88.2396 0)
+    (property "Value" "SERIAL /NC" (at 56.642 88.2396 0)
       (effects (font (size 1.27 1.27)) (justify left))
     )
@@
         )
       )
+    )
+  )
+  (symbol (lib_id "Power_Protection:SZNUP2105L") (at 143.51 73.025 0) (unit 1)
+    (in_bom yes) (on_board yes) (dnp no)
+    (property "Reference" "D8" (at 148.717 71.8566 0)
+      (effects (font (size 1.27 1.27)) (justify left))
+    )
+    (property "Value" "ESD24VS2U" (at 148.717 74.168 0)
+      (effects (font (size 1.27 1.27)) (justify left))
+    )
+    (property "Footprint" "Package_TO_SOT_SMD:SOT-23" (at 149.225 74.295 0)
+      (effects (font (size 1.27 1.27)) (justify left) hide)
+    )
+    (property "Datasheet" "https://www.infineon.com/dgdl/Infineon-ESD24VS2U-DS-v01_01-en.pdf?fileId=db3a3043340fff53013413a2249d2ff3" (at 146.685 69.85 0)
+      (effects (font (size 1.27 1.27)) hide)
+    )
+    (property "MPN" "ESD24VS2UE6327HTSA1" (at 143.51 73.025 0)
+      (effects (font (size 1.27 1.27)) hide)
+    )
+    (property "Description" "41V Clamp 5A (8/20µs) Ipp Tvs Diode Surface Mount PG-SOT23" (at 143.51 73.025 0)
+      (effects (font (size 1.27 1.27)) hide)
+    )
+    (property "Link" "https://www.digikey.jp/en/products/detail/infineon-technologies/ESD24VS2UE6327HTSA1/1785650" (at 143.51 73.025 0)
+      (effects (font (size 1.27 1.27)) hide)
+    )
+    (pin "3")
+    (pin "1")
+    (pin "2")
+    (instances
+      (project "LTC6811_ESP32"
+        (path "/6a86ff6f-b159-4c4c-8a40-e732cc82e010/00000000-0000-0000-0000-00005a91e16c"
+          (reference "D8") (unit 1)
+        )
+        (path "/6a86ff6f-b159-4c4c-8a40-e732cc82e010/00000000-0000-0000-0000-00005c246ca0"
+          (reference "D7") (unit 1)
+        )
+      )

Commit message: Add files via upload
Parts:
- R49, R50: Link (none) -> https://www.digikey.jp/en/products/detail/yageo/RC0603FR-07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
- R51, R52: Link (none) -> https://www.digikey.jp/en/products/detail/stackpole-electro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; MPN RC0603FR-0710KL -> RMCF0603FT10K0
Changed lines of the file:
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@@
+      (effects (font (size 1.27 1.27)) hide)
+    )
+    (property "Description" "USB Bridge, USB to UART USB 2.0 UART Interface 24-QFN (4x4)" (at 106.68 59.055 0)
       (effects (font (size 1.27 1.27)) hide)
     )
@@
       (effects (font (size 1.27 1.27)) hide)
     )
-    (property "Datasheet" "~" (at 69.85 56.515 0)
+    (property "Datasheet" "https://www.yageo.com/upload/media/product/app/datasheet/rchip/pyu-rc_group_51_rohs_l.pdf" (at 69.85 56.515 0)
       (effects (font (size 1.27 1.27)) hide)
     )
@@
       (effects (font (size 1.27 1.27)) hide)
     )
+    (property "Description" "240 Ohms ±1% 0.1W, 1/10W Chip Resistor 0603 (1608 Metric) Moisture Resistant Thick Film" (at 69.85 56.515 0)
+      (effects (font (size 1.27 1.27)) hide)
+    )
+    (property "Link" "https://www.digikey.jp/en/products/detail/yageo/RC0603FR-07240RL/727081?s=N4IgTCBcDaIEoGEAMA2JBmAYnAtEg7GACxJwAyIAugL5A" (at 69.85 56.515 0)
+      (effects (font (size 1.27 1.27)) hide)
+    )
     (pin "1")
     (pin "2")
@@
       (effects (font (size 1.27 1.27)) hide)
     )
-    (property "Datasheet" "~" (at 69.85 59.055 0)
+    (property "Datasheet" "https://www.yageo.com/upload/media/product/app/datasheet/rchip/pyu-rc_group_51_rohs_l.pdf" (at 69.85 59.055 0)
       (effects (font (size 1.27 1.27)) hide)
     )
@@
       (effects (font (size 1.27 1.27)) hide)
     )
+    (property "Description" "240 Ohms ±1% 0.1W, 1/10W Chip Resistor 0603 (1608 Metric) Moisture Resistant Thick Film" (at 69.85 59.055 0)
+      (effects (font (size 1.27 1.27)) hide)
+    )
+    (property "Link" "https://www.digikey.jp/en/products/detail/yageo/RC0603FR-07240RL/727081?s=N4IgTCBcDaIEoGEAMA2JBmAYnAtEg7GACxJwAyIAugL5A" (at 69.85 59.055 0)
+      (effects (font (size 1.27 1.27)) hide)
+    )
     (pin "1")
     (pin "2")
@@
       (effects (font (size 1.27 1.27)) hide)
     )
-    (property "Datasheet" "~" (at 73.66 71.755 0)
-      (effects (font (size 1.27 1.27)) hide)
-    )
-    (property "MPN" "RC0603FR-0710KL" (at 73.66 71.755 0)
+    (property "Datasheet" "https://www.seielect.com/catalog/sei-rmcf_rmcp.pdf" (at 73.66 71.755 0)
+      (effects (font (size 1.27 1.27)) hide)
+    )
+    (property "MPN" "RMCF0603FT10K0" (at 73.66 71.755 0)
+      (effects (font (size 1.27 1.27)) hide)
+    )
+    (property "Description" "10 kOhms ±1% 0.1W, 1/10W Chip Resistor 0603 (1608 Metric) Automotive AEC-Q200 Thick Film" (at 73.66 71.755 0)
+      (effects (font (size 1.27 1.27)) hide)
+    )
+    (property "Link" "https://www.digikey.jp/en/products/detail/stackpole-electronics-inc/RMCF0603FT10K0/1761235?s=N4IgTCBcDaIEoFkDCAxADANjQZhQFQEY0BpNEAXQF8g" (at 73.66 71.755 0)
       (effects (font (size 1.27 1.27)) hide)
     )
@@
       (effects (font (size 1.27 1.27)) hide)
     )
-    (property "Datasheet" "~" (at 157.48 42.545 0)
-      (effects (font (size 1.27 1.27)) hide)
-    )
-    (property "MPN" "RC0603FR-0710KL" (at 157.48 42.545 0)
-      (effects (font (size 1.27 1.27)) hide)
-    )
+    (property "Datasheet" "https://www.seielect.com/catalog/sei-rmcf_rmcp.pdf" (at 157.48 42.545 0)
+      (effects (font (size 1.27 1.27)) hide)
+    )
+    (property "MPN" "RMCF0603FT10K0" (at 157.48 42.545 0)
+      (effects (font (size 1.27 1.27)) hide)
+    )
+    (property "Description" "10 kOhms ±1% 0.1W, 1/10W Chip Resistor 0603 (1608 Metric) Automotive AEC-Q200 Thick Film" (at 157.48 42.545 0)
+      (effects (font (size 1.27 1.27)) hide)
+    )
+    (property "Link" "https://www.digikey.jp/en/products/detail/stackpole-electronics-inc/RMCF0603FT10K0/1761235?s=N4IgTCBcDaIEoFkDCAxADANjQZhQFQEY0BpNEAXQF8g" (at 157.48 42.545 0)
+      (effects (font (size 1.27 1.27)) hide)
+    )

Commit message: Add files via upload
Connections:
- net +3V3: now also J8.5 (Pin_5); no longer J8.1 (Pin_1)
- net GND: now also J8.1 (Pin_1); no longer J8.5 (Pin_5)
- net RXD: now also J8.2 (Pin_2); no longer J8.4 (Pin_4)
Changed lines of the file:
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@@
     )
   )
-  (symbol (lib_id "BMS-Master-rescue:Conn_01x05-Connector_Generic-BMS-Master-rescue") (at 54.61 86.995 0) (unit 1)
+  (symbol (lib_id "BMS-Master-rescue:Conn_01x05-Connector_Generic-BMS-Master-rescue") (at 54.61 86.995 0) (mirror x) (unit 1)
     (in_bom yes) (on_board yes) (dnp no)
-    (property "Reference" "J8" (at 56.642 85.9282 0)
+    (property "Reference" "J8" (at 56.642 88.0618 0)
       (effects (font (size 1.27 1.27)) (justify left))
     )
-    (property "Value" "SERIAL /NC" (at 56.642 88.2396 0)
+    (property "Value" "SERIAL /NC" (at 56.642 85.7504 0)
       (effects (font (size 1.27 1.27)) (justify left))
     )
