File: cell.kicad_sch (KiCad schematic)
At the start: 6 parts, among them Q11 TSM2323

Commit message: Add files via upload
Parts:
- removed Q11: TSM2323, TO_SOT_Packages_SMD:SOT-23, symbol Device:Q_PMOS_GSD
- added Q3: TSM2323, Package_TO_SOT_SMD:SOT-23, symbol Device:Q_PMOS_GSD
- renumbered C37 to C59, D24 to D13, R62 to R68, R63 to R69, R64 to R70
Connections:
- net C+: now also Q3.2 (S)
- net at R70.2: now also Q3.1 (G)
- net at R68.2: now also Q3.3 (D)
Other:
- company: (none) -> teTra
- moved on the sheet: C59, D13, R68, R69, R70

Commit message: Add files via upload
Parts:
- C59: value 100n -> 100nF 100V; Link (none) -> https://www.digikey.jp/en/products/detail/samsung-electro-m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; MPN CC0603KRX7R0BB104 -> CL10B104KC8NNNC
- D13: Link (none) -> https://www.digikey.jp/en/products/detail/nexperia-usa-inc/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
- R68: value 36 -> 36R
- R69: value 100 -> 100R
- R70: value 3.3k -> 3.3K
Connections:
- net GND renamed GND_PACK

Commit message: Add files via upload
Parts:
- Q3: Link (none) -> https://www.digikey.jp/en/products/detail/taiwan-semiconduc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
- R68: value 36R -> 36R 1W 2512; Link (none) -> https://www.digikey.jp/en/products/detail/stackpole-electro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
- R69: Link (none) -> https://www.digikey.jp/en/products/detail/yageo/RC0603FR-07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
- R70: Link (none) -> https://www.digikey.jp/en/products/detail/yageo/RC0603FR-07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; MPN RC0603JR-073K3L -> RC0603FR-073K3L
Changed lines of the file:
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@@
       (effects (font (size 1.27 1.27)) hide)
     )
-    (property "Datasheet" "~" (at 69.215 48.895 0)
+    (property "Datasheet" "https://www.taiwansemi.com/assets/uploads/datasheet/TSM2323_F15.pdf" (at 69.215 48.895 0)
       (effects (font (size 1.27 1.27)) hide)
     )
     (property "MPN" "TSM2323CX RFG " (at 69.215 48.895 0)
+      (effects (font (size 1.27 1.27)) hide)
+    )
+    (property "Description" "P-Channel 20 V 4.7A (Ta) 1.25W (Ta) Surface Mount SOT-23" (at 69.215 48.895 0)
+      (effects (font (size 1.27 1.27)) hide)
+    )
+    (property "Link" "https://www.digikey.jp/en/products/detail/taiwan-semiconductor-corporation/TSM2323CX-RFG/7360264?s=N4IgTCBcDaICoGUCyYDMaDCANABAJQDEBxHEAXQF8g" (at 69.215 48.895 0)
       (effects (font (size 1.27 1.27)) hide)
     )
@@
       (effects (font (size 1.27 1.27)) hide)
     )
-    (property "Datasheet" "~" (at 88.265 48.895 0)
-      (effects (font (size 1.27 1.27)) hide)
-    )
-    (property "MPN" "RC0603JR-073K3L" (at 88.265 48.895 0)
+    (property "Datasheet" "https://www.yageo.com/upload/media/product/app/datasheet/rchip/pyu-rc_group_51_rohs_l.pdf" (at 88.265 48.895 0)
+      (effects (font (size 1.27 1.27)) hide)
+    )
+    (property "MPN" "RC0603FR-073K3L" (at 88.265 48.895 0)
+      (effects (font (size 1.27 1.27)) hide)
+    )
+    (property "Description" "3.3 kOhms ±1% 0.1W, 1/10W Chip Resistor 0603 (1608 Metric) Moisture Resistant Thick Film" (at 88.265 48.895 0)
+      (effects (font (size 1.27 1.27)) hide)
+    )
+    (property "Link" "https://www.digikey.jp/en/products/detail/yageo/RC0603FR-073K3L/727126?s=N4IgTCBcDaIEoGEAMA2JBmAYnAtEg7OgNboAyIAugL5A" (at 88.265 48.895 0)
       (effects (font (size 1.27 1.27)) hide)
     )
@@
       (effects (font (size 1.27 1.27)) (justify right))
     )
-    (property "Value" "36R" (at 68.453 66.548 0)
+    (property "Value" "36R 1W 2512" (at 68.453 66.548 0)
       (effects (font (size 1.27 1.27)) (justify right))
     )
@@
       (effects (font (size 1.27 1.27)) hide)
     )
-    (property "Datasheet" "~" (at 66.675 65.405 0)
+    (property "Datasheet" "https://www.seielect.com/catalog/sei-rmcf_rmcp.pdf" (at 66.675 65.405 0)
       (effects (font (size 1.27 1.27)) hide)
     )
     (property "MPN" "RTT25360JTE" (at 66.675 65.405 0)
+      (effects (font (size 1.27 1.27)) hide)
+    )
+    (property "Description" "36 Ohms ±5% 1W Chip Resistor 2512 (6432 Metric) Automotive AEC-Q200 Thick Film" (at 66.675 65.405 0)
+      (effects (font (size 1.27 1.27)) hide)
+    )
+    (property "Link" "https://www.digikey.jp/en/products/detail/stackpole-electronics-inc/RMCF2512JT36R0/1716346" (at 66.675 65.405 0)
       (effects (font (size 1.27 1.27)) hide)
     )
@@
       (effects (font (size 1.27 1.27)) hide)
     )
-    (property "Datasheet" "~" (at 88.265 32.385 0)
+    (property "Datasheet" "https://www.yageo.com/upload/media/product/app/datasheet/rchip/pyu-rc_group_51_rohs_l.pdf" (at 88.265 32.385 0)
       (effects (font (size 1.27 1.27)) hide)
     )
@@
       (effects (font (size 1.27 1.27)) hide)
     )
+    (property "Description" "100 Ohms ±1% 0.1W, 1/10W Chip Resistor 0603 (1608 Metric) Moisture Resistant Thick Film" (at 88.265 32.385 0)
+      (effects (font (size 1.27 1.27)) hide)
+    )
+    (property "Link" "https://www.digikey.jp/en/products/detail/yageo/RC0603FR-07100RL/726888?s=N4IgTCBcDaIEoGEAMA2JBmAYnAtEg7AIxJJwAyIAugL5A" (at 88.265 32.385 0)
+      (effects (font (size 1.27 1.27)) hide)
+    )
