File: LTC6811_ESP32_V1.2/CAN.kicad_sch (KiCad schematic)
At the start: 6 parts, among them U11 ISO1050DUBR

Commit message: add BOM
Parts:
- C42, C44: value 1uF 25V -> 1uF/25V; symbol BMS-Master-rescue:C-Device-BMS-Master-rescue -> Device:C
- C43: value 100nF 100V -> 100nF/100V; symbol BMS-Master-rescue:C-Device-BMS-Master-rescue -> Device:C
- C45: value 100nF 50V -> 100nF/100V; symbol BMS-Master-rescue:C-Device-BMS-Master-rescue -> Device:C; Link https://www.digikey.jp/en/products/detail/nextgen-component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 -> https://www.digikey.jp/en/products/detail/samsung-electro-m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; MPN 0603B104K500XD -> CL10B104KC8NNNC
