File: LTC6811_ESP32_V1.2/MCU.kicad_sch (KiCad schematic)
At the start: 18 parts, among them J5 UART /NC, J6 JTAG /NC, J7 Boot Option /NC, U8 ESP32-DevKitC V4, U9 LTC6820

Commit message: Add files via upload
Changed lines of the file:
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@@
     (stroke (width 0) (type default))
   )
-  (wire (pts (xy 105.41 83.185) (xy 105.41 93.345))
+  (wire (pts (xy 106.045 83.185) (xy 106.045 93.345))
     (stroke (width 0) (type default))
   )
@@
     (stroke (width 0) (type default))
   )
-  (wire (pts (xy 112.395 46.355) (xy 94.615 46.355))
+  (wire (pts (xy 106.045 46.355) (xy 94.615 46.355))
     (stroke (width 0) (type default))
   )
@@
     (stroke (width 0) (type default))
   )
+  (wire (pts (xy 106.045 60.325) (xy 112.395 60.325))
+    (stroke (width 0) (type default))
+  )
   (wire (pts (xy 102.235 132.08) (xy 111.76 132.08))
     (stroke (width 0) (type default))
@@
     (stroke (width 0) (type default))
   )
-  (wire (pts (xy 105.41 93.345) (xy 112.395 93.345))
+  (wire (pts (xy 106.045 93.345) (xy 112.395 93.345))
     (stroke (width 0) (type default))
   )
@@
     (stroke (width 0.508) (type dash))
   )
-  (wire (pts (xy 112.395 46.355) (xy 112.395 60.325))
+  (wire (pts (xy 106.045 46.355) (xy 106.045 60.325))
     (stroke (width 0) (type default))
   )
@@
     (stroke (width 0) (type default))
   )
-  (wire (pts (xy 105.41 83.185) (xy 112.395 83.185))
-    (stroke (width 0) (type default))
-  )
+  (wire (pts (xy 106.045 83.185) (xy 112.395 83.185))
+    (stroke (width 0) (type default))
+  )

Commit message: Add files via upload
Connections:
- net MTCK: now also J6.4 (Pin_4); no longer J6.3 (Pin_3)
- net MTDO: now also J6.3 (Pin_3); no longer J6.4 (Pin_4)
- no-connect marks 4 -> 8
Other:
- moved on the sheet: C32, C33, J5, J6, J7, R43, U8

Commit message: Add files via upload
Connections:
- net CAN_RX: now also J5.2 (Pin_2); no longer J5.3 (Pin_3)
- net CAN_TX: now also J5.3 (Pin_3); no longer J5.2 (Pin_2)
Changed lines of the file:
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@@
     (effects (font (size 1.27 1.27)) (justify right bottom))
   )
-  (label "CAN_RX" (at 127.635 133.985 0) (fields_autoplaced)
+  (label "CAN_RX" (at 127.635 131.445 0) (fields_autoplaced)
     (effects (font (size 1.27 1.27)) (justify left bottom))
   )
@@
     (effects (font (size 1.27 1.27)) (justify left bottom))
   )
-  (label "CAN_TX" (at 127.635 131.445 0) (fields_autoplaced)
+  (label "CAN_TX" (at 127.635 133.985 0) (fields_autoplaced)
     (effects (font (size 1.27 1.27)) (justify left bottom))
   )

Commit message: add BOM
Parts:
- C32, C33: value 100nF 50V -> 100nF/100V; Link https://www.digikey.jp/en/products/detail/nextgen-component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 -> https://www.digikey.jp/en/products/detail/samsung-electro-m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; MPN 0603B104K500XD -> CL10B104KC8NNNC
- C34, C35: value 10nF 100V -> 10nF/100V; symbol BMS-Master-rescue:C-Device -> Device:C
- C36: value 1uF 25V -> 1uF/25V; symbol BMS-Master-rescue:C-Device -> Device:C
- C37: value 100nF 100V -> 100nF/100V; symbol BMS-Master-rescue:C-Device-BMS-Master-rescue -> Device:C
- J5, J6: Link https://www.digikey.jp/en/products/detail/samtec-inc/TSW-10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 -> https://www.digikey.jp/en/products/detail/amphenol-cs-comme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; MPN TSW-104-07-G-S -> G800W304018EU
- J7: Link (none) -> https://www.digikey.jp/en/products/detail/amphenol-cs-comme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; MPN (none) -> G800W306018EU
- R44, R45, R46, R47, R48: symbol Device:R -> Device:R_Small
