File: LTC6811_ESP32_V1.2/PowerMonitor.kicad_sch (KiCad schematic)
At the start: 51 parts, among them U2 AMC1301 or AMC1302, U3 AMC1301, U5 OPA2197IDR, U6 ISL28022

Commit message: Add files via upload
Parts:
- R17: footprint Resistor_SMD:R_2010_5025Metric -> Resistor_SMD:R_0603_1608Metric; Link https://www.digikey.jp/en/products/detail/yageo/RC2010JK-07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 -> https://www.digikey.jp/en/products/detail/vishay-dale/CRCW0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; MPN RC2010JK-071KL -> CRCW06031K00FKEA
- U2, U3: symbol ENNOID:AMC1301 -> Amplifier_Audio:AMC1301
Connections:
- net GND: no longer BAT-1.1 (Pin_1), R13.2, R17.1
- net Vbat renamed VBAT_SENSE
- new net BAT-: BAT-1.1 (Pin_1), R13.2, R17.1
Other:
- moved on the sheet: BAT-1

Commit message: Add files via upload
Parts:
- R11, R12, R14, R9: symbol BMS-Master-rescue:R-Device-BMS-Master-rescue -> Device:R_Small
Other:
- moved on the sheet: R11, R12, R14, R15, R18, R9, U5A

Commit message: add BOM
Parts:
- C10, C68: value 220pF 50V -> 220pF/50V; symbol BMS-Master-rescue:C-Device -> Device:C
- C11, C13, C14, C3, C52, C58, C72, C73: value 100nF 100V -> 100nF/100V; symbol BMS-Master-rescue:C-Device -> Device:C
- C12, C49: value 330pF 100V -> 330pF/100V; symbol BMS-Master-rescue:C-Device -> Device:C; Link https://search.murata.co.jp/Ceramy/image/img/A01X/G101/ENG/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 -> https://www.digikey.jp/en/products/detail/murata-electronic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
- C15, C62: value 2.2uF 16V -> 2.2uF/25V; symbol BMS-Master-rescue:C-Device -> Device:C; Link https://www.digikey.jp/en/products/detail/kemet/C0603C225K4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 -> https://www.digikey.jp/en/products/detail/murata-electronic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; MPN C0603C225K4PAC7867 -> GRM188R61E225KA12D
- C36: value 1uF 25V -> 1uF/25V; symbol BMS-Master-rescue:C-Device -> Device:C
- C65, C9: value 2.2nF 16V -> 2.2nF/16V; symbol BMS-Master-rescue:C-Device -> Device:C
- C67: value 100nF 100V -> 100nF/100V
- R15, R16, R17, R18, R19, R20, R21, R22, R23, R24, R25, R26, R27, R28, R29, R30, R31, R32, R33, R34, R35, R36: symbol Device:R -> Device:R_Small
- U5: footprint Housings_SOIC:SOIC-8_3.9x4.9mm_Pitch1.27mm -> PCM_4ms_Package_SOIC:SOIC-8_3.9x4.9mm_Pitch1.27mm; Link (none) -> https://www.digikey.jp/en/products/detail/texas-instruments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
- U6: symbol BMS-Master-rescue:INA226-Analog_ADC-BMS-Master-rescue -> Analog_ADC:‎ISL28022
Other:
- moved on the sheet: R35, R36
