File: LTC6811_ESP32_V1.2/PowerSupply.kicad_sch (KiCad schematic)
At the start: 20 parts, among them J1 +12V, J9 GND, U1 TPS76350, U4 SN6501DBV, U7 TPS563231

Commit message: Add files via upload
Parts:
- removed J1: +12V, Connector_PinHeader_2.54mm:PinHeader_1x01_P2.54mm_Vertical, symbol Connector_Generic:Conn_01x01
- removed J9: GND, Connector_PinHeader_2.54mm:PinHeader_1x01_P2.54mm_Vertical, symbol Connector_Generic:Conn_01x01
- added J15: PB MB, Connector_JST:JST_VH_B2P-VH-B_1x02_P3.96mm_Vertical, symbol Connector_Generic:Conn_01x02
- TR1: value TRANSF5 -> Converters
Connections:
- net +12V: now also J15.1 (Pin_1)
- net GND: now also J15.2 (Pin_2)
- net at C28.2, U7.4 (BST): no longer L1.1
- net at C28.1, U7.2 (SW): now also L1.1
- net at U4.1 (D1): now also TR1.3; no longer TR1.1
- net at U4.3 (D2): now also TR1.1; no longer TR1.3
- net at D5.2 (A): now also TR1.6; no longer TR1.4
- net at D4.2 (A): now also TR1.4; no longer TR1.6
Other:
- moved on the sheet: C1, C25, C28, D3, L1, R10, R41, R42

Commit message: Add files via upload
Parts:
- removed C1: 10uF 25V, Capacitor_SMD:C_0805_2012Metric, symbol Device:C
- removed C25: 47uF/10V, Capacitor_SMD:C_1206_3216Metric, symbol Device:C
- removed R41: 45.3K, Resistor_SMD:R_0603_1608Metric, symbol Device:R_Small
- removed R42: 10K, Resistor_SMD:R_0603_1608Metric, symbol Device:R_Small
- removed U7: TPS563231, Package_TO_SOT_SMD:SOT-563, symbol Regulator_Switching:TPS563231
- added C19 (x2): 10uF/16V, Capacitor_SMD:C_0805_2012Metric, symbol Device:C
- added C3: 2.2uF 50V, Capacitor_SMD:C_0603_1608Metric, symbol Device:C
- added D1: LED Red, LED_SMD:LED_0603_1608Metric, symbol Device:LED
- added R1: 470R, Resistor_SMD:R_0603_1608Metric, symbol Device:R_Small
- added R28: 22.1K, Resistor_SMD:R_0603_1608Metric, symbol Device:R_Small
- added R9: 100K, Resistor_SMD:R_0603_1608Metric, symbol Device:R_Small
- added U7: LM51420, Package_TO_SOT_SMD:SOT-23-6_Handsoldering, symbol Regulator_Switching:LMR51420
- R10: symbol BMS-Master-rescue:R-Device-BMS-Master-rescue -> Device:R_Small
Connections:
- net +12V: now also C3.1, U7.3 (VIN), U7.5 (EN)
- net +3V3: now also C19.1, C19.1, R1.2, R9.1
- net GND: now also C19.2, C19.2, C3.2, D1.1 (K), R28.2, U7.1 (GND)
- net at C28.1, L1.1: now also U7.2 (SW)
- net at C28.2: now also U7.6 (CB)
- new net: D1.2 (A), R1.1
- new net: R28.1, R9.2, U7.4 (FB)
Other:
- note added: "4.5 V to 36 V"
- note added: "I_{Max}=2A"
- note removed: "4.5 V to 17 V"
- note removed: "I_{Max}=3A"

Commit message: finished
Parts:
- added TP1, TP2: TestPoint, TestPoint:TestPoint_Pad_D1.0mm, symbol Connector:TestPoint
Connections:
- net +12V: now also J15.2 (Pin_2); no longer J15.1 (Pin_1)
- net +3V3: now also TP2.1
- net GND: now also J15.1 (Pin_1); no longer J15.2 (Pin_2)
- net ISO+5V: now also TP1.1
Other:
- moved on the sheet: J15
Changed lines of the file:
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@@
+    (stroke (width 0) (type default))
+  )
+  (wire (pts (xy 205.74 106.045) (xy 213.36 106.045))
     (stroke (width 0) (type default))
   )
@@
     (stroke (width 0) (type default))
   )
+  (wire (pts (xy 205.74 102.235) (xy 213.36 102.235))
+    (stroke (width 0) (type default))
+  )
   (wire (pts (xy 164.465 107.95) (xy 164.465 111.76))
     (stroke (width 0) (type default))
@@
   )
   (text "4.5 V to 36 V\n" (at 62.23 50.8 0)
+    (effects (font (size 1.27 1.27)) (justify left bottom))
+  )
+  (label "+3V3" (at 206.375 106.045 0) (fields_autoplaced)
+    (effects (font (size 1.27 1.27)) (justify left bottom))
+  )
+  (label "ISO+5V" (at 205.74 102.235 0) (fields_autoplaced)
     (effects (font (size 1.27 1.27)) (justify left bottom))
   )
@@
     )
   )
+  (symbol (lib_id "Connector:TestPoint") (at 213.36 106.045 270) (unit 1)
+    (in_bom yes) (on_board yes) (dnp no)
+    (property "Reference" "TP2" (at 217.932 108.585 0)
+      (effects (font (size 1.27 1.27)) (justify left) hide)
+    )
+    (property "Value" "TestPoint" (at 218.44 106.045 90)
+      (effects (font (size 1.27 1.27)) (justify left))
+    )
+    (property "Footprint" "TestPoint:TestPoint_Pad_D1.0mm" (at 213.36 111.125 0)
+      (effects (font (size 1.27 1.27)) hide)
+    )
+    (property "Datasheet" "~" (at 213.36 111.125 0)
+      (effects (font (size 1.27 1.27)) hide)
+    )
+    (pin "1")
+    (instances
+      (project "LTC6811_ESP32_V1.2"
+        (path "/6a86ff6f-b159-4c4c-8a40-e732cc82e010/00000000-0000-0000-0000-00005ac18063"
+          (reference "TP2") (unit 1)
+        )
+      )
+    )
+  )
   (symbol (lib_id "BMS-Master-rescue:+3.3V-power-BMS-Master-rescue") (at 137.16 64.135 0) (unit 1)
     (in_bom yes) (on_board yes) (dnp no)
@@
         (path "/6a86ff6f-b159-4c4c-8a40-e732cc82e010/00000000-0000-0000-0000-00005ac18063"
           (reference "#PWR022") (unit 1)
+        )
+      )
+    )
+  )
+  (symbol (lib_id "Connector:TestPoint") (at 213.36 102.235 270) (unit 1)
+    (in_bom yes) (on_board yes) (dnp no)
+    (property "Reference" "TP1" (at 217.932 104.775 0)
+      (effects (font (size 1.27 1.27)) (justify left) hide)
+    )
+    (property "Value" "TestPoint" (at 218.44 102.235 90)
+      (effects (font (size 1.27 1.27)) (justify left))
+    )
+    (property "Footprint" "TestPoint:TestPoint_Pad_D1.0mm" (at 213.36 107.315 0)
+      (effects (font (size 1.27 1.27)) hide)
+    )
+    (property "Datasheet" "~" (at 213.36 107.315 0)
+      (effects (font (size 1.27 1.27)) hide)
+    )
+    (pin "1")
+    (instances
+      (project "LTC6811_ESP32_V1.2"
+        (path "/6a86ff6f-b159-4c4c-8a40-e732cc82e010/00000000-0000-0000-0000-00005ac18063"
+          (reference "TP1") (unit 1)
         )
       )
@@
     )
   )
-  (symbol (lib_id "Connector_Generic:Conn_01x02") (at 51.435 59.055 0) (mirror y) (unit 1)
-    (in_bom yes) (on_board yes) (dnp no)
-    (property "Reference" "J15" (at 49.403 59.2582 0)
-      (effects (font (size 1.27 1.27)) (justify left))
-    )
-    (property "Value" "PB MB" (at 49.403 61.5696 0)
-      (effects (font (size 1.27 1.27)) (justify left))
-    )
-    (property "Footprint" "Connector_JST:JST_VH_B2P-VH-B_1x02_P3.96mm_Vertical" (at 51.435 59.055 0)
-      (effects (font (size 1.27 1.27)) hide)
-    )
-    (property "Datasheet" "https://tools.molex.com/pdm_docs/sd/705430001_sd.pdf" (at 51.435 59.055 0)
-      (effects (font (size 1.27 1.27)) hide)
-    )
-    (property "MPN" "70543-0001" (at 51.435 59.055 0)
-      (effects (font (size 1.27 1.27)) hide)
-    )
-    (property "Link" "https://www.digikey.jp/en/products/detail/molex/0705430001/114915?s=N4IgTCBcDaIOwAYCsAWAzAWgdgjCAugL5A" (at 51.435 59.055 0)
-      (effects (font (size 1.27 1.27)) hide)
-    )
-    (property "Description" "Connector Header Through Hole 2 position 0.100\" (2.54mm)" (at 51.435 59.055 0)
-      (effects (font (size 1.27 1.27)) hide)
-    )
+  (symbol (lib_id "Connector_Generic:Conn_01x02") (at 51.435 61.595 180) (unit 1)
+    (in_bom yes) (on_board yes) (dnp no)
+    (property "Reference" "J15" (at 49.403 61.3918 0)
+      (effects (font (size 1.27 1.27)) (justify left))
+    )
+    (property "Value" "PB MB" (at 49.403 59.0804 0)
+      (effects (font (size 1.27 1.27)) (justify left))
+    )
+    (property "Footprint" "Connector_JST:JST_VH_B2P-VH-B_1x02_P3.96mm_Vertical" (at 51.435 61.595 0)
+      (effects (font (size 1.27 1.27)) hide)
+    )
+    (property "Datasheet" "https://tools.molex.com/pdm_docs/sd/705430001_sd.pdf" (at 51.435 61.595 0)
+      (effects (font (size 1.27 1.27)) hide)
+    )
+    (property "MPN" "70543-0001" (at 51.435 61.595 0)
+      (effects (font (size 1.27 1.27)) hide)
+    )
+    (property "Link" "https://www.digikey.jp/en/products/detail/molex/0705430001/114915?s=N4IgTCBcDaIOwAYCsAWAzAWgdgjCAugL5A" (at 51.435 61.595 0)
+      (effects (font (size 1.27 1.27)) hide)
+    )
+    (property "Description" "Connector Header Through Hole 2 position 0.100\" (2.54mm)" (at 51.435 61.595 0)
+      (effects (font (size 1.27 1.27)) hide)
+    )

Commit message: add BOM
Parts:
- removed C1, C5: 10uF 25V, Capacitor_SMD:C_0805_2012Metric, symbol Device:C
- removed R9: 100K, Resistor_SMD:R_0603_1608Metric, symbol Device:R_Small
- added C19 (x2): 10uF/16V, Capacitor_SMD:C_0805_2012Metric, symbol Device:C
- added R65: 100K, Resistor_SMD:R_0603_1608Metric, symbol Device:R_Small
- C26: Link (none) -> https://www.digikey.jp/en/products/detail/samsung-electro-m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; 购买链接 https://www.digikey.jp/en/products/detail/samsung-electro-m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 -> (none)
- C28: value 100nF 100V -> 100nF/100V
- C3: value 100nF 100V -> 100nF/100V; symbol BMS-Master-rescue:C-Device -> Device:C
- C3: value 2.2uF 50V -> 2.2uF/25V; Link https://www.digikey.jp/en/products/detail/murata-electronics/GRT188R61H225KE13D/5416754?s=N4IgTCBcDaIOICUAqBGAHGhA2FAJMYArANICiKAzACIgC6AvkA -> https://www.digikey.jp/en/products/detail/murata-electronics/GRM188R61E225KA12D/4905349; MPN GRT188R61H225KE13D -> GRM188R61E225KA12D
- J15: Link https://www.digikey.jp/en/products/detail/molex/0705430001/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 -> https://www.digikey.jp/en/products/detail/jst-sales-america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; MPN 70543-0001 -> B2P-VH
- TR1: value Converters -> Transformer
- U1: symbol BMS-Master-rescue:TPS76350-Regulator_Linear -> Power_Supervisor:TPS76350
- U7: value LM51420 -> LMR51420XDDCR; Link (none) -> https://www.digikey.jp/en/products/detail/texas-instruments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
Connections:
- net +3V3: now also C19.1, R65.2
- net GND: now also C19.2
- net GND_PACK: now also C19.2
- net ISO+5V: now also C19.1
- net at R28.1, U7.4 (FB): now also R65.1
