File: LTC6811_ESP32_V1p2/_autosave-LTC6811_ESP32_V1p2.kicad_pcb (KiCad board)
At the start: 2 copper layers, 130 x 90 mm, 260 parts, among them J1 PB MB, J10 Hole /NC, J11 Hole /NC, J12 Hole /NC, J13 B7B-XH-A, J14 B7B-XH-A, J15 PB MB, J2 OLED /NC, J3 CAN /NC, J4 USB, J5 UART /NC, J6 JTAG /NC, J7 Boot Option /NC, J8 SERIAL /NC, J9 Hole /NC, Q1 BSS138, Q10 TSM2323, Q11 TSM2323, Q12 TSM2323, Q13 TSM2323, Q14 TSM2323, Q2 NSV1C201MZ4, Q3 TSM2323, Q4 TSM2323, Q5 TSM2323, Q6 TSM2323, Q7 TSM2323, Q8 TSM2323, Q9 TSM2323, U1 TPS76350, U10 CP2104, U11 ISO1050DUBR, U12 LTC6811HG-1, U2 AMC1301 or AMC1302, U3 AMC1301, U4 SN6501DBV, U5 OPA2197IDR, U6 ISL28022, U7 LMR51420XDDCR, U8 ESP32-DevKitC V4, U9 LTC6820

Commit message: fix thermal lilef
fix thermal lilef
Routing:
- net GND: track 88.6 -> 85.8 mm
- net /USB/D-: track 13.5 -> 15.1 mm
- net /USB/D+: track 18.2 -> 19.6 mm
- net /USB/Vusb: track 10.8 -> 11.7 mm, vias 0 -> 2
Changed lines of the file:
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@@
   (segment (start 118.775 112.5) (end 117.3 113.975) (width 0.6) (layer "F.Cu") (net 4))
   (segment (start 123.1 112.5) (end 118.775 112.5) (width 0.6) (layer "F.Cu") (net 4))
-  (segment (start 66.38845 114.9) (end 68.38845 112.9) (width 0.5) (layer "F.Cu") (net 4))
   (segment (start 103.6 109) (end 104.5 109) (width 0.3) (layer "F.Cu") (net 4))
   (segment (start 78.544999 121.990001) (end 78.26 122.275) (width 0.5) (layer "F.Cu") (net 4))
@@
   (via (at 85.1 124.5) (size 0.8) (drill 0.4) (layers "F.Cu" "B.Cu") (free) (net 4))
   (via (at 95.1 92.5) (size 0.8) (drill 0.4) (layers "F.Cu" "B.Cu") (free) (net 4))
-  (via (at 71.1 116.5) (size 0.8) (drill 0.4) (layers "F.Cu" "B.Cu") (free) (net 4))
+  (via (at 72.45 118.3) (size 0.8) (drill 0.4) (layers "F.Cu" "B.Cu") (free) (net 4))
   (via (at 123.1 100.5) (size 0.8) (drill 0.4) (layers "F.Cu" "B.Cu") (free) (net 4))
   (via (at 117.1 96.5) (size 0.8) (drill 0.4) (layers "F.Cu" "B.Cu") (free) (net 4))
@@
   (segment (start 160.22 77.94) (end 161.63 76.53) (width 0.3) (layer "F.Cu") (net 27))
   (segment (start 69.825 107.325) (end 68.8375 106.3375) (width 0.4) (layer "F.Cu") (net 28))
-  (segment (start 69.825 114.375) (end 69.825 107.75) (width 0.4) (layer "F.Cu") (net 28))
+  (segment (start 70.2 114.8) (end 68.69235 114.8) (width 0.4) (layer "F.Cu") (net 28))
   (segment (start 69.825 107.75) (end 69.825 107.325) (width 0.4) (layer "F.Cu") (net 28))
-  (segment (start 69.4 114.8) (end 69.825 114.375) (width 0.4) (layer "F.Cu") (net 28))
+  (segment (start 69.775 111.575) (end 70.2 112) (width 0.4) (layer "F.Cu") (net 28))
+  (segment (start 69.775 110.9) (end 69.775 111.575) (width 0.4) (layer "F.Cu") (net 28))
+  (segment (start 69.825 110.85) (end 69.775 110.9) (width 0.4) (layer "F.Cu") (net 28))
   (segment (start 68.8375 105.65) (end 68.8375 105.25) (width 0.4) (layer "F.Cu") (net 28))
   (segment (start 68.8375 106.3375) (end 68.8375 105.65) (width 0.4) (layer "F.Cu") (net 28))
-  (segment (start 68.69235 114.8) (end 69.4 114.8) (width 0.4) (layer "F.Cu") (net 28))
+  (segment (start 69.825 107.75) (end 69.825 110.85) (width 0.4) (layer "F.Cu") (net 28))
+  (via (at 70.2 112) (size 0.6) (drill 0.3) (layers "F.Cu" "B.Cu") (net 28))
+  (via (at 70.2 114.8) (size 0.6) (drill 0.3) (layers "F.Cu" "B.Cu") (net 28))
+  (segment (start 70.2 112) (end 70.2 114.8) (width 0.4) (layer "B.Cu") (net 28))
   (segment (start 156.9175 78.943553) (end 160.720659 78.943553) (width 0.3) (layer "F.Cu") (net 29))
   (segment (start 162.78 75.43) (end 164.3225 73.8875) (width 0.3) (layer "F.Cu") (net 29))
@@
   (segment (start 182.825 65.8) (end 180.975 65.8) (width 0.8) (layer "F.Cu") (net 79))
   (segment (start 180.975 64.8) (end 179.7 63.525) (width 0.8) (layer "F.Cu") (net 79))
+  (segment (start 71.05 115.5) (end 69.91005 115.5) (width 0.4) (layer "F.Cu") (net 80))
   (segment (start 66.5 109.7) (end 66.5 108.700002) (width 0.4) (layer "F.Cu") (net 80))
-  (segment (start 68.69235 115.450001) (end 69.84235 115.450001) (width 0.4) (layer "F.Cu") (net 80))
-  (segment (start 69.84235 115.450001) (end 70.64038 114.651971) (width 0.4) (layer "F.Cu") (net 80))
+  (segment (start 69.86005 115.45) (end 68.69235 115.450001) (width 0.4) (layer "F.Cu") (net 80))
   (segment (start 67.15 107.53) (end 66.5 108.18) (width 0.3) (layer "F.Cu") (net 80))
   (segment (start 66.5 108.7) (end 66.5 108.700002) (width 0.3) (layer "F.Cu") (net 80))
   (segment (start 67.15 106.3375) (end 67.15 107.53) (width 0.3) (layer "F.Cu") (net 80))
+  (segment (start 69.91005 115.5) (end 69.86005 115.45) (width 0.4) (layer "F.Cu") (net 80))
   (segment (start 66.5 108.18) (end 66.5 108.7) (width 0.3) (layer "F.Cu") (net 80))
-  (via (at 70.64038 114.651971) (size 0.6) (drill 0.3) (layers "F.Cu" "B.Cu") (net 80))
+  (segment (start 71.1 115.45) (end 71.05 115.5) (width 0.4) (layer "F.Cu") (net 80))
+  (via (at 71.1 115.45) (size 0.6) (drill 0.3) (layers "F.Cu" "B.Cu") (net 80))
   (via (at 66.5 109.7) (size 0.5) (drill 0.3) (layers "F.Cu" "B.Cu") (net 80))
-  (segment (start 70.64038 112.20962) (end 70.64038 114.651971) (width 0.4) (layer "B.Cu") (net 80))
-  (segment (start 68.1 109.7) (end 69.1 110.7) (width 0.4) (layer "B.Cu") (net 80))
+  (segment (start 71.1 111.91005) (end 71.1 115.45) (width 0.4) (layer "B.Cu") (net 80))
+  (segment (start 68.88995 109.7) (end 71.1 111.91005) (width 0.4) (layer "B.Cu") (net 80))
   (segment (start 66.5 109.7) (end 68.1 109.7) (width 0.4) (layer "B.Cu") (net 80))
-  (segment (start 69.1 110.7) (end 69.13076 110.7) (width 0.4) (layer "B.Cu") (net 80))
-  (segment (start 69.13076 110.7) (end 70.64038 112.20962) (width 0.4) (layer "B.Cu") (net 80))
+  (segment (start 68.1 109.7) (end 68.88995 109.7) (width 0.4) (layer "B.Cu") (net 80))
+  (segment (start 71.38995 116.15) (end 69.89235 116.15) (width 0.4) (layer "F.Cu") (net 81))
   (segment (start 65.07 107.7) (end 64.6 108.17) (width 0.3) (layer "F.Cu") (net 81))
   (segment (start 64.6 108.17) (end 64.6 108.7) (width 0.3) (layer "F.Cu") (net 81))
   (segment (start 64.6 108.72) (end 64.93 109.05) (width 0.4) (layer "F.Cu") (net 81))
   (segment (start 66.057106 107.7) (end 65.07 107.7) (width 0.3) (layer "F.Cu") (net 81))
-  (segment (start 68.69235 116.1) (end 70.2 116.1) (width 0.4) (layer "F.Cu") (net 81))
+  (segment (start 69.89235 116.15) (end 69.84235 116.1) (width 0.4) (layer "F.Cu") (net 81))
+  (segment (start 69.84235 116.1) (end 68.69235 116.1) (width 0.4) (layer "F.Cu") (net 81))
   (segment (start 64.93 109.05) (end 65.55 109.05) (width 0.4) (layer "F.Cu") (net 81))
   (segment (start 66.65 106.3375) (end 66.65 107.107106) (width 0.3) (layer "F.Cu") (net 81))
+  (segment (start 71.900003 115.45) (end 71.900003 115.639947) (width 0.4) (layer "F.Cu") (net 81))
+  (segment (start 71.900003 115.639947) (end 71.38995 116.15) (width 0.4) (layer "F.Cu") (net 81))
   (segment (start 66.65 107.107106) (end 66.057106 107.7) (width 0.3) (layer "F.Cu") (net 81))
-  (segment (start 70.2 116.1) (end 71.5 114.8) (width 0.4) (layer "F.Cu") (net 81))
+  (via (at 71.900003 115.45) (size 0.6) (drill 0.3) (layers "F.Cu" "B.Cu") (net 81))
   (via (at 65.55 109.05) (size 0.5) (drill 0.3) (layers "F.Cu" "B.Cu") (net 81))
-  (via (at 71.5 114.8) (size 0.6) (drill 0.3) (layers "F.Cu" "B.Cu") (net 81))
-  (segment (start 71.5 111.999988) (end 68.550012 109.05) (width 0.4) (layer "B.Cu") (net 81))
-  (segment (start 71.5 111.999988) (end 71.5 114.8) (width 0.4) (layer "B.Cu") (net 81))
+  (segment (start 69.088478 109.05) (end 71.900003 111.861525) (width 0.4) (layer "B.Cu") (net 81))
+  (segment (start 71.900003 111.861525) (end 71.900003 115.45) (width 0.4) (layer "B.Cu") (net 81))
   (segment (start 68.550012 109.05) (end 65.55 109.05) (width 0.4) (layer "B.Cu") (net 81))
+  (segment (start 68.550012 109.05) (end 69.088478 109.05) (width 0.4) (layer "B.Cu") (net 81))
   (segment (start 119.6525 88.765) (end 117.19 88.765) (width 0.5) (layer "F.Cu") (net 82))
   (segment (start 117.19 88.765) (end 117.125 88.7) (width 0.5) (layer "F.Cu") (net 82))
