File: LTC6811_ESP32_V1p2/LTC6811_ESP32_V1p2.kicad_pcb (KiCad board)
At the start: 2 copper layers, 130 x 90 mm, 260 parts, among them J1 PB MB, J10 Hole /NC, J11 Hole /NC, J12 Hole /NC, J13 B7B-XH-A, J14 B7B-XH-A, J15 PB MB, J2 OLED /NC, J3 CAN /NC, J4 USB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

Commit message: add ignore gerber
add ignore gerber
Routing:
- net GND: track 88.6 -> 85.8 mm
- net /USB/D-: track 13.5 -> 15.1 mm
- net /USB/D+: track 18.2 -> 19.6 mm
- net /USB/Vusb: track 10.8 -> 11.7 mm, vias 0 -> 2
