File: Master/ESP32_Master/ESP32_Master.kicad_pcb (KiCad board)
At the start: 2 copper layers, 150 x 90 mm, 122 parts, among them J1 PB MB, J10 Hole /NC, J11 Hole /NC, J12 Hole /NC, J2 OLED /NC, J3 PA MA, J4 USB, J5 UART /NC, J6 JTAG /NC, J7 Check_Votage, J8 Check_Votage, J9 Hole /NC, Q1 BSS138, U1 TPS76350, U10 CP2104, U2 AMC1301 or AMC1302, U3 AMC1301, U4 SN6501DBV, U5 OPA2197IDR, U6 ISL28022, U7 LMR51420XDDCR, U8 ESP32-DevKitC V4, U9 LTC6820

Commit message: Add files via upload
Parts:
- removed BAT-1: BAT-, Battery:Battery_6mm×10mm_Cell_half_2
- removed BZ1: AI-1027-TWT-5V, Buzzer_Beeper:Beeper_AI-1027-TWT-5V
- removed C38, C41: 2.2uF/25V, Capacitor_SMD:C_0603_1608Metric
- removed C39: 4.7uF/16V, Capacitor_SMD:C_0603_1608Metric
- removed C40: 100nF/100V, Capacitor_SMD:C_0603_1608Metric
- removed CURRENT-1: CURRENT-, Battery:Battery_6mm×10mm_Cell_half_2
- removed D2: LED Red, LED_SMD:LED_0603_1608Metric
- removed D7: ESD24VS2U, Package_TO_SOT_SMD:SOT-23
- removed J2: OLED /NC, Connector_PinHeader_2.54mm:PinHeader_1x05_P2.54mm_Vertical
- removed J5: UART /NC, Connector_PinHeader_2.54mm:PinHeader_1x04_P2.54mm_Vertical
- removed Q1: BSS138, Package_TO_SOT_SMD:SOT-23
- removed R2: 470R, Resistor_SMD:R_0603_1608Metric
- removed R49, R50: 0, Resistor_SMD:R_0603_1608Metric
- removed R5: 1.5K, Resistor_SMD:R_0603_1608Metric
- removed R51, R52: 10K, Resistor_SMD:R_0603_1608Metric
- removed R7, R8: 4.7K, Resistor_SMD:R_0603_1608Metric
- removed U10: CP2104, Package_DFN_QFN:HVQFN-24-1EP_4x4mm_P0.5mm_EP2.6x2.6mm
- added C30: 100nF/100V, Capacitor_SMD:C_0603_1608Metric, F.Cu at (62.3, 164.7)
- added C31: 100nF/100V, Capacitor_SMD:C_0603_1608Metric, F.Cu at (62.3, 167.2)
- added J13: Conn_01x02_Socket, Connector_PinSocket_2.54mm:PinSocket_1x02_P2.54mm_Vertical, F.Cu at (139.5, 130.4)
- added R3: 0, Resistor_SMD:R_0603_1608Metric, F.Cu at (137.2, 173.9)
- added R4: 0, Resistor_SMD:R_0603_1608Metric, F.Cu at (137.2, 176.4)
- added U12: MCP2562-E-SN, Package_SO:SOIC-8_3.9x4.9mm_P1.27mm, F.Cu at (128.8, 176.0)
- J4: value USB -> Conn_01x03_Pin; footprint Connector_USB:Micro_USB_B-2013499-1 -> Connector_PinHeader_2.54mm:PinHeader_1x03_P2.54mm_Vertical
- R13: footprint Resistor_SMD:R_PSR500HTQFB0L10_Metric_Pad5.2x8.75mm_HandSolder -> Resistor_SMD:R_PSR500HTQFB0L10_Metric_Pad5.2x8.75mm_Hole
- R6: value 4.7K -> 120R
- moved J4 91.1 mm to (155.6, 135.9)
- moved J7 76.0 mm to (143.5, 175.6)
- moved J8 74.4 mm to (153.6, 167.1)
- moved R12 74.1 mm to (96.9, 141.5)
- moved R11 74.1 mm to (100.5, 141.5)
- moved R14 74.1 mm to (93.4, 141.5)
- moved R9 74.1 mm to (104.1, 141.5)
- moved R15 71.0 mm to (93.4, 139.2), turned to 0 degrees
- moved R19 67.0 mm to (92.6, 136.3), turned to 90 degrees
- moved R18 66.8 mm to (94.2, 136.3), turned to -90 degrees
- moved C6 64.1 mm to (90.3, 133.9), turned to 180 degrees
- moved C7 63.6 mm to (93.4, 133.9), turned to 0 degrees
- moved C13 61.3 mm to (64.0, 172.5)
- moved C27 61.3 mm to (55.4, 172.5)
- moved TR1 61.3 mm to (71.1, 171.5)
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Connections:
- net /PowerMonitor/CURRENT renamed /PowerMonitor/INN
- J4 pad 1: /USB/Vusb -> unconnected-(J4-Pin_1-Pad1)
- J4 pad 2: /USB/D- -> Net-(J4-Pin_2)
- J4 pad 3: /USB/D+ -> Net-(J13-Pin_2)
- J8 pad 1: GNDA -> /GNDA
- R13 pad 1: GNDA -> /GNDA
- R16 pad 1: GNDA -> /GNDA
- R6 pad 1: /MCU/OLED_RST -> Net-(J13-Pin_1)
- R6 pad 2: +3V3 -> Net-(J4-Pin_2)
- U8 pad 10: /MCU/LED0 -> unconnected-(U8-IO26-Pad10)
- U8 pad 19: /MCU/5V -> +5V
- U8 pad 20: /MCU/OLED_RST -> unconnected-(U8-CLK-Pad20)
- U8 pad 21: /MCU/OLED_SDA -> unconnected-(U8-SD0-Pad21)
- U8 pad 22: /MCU/OLED_SCL -> unconnected-(U8-SD1-Pad22)
- U8 pad 34: /MCU/RX_USB -> unconnected-(U8-RXD0-Pad34)
- U8 pad 35: /MCU/TX_USB -> unconnected-(U8-TXD0-Pad35)
- U8 pad 5: unconnected-(U8-IO34-Pad5) -> /MCU/CAN_RX
- U8 pad 7: unconnected-(U8-IO32-Pad7) -> /MCU/CAN_TX
- U8 pad 9: /MCU/BUZZER -> unconnected-(U8-IO25-Pad9)
Routing:
- net /PowerMonitor/INN: track 0.00 -> 11.9 mm
- net /GNDA: track 0.00 -> 11.7 mm
- net Net-(U2-VINP): track 0.00 -> 4.50 mm
- net Net-(U2-VINN): track 0.00 -> 4.50 mm
Other:
- board size 150 x 90 mm -> 99.9 x 90 mm

Commit message: Add files via upload
Parts:
- removed R3, R4: 0, Resistor_SMD:R_0603_1608Metric
- moved U12 120.3 mm to (55.1, 80.9), turned to 180 degrees
- moved J4 111.4 mm to (52.8, 93.1), turned to 90 degrees
- moved J3 103.2 mm to (95.8, 145.6), turned to 180 degrees
- moved J13 95.5 mm to (53.2, 89.4), turned to 90 degrees
- moved R37 90.6 mm to (95.9, 61.1), turned to 180 degrees
- moved R38 88.2 mm to (95.9, 62.9), turned to 180 degrees
- moved C30 87.9 mm to (53.4, 77.3), turned to 180 degrees
- moved C31 86.2 mm to (59.7, 81.1), turned to 90 degrees
- moved TR2 83.8 mm to (93.8, 129.1), turned to 180 degrees
- moved C28 83.2 mm to (93.0, 66.2), turned to 90 degrees
- moved U7 82.7 mm to (95.7, 66.8), turned to 90 degrees
- moved C3 82.4 mm to (98.5, 67.3), turned to 90 degrees
- moved J9 81.9 mm to (114.1, 65.4)
- moved R1 78.0 mm to (87.7, 50.0)
- moved TP2 78.0 mm to (91.9, 48.9)
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Connections:
- net Net-(U6-Vin+) renamed /PowerMonitor/Vin+
- net Net-(U6-Vin-) renamed /PowerMonitor/Vin-
- C1 pad 2: GNDREF -> GNDA
- C2 pad 2: GNDREF -> GNDA
- C26 pad 2: GNDREF -> GNDA
- D3 pad 1: GNDREF -> GNDA
- TR1 pad 5: GNDREF -> GNDA
- U1 pad 2: GNDREF -> GNDA
- U8 pad 5: /MCU/CAN_RX -> /CAN/CAN_RX
- U8 pad 7: /MCU/CAN_TX -> /CAN/CAN_TX
Routing:
- net /PowerMonitor/ISO+5V: track 0.00 -> 76.2 mm
- net /MCU/MOSI: track 0.00 -> 49.9 mm
- net /MCU/MISO: track 0.00 -> 29.2 mm
- net /MCU/SCK: track 0.00 -> 23.3 mm
- net /MCU/SCL: track 0.00 -> 21.3 mm
- net /MCU/IM: track 0.00 -> 18.5 mm
- net /MCU/IP: track 0.00 -> 18.4 mm
- net /MCU/SS: track 0.00 -> 18.2 mm
- net /MCU/SDA: track 0.00 -> 14.7 mm
- net GNDA: track 0.00 -> 14.7 mm
- net Net-(D4-K): track 0.00 -> 12.5 mm, vias 0 -> 2
- net +3V3: track 0.00 -> 11.0 mm
- net /PA: track 0.00 -> 8.94 mm
- net /MA: track 0.00 -> 8.90 mm
- net /PowerMonitor/Vin+: track 0.00 -> 6.79 mm
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Other:
- board text added: "PACK+"

Commit message: Add files via upload
Parts:
- removed J13: Conn_01x02_Socket, Connector_PinSocket_2.54mm:PinSocket_1x02_P2.54mm_Vertical
- removed J4: Conn_01x03_Pin, Connector_PinHeader_2.54mm:PinHeader_1x03_P2.54mm_Vertical
- removed R6: 120R, Resistor_SMD:R_0603_1608Metric
- removed U12: MCP2562-E-SN, Package_SO:SOIC-8_3.9x4.9mm_P1.27mm
- added C22: 1uF/25V, Capacitor_SMD:C_0603_1608Metric, F.Cu at (94.5, 82.9)
- added C29: 100nF/100V, Capacitor_SMD:C_0603_1608Metric, F.Cu at (94.5, 81.2)
- added D2: ESD24VS2U, Package_TO_SOT_SMD:SOT-23, F.Cu at (99.1, 65.9)
- added J2: CAN, Connector_PinHeader_2.54mm:PinHeader_1x04_P2.54mm_Vertical, F.Cu at (102.9, 62.0)
- added U10: ISO1050DUBR, Package_SO:SOP-8_6.62x9.15mm_P2.54mm, F.Cu at (99.1, 74.2)
- C30: value 100nF/100V -> 1uF/25V
- TP1: value TestPoint -> IOS+5V
- TP2: value TestPoint -> +3V3
- moved LOGO1 106.7 mm to (77.0, 119.8)
- moved J1 85.2 mm to (54.6, 135.0), turned to 90 degrees
- moved R37 83.0 mm to (64.4, 138.0), turned to 0 degrees
- moved R38 79.9 mm to (64.4, 136.3), turned to 0 degrees
- moved C3 74.2 mm to (61.7, 131.8), turned to -90 degrees
- moved TP2 73.7 mm to (64.4, 117.3), turned to 180 degrees
- moved U7 72.6 mm to (64.6, 132.4), turned to -90 degrees
- moved C28 71.6 mm to (67.2, 133.0), turned to -90 degrees
- moved R1 70.4 mm to (67.2, 117.3), turned to 180 degrees
- moved D1 66.5 mm to (70.3, 117.3), turned to 180 degrees
- moved L1 61.3 mm to (64.4, 126.2), turned to 90 degrees
- moved C24 52.2 mm to (65.3, 121.5), turned to 0 degrees
- moved C10 48.8 mm to (65.3, 119.4), turned to 0 degrees
- moved C30 43.0 mm to (94.5, 64.8)
- moved C31 37.8 mm to (94.5, 66.4), turned to 0 degrees
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Connections:
- C30 pad 1: GND -> /CAN/5V_CAN
- C30 pad 2: +3V3 -> /CAN/CAN_GND
- C31 pad 1: GND -> /CAN/CAN_GND
- C31 pad 2: +5V -> /CAN/5V_CAN
- J1 pad 1: +12V -> GND
- J1 pad 2: GND -> +12V
- J8 pad 1: /GNDA -> GNDA
- R13 pad 1: /GNDA -> GNDA
- R16 pad 1: /GNDA -> GNDA
- U8 pad 34: unconnected-(U8-RXD0-Pad34) -> /CAN/CAN_RX
- U8 pad 35: unconnected-(U8-TXD0-Pad35) -> /CAN/CAN_TX
- U8 pad 5: /CAN/CAN_RX -> unconnected-(U8-IO34-Pad5)
- U8 pad 7: /CAN/CAN_TX -> unconnected-(U8-IO32-Pad7)
Routing:
- net +3V3: track 11.0 -> 235.9 mm, vias 0 -> 6
- net +12V: track 0.00 -> 100.5 mm, vias 0 -> 2
- net +5V: track 0.00 -> 35.1 mm
- net /PowerMonitor/VBAT_SENSE: track 2.18 -> 33.5 mm
- net /MCU/MTDO: track 0.00 -> 29.9 mm, vias 0 -> 1
- net /CAN/CAN_TX: track 0.00 -> 16.0 mm
- net /CAN/CAN_RX: track 0.00 -> 13.3 mm
- net /MCU/MOSI: track 49.9 -> 37.2 mm
- net GNDA: track 14.7 -> 26.4 mm
- net /GNDA: track 11.7 -> 0.00 mm
- net /CAN/CANH: track 0.00 -> 8.25 mm
- net /CAN/CAN_GND: track 0.00 -> 7.85 mm
- net /CAN/5V_CAN: track 0.00 -> 7.85 mm
- net /CAN/CANL: track 0.00 -> 7.68 mm
- net Net-(U9-ICMP): track 0.00 -> 7.14 mm
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- added copper zone on B.Cu, net /CAN/CAN_GND
- added copper zone on F.Cu, net /CAN/CAN_GND
- added copper zone on B.Cu, net /PowerMonitor/INN
- added copper zone on F.Cu, net /PowerMonitor/INN
- added copper zone on B.Cu, net GND
- added copper zone on F.Cu, net GND
- added copper zone on B.Cu, net GNDA
- added copper zone on F.Cu, net GNDA
Other:
- board text added: "2024/06/07"
- board text added: "5V CANL CANH GND"
- board text removed: "+3.3V"
- board text removed: "+3V3"
- board text removed: "2024/06/03"
- board text removed: "3V3"
- board text removed: "RST"
- board text removed: "RX"
- board text removed: "SCL"
- board text removed: "SDA"
- board text removed: "TX"
- board text removed: "UART"

Commit message: Add files via upload
Parts:
- C1, C10, C13, C24, C27: footprint Capacitor_SMD:C_0805_2012Metric -> C_0805_2012Metric
- C11, C12, C14, C15, C16, C17, C18, C19, C2, C20, C21, C22, C23, C25, C26, C28, C29, C3, C30, C31, C32, C33, C34, C35, C36, C37, C4, C5, C6, C7, C71, C8, C9: footprint Capacitor_SMD:C_0603_1608Metric -> C_0603_1608Metric
- D1, D3: footprint LED_SMD:LED_0603_1608Metric -> LED_0603_1608Metric
- D2: footprint Package_TO_SOT_SMD:SOT-23 -> SOT-23
- D4, D5: footprint Diode_SMD:D_SOD-123 -> D_SOD-123
- J1, J3, J7, J8: footprint Connector_JST:JST_VH_B2P-VH-B_1x02_P3.96mm_Vertical -> JST_VH_B2P-VH-B_1x02_P3.96mm_Vertical
- J10, J11, J12, J9: footprint MountingHole:MountingHole_3.2mm_M3_ISO7380_Pad -> MountingHole_3.2mm_M3_ISO7380_Pad
- J2, J6: footprint Connector_PinHeader_2.54mm:PinHeader_1x04_P2.54mm_Vertical -> PinHeader_1x04_P2.54mm_Vertical
- L1: footprint Inductor_SMD:L_Bourns_SRP5030T -> L_Bourns_SRP5030T
- LOGO1: footprint Symbol:teTra-LOGO -> teTra-LOGO
- R1, R10, R16, R17, R18, R19, R20, R21, R22, R23, R24, R25, R26, R27, R28, R29, R30, R31, R32, R33, R34, R35, R36, R37, R38, R43, R44, R45, R46, R47, R48: footprint Resistor_SMD:R_0603_1608Metric -> R_0603_1608Metric
- R11, R12, R14, R15, R9: footprint Resistor_SMD:R_0805_2012Metric -> R_0805_2012Metric
- R13: footprint Resistor_SMD:R_PSR500HTQFB0L10_Metric_Pad5.2x8.75mm_Hole -> R_PSR500HTQFB0L10_Metric_Pad5.2x8.75mm_Hole
- TP1, TP2: footprint TestPoint:TestPoint_Pad_D1.0mm -> TestPoint_Pad_D1.0mm
- TR1: footprint Connector_Wuerth:WURTH-760390015 -> WURTH-760390015
- TR2: footprint Transformer_SMD:HM2108NL -> HM2108NL
- U1, U4: footprint Package_TO_SOT_SMD:SOT-23-5 -> SOT-23-5
- U10: footprint Package_SO:SOP-8_6.62x9.15mm_P2.54mm -> SOP-8_6.62x9.15mm_P2.54mm
- U2, U3: footprint Package_SO:SSO-8_6.8x5.9mm_P1.27mm_Clearance8mm -> SSO-8_6.8x5.9mm_P1.27mm_Clearance8mm
- U5: footprint Package_SO:SOIC-8_3.9x4.9mm_P1.27mm -> SOIC-8_3.9x4.9mm_P1.27mm
- U6: footprint Package_SO:MSOP-10_3x3mm_P0.5mm -> MSOP-10_3x3mm_P0.5mm
- U7: footprint Package_TO_SOT_SMD:SOT-23-6_Handsoldering -> SOT-23-6_Handsoldering
- U8: footprint RF_Module:ESP32-DevKitc V4_DIP-38_27.9mm×48.2mm -> ESP32-DevKitc V4_DIP-38_27.9mm×48.2mm
- U9: footprint Package_SO:MSOP-16_3x4mm_P0.5mm -> MSOP-16_3x4mm_P0.5mm
- moved J11 0.18 mm to (55.1, 65.0), turned to 180 degrees
Routing:
- net +5V: track 35.1 -> 0.00 mm
- net unconnected-(U8-IO32-Pad7): track 2.72 -> 0.00 mm
- net unconnected-(U8-IO34-Pad5): track 2.65 -> 0.00 mm
- net /CAN/CAN_GND: track 7.85 -> 7.68 mm, vias 0 -> 28
- net GNDA: vias 0 -> 88
- net GND: vias 0 -> 174
- net /PowerMonitor/INN: vias 0 -> 18
Other:
- board text removed: "ISO+5V"

Commit message: Add files via upload
Parts:
- moved TR2 0.15 mm to (94.0, 129.1)
- moved U3 0.10 mm to (113.1, 129.1)
- turned C33 to 0 degrees
Routing:
- net GND: track 2.20 -> 25.4 mm, vias 174 -> 220
- net /MCU/NRST: track 7.08 -> 8.17 mm
- net GNDA: vias 88 -> 90

Commit message: Add files via upload
Parts:
- C1, C10, C13, C24, C27: footprint C_0805_2012Metric -> Capacitor_SMD:C_0805_2012Metric
- C11, C12, C14, C15, C16, C17, C18, C19, C2, C20, C21, C22, C23, C25, C26, C28, C29, C3, C30, C31, C32, C33, C34, C35, C36, C37, C4, C5, C6, C7, C71, C8, C9: footprint C_0603_1608Metric -> Capacitor_SMD:C_0603_1608Metric
- D1, D3: footprint LED_0603_1608Metric -> LED_SMD:LED_0603_1608Metric
- D2: footprint SOT-23 -> Package_TO_SOT_SMD:SOT-23
- D4, D5: footprint D_SOD-123 -> Diode_SMD:D_SOD-123
- J1, J3, J7, J8: footprint JST_VH_B2P-VH-B_1x02_P3.96mm_Vertical -> Connector_JST:JST_VH_B2P-VH-B_1x02_P3.96mm_Vertical
- J10, J11, J12, J9: footprint MountingHole_3.2mm_M3_ISO7380_Pad -> MountingHole:MountingHole_3.2mm_M3_ISO7380_Pad
- J2, J6: footprint PinHeader_1x04_P2.54mm_Vertical -> Connector_PinHeader_2.54mm:PinHeader_1x04_P2.54mm_Vertical
- L1: footprint L_Bourns_SRP5030T -> Inductor_SMD:L_Bourns_SRP5030T
- LOGO1: footprint teTra-LOGO -> Symbol:teTra-LOGO
- R1, R10, R16, R17, R18, R19, R20, R21, R22, R23, R24, R25, R26, R27, R28, R29, R30, R31, R32, R33, R34, R35, R36, R37, R38, R43, R44, R45, R46, R47, R48: footprint R_0603_1608Metric -> Resistor_SMD:R_0603_1608Metric
- R11, R12, R14, R15, R9: footprint R_0805_2012Metric -> Resistor_SMD:R_0805_2012Metric
- R13: footprint R_PSR500HTQFB0L10_Metric_Pad5.2x8.75mm_Hole -> Resistor_SMD:R_PSR500HTQFB0L10_Metric_Pad5.2x8.75mm_Hole
- TP1, TP2: footprint TestPoint_Pad_D1.0mm -> TestPoint:TestPoint_Pad_D1.0mm
- TR1: footprint WURTH-760390015 -> Connector_Wuerth:WURTH-760390015
- TR2: footprint HM2108NL -> Transformer_SMD:HM2108NL
- U1, U4: footprint SOT-23-5 -> Package_TO_SOT_SMD:SOT-23-5
- U10: footprint SOP-8_6.62x9.15mm_P2.54mm -> Package_SO:SOP-8_6.62x9.15mm_P2.54mm
- U2, U3: footprint SSO-8_6.8x5.9mm_P1.27mm_Clearance8mm -> Package_SO:SSO-8_6.8x5.9mm_P1.27mm_Clearance8mm
- U5: footprint SOIC-8_3.9x4.9mm_P1.27mm -> Package_SO:SOIC-8_3.9x4.9mm_P1.27mm
- U6: footprint MSOP-10_3x3mm_P0.5mm -> Package_SO:MSOP-10_3x3mm_P0.5mm
- U7: footprint SOT-23-6_Handsoldering -> Package_TO_SOT_SMD:SOT-23-6_Handsoldering
- U8: footprint ESP32-DevKitc V4_DIP-38_27.9mm×48.2mm -> RF_Module:ESP32-DevKitc V4_DIP-38_27.9mm×48.2mm
- U9: footprint MSOP-16_3x4mm_P0.5mm -> Package_SO:MSOP-16_3x4mm_P0.5mm
- moved J11 0.07 mm to (55.1, 65.1)
- turned C33 to 90 degrees
Routing:
- net GND: track 25.4 -> 2.20 mm, vias 220 -> 174
- net /MCU/NRST: track 8.17 -> 7.08 mm
- net /CAN/CAN_GND: track 7.68 -> 7.85 mm, vias 28 -> 0
- net GNDA: vias 90 -> 88
Other:
- board text added: "2024/06/10"
- board text removed: "2024/06/07"
