File: Master/ESP32_Master/ESP32_Master.kicad_sch (KiCad schematic)
At the start: 20 parts, among them J10 Hole /NC, J11 Hole /NC, J12 Hole /NC, J2 OLED /NC, J3 PA MA, J4 USB, J7 Check_Votage, J8 Check_Votage, J9 Hole /NC, Q1 BSS138

Commit message: Add files via upload
Parts:
- removed BAT-1: BAT-, Battery:Battery_6mm×10mm_Cell_half_2, symbol Connector_Generic:Conn_01x01
- removed BZ1: AI-1027-TWT-5V, Buzzer_Beeper:Beeper_AI-1027-TWT-5V, symbol Device:Buzzer
- removed CURRENT-1: CURRENT-, Battery:Battery_6mm×10mm_Cell_half_2, symbol Connector_Generic:Conn_01x01
- removed D2: LED Red, LED_SMD:LED_0603_1608Metric, symbol Device:LED
- removed J2: OLED /NC, Connector_PinHeader_2.54mm:PinHeader_1x05_P2.54mm_Vertical, symbol Connector_Generic:Conn_01x05
- removed J4: USB, Connector_USB:Micro_USB_B-2013499-1, symbol Connector:USB_B_Micro
- removed Q1: BSS138, Package_TO_SOT_SMD:SOT-23, symbol Transistor_FET:BSS138
- removed R2: 470R, Resistor_SMD:R_0603_1608Metric, symbol Device:R_Small
- removed R5: 1.5K, Resistor_SMD:R_0603_1608Metric, symbol Device:R_Small
- removed R6, R7, R8: 4.7K, Resistor_SMD:R_0603_1608Metric, symbol Device:R_Small
- added R3, R4: 0, Resistor_SMD:R_0603_1608Metric, symbol Device:R_Small
Connections:
- net GNDA: no longer J8.1 (Pin_1)
- new net CAN/CAN_RX: R3.2
- new net CAN/CAN_TX: R4.2
- new net MCU/CAN_RX: R3.1
- new net MCU/CAN_TX: R4.1
- new net PowerMonitor/INP: J8.1 (Pin_1)
- no-connect marks 5 -> 4
Other:
- removed sheet USB
- added sheet CAN (CAN.kicad_sch)
- sheet MCU ports: added CAN_RX, CAN_TX; removed BUZZER, LED0, OLED_RST, OLED_SCL, OLED_SDA, RX_USB, TX_USB
- sheet PowerMonitor ports: added INP; removed BAT-, CURRENT
- moved on the sheet: J10, J11, J12, J3, J9

Commit message: Add files via upload
Parts:
- removed R3, R4: 0, Resistor_SMD:R_0603_1608Metric, symbol Device:R_Small

Commit message: Add files via upload
Parts:
- added J2: CAN, Connector_PinHeader_2.54mm:PinHeader_1x04_P2.54mm_Vertical, symbol Connector:Conn_01x04_Pin
Connections:
- new net CAN/5V_CAN: J2.4 (Pin_4)
- new net CAN/CANH: J2.2 (Pin_2)
- new net CAN/CANL: J2.3 (Pin_3)
- new net CAN/CAN_GND: J2.1 (Pin_1)
Other:
- sheet CAN ports: added 5V_CAN, CANH, CANL, CAN_GND; removed none
Changed lines of the file:
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@@
+    (stroke (width 0) (type default))
+  )
+  (wire (pts (xy 259.08 109.22) (xy 266.7 109.22))
     (stroke (width 0) (type default))
   )
@@
     (stroke (width 0) (type default))
   )
+  (wire (pts (xy 259.08 104.14) (xy 266.7 104.14))
+    (stroke (width 0) (type default))
+  )
+  (wire (pts (xy 259.08 111.76) (xy 266.7 111.76))
+    (stroke (width 0) (type default))
+  )
   (wire (pts (xy 227.965 109.22) (xy 240.665 109.22))
     (stroke (width 0) (type default))
   )
   (wire (pts (xy 112.395 106.045) (xy 120.65 106.045))
+    (stroke (width 0) (type default))
+  )
+  (wire (pts (xy 259.08 106.68) (xy 266.7 106.68))
     (stroke (width 0) (type default))
   )
@@
         (path "/6a86ff6f-b159-4c4c-8a40-e732cc82e010"
           (reference "J3") (unit 1)
+        )
+      )
+    )
+  )
+  (symbol (lib_id "Connector:Conn_01x04_Pin") (at 271.78 106.68 0) (mirror y) (unit 1)
+    (in_bom yes) (on_board yes) (dnp no)
+    (property "Reference" "J2" (at 273.05 106.68 0)
+      (effects (font (size 1.27 1.27)) (justify right))
+    )
+    (property "Value" "CAN" (at 266.7 114.3 0)
+      (effects (font (size 1.27 1.27)) (justify right))
+    )
+    (property "Footprint" "Connector_PinHeader_2.54mm:PinHeader_1x04_P2.54mm_Vertical" (at 271.78 106.68 0)
+      (effects (font (size 1.27 1.27)) hide)
+    )
+    (property "Datasheet" "~" (at 271.78 106.68 0)
+      (effects (font (size 1.27 1.27)) hide)
+    )
+    (pin "1")
+    (pin "4")
+    (pin "2")
+    (pin "3")
+    (instances
+      (project "ESP32_Master"
+        (path "/6a86ff6f-b159-4c4c-8a40-e732cc82e010"
+          (reference "J2") (unit 1)
+        )
+      )
+    )
+  )
+  (symbol (lib_id "power:GNDA") (at 106.299 136.652 0) (unit 1)
+    (in_bom yes) (on_board yes) (dnp no)
+    (property "Reference" "#PWR09" (at 106.299 143.002 0)
+      (effects (font (size 1.27 1.27)) hide)
+    )
+    (property "Value" "GNDA" (at 106.299 140.462 0)
+      (effects (font (size 1.27 1.27)))
+    )
+    (property "Footprint" "" (at 106.299 136.652 0)
+      (effects (font (size 1.27 1.27)) hide)
+    )
+    (property "Datasheet" "" (at 106.299 136.652 0)
+      (effects (font (size 1.27 1.27)) hide)
+    )
+    (pin "1")
+    (instances
+      (project "ESP32_Master"
+        (path "/6a86ff6f-b159-4c4c-8a40-e732cc82e010"
+          (reference "#PWR09") (unit 1)
         )
       )
@@
       (effects (font (size 1.27 1.27)) (justify left top))
     )
+    (pin "5V_CAN" input (at 259.08 111.76 0)
+      (effects (font (size 1.27 1.27)) (justify right))
+    )
+    (pin "CANL" input (at 259.08 109.22 0)
+      (effects (font (size 1.27 1.27)) (justify right))
+    )
+    (pin "CANH" input (at 259.08 106.68 0)
+      (effects (font (size 1.27 1.27)) (justify right))
+    )
+    (pin "CAN_GND" input (at 259.08 104.14 0)
+      (effects (font (size 1.27 1.27)) (justify right))
+    )
+    (pin "CAN_TX" input (at 240.665 109.22 180)
+      (effects (font (size 1.27 1.27)) (justify left))
+    )
     (pin "CAN_RX" output (at 240.665 106.68 180)
       (effects (font (size 1.27 1.27)) (justify left))
     )
-    (pin "CAN_TX" input (at 240.665 109.22 180)
-      (effects (font (size 1.27 1.27)) (justify left))
-    )
