File: Master/ESP32_Master/MCU.kicad_sch (KiCad schematic)
At the start: 17 parts, among them J5 UART /NC, J6 JTAG /NC, U8 ESP32-DevKitC V4, U9 LTC6820

Commit message: Add files via upload
Parts:
- removed J5: UART /NC, Connector_PinHeader_2.54mm:PinHeader_1x04_P2.54mm_Vertical, symbol Connector_Generic:Conn_01x04
Connections:
- net CAN_RX: now reaches U8.5 (IO34)
- net CAN_TX: now reaches U8.7 (IO32)
- net 5V renamed +5V
- net BUZZER: no longer names the net of U8.9 (IO25)
- net LED0: no longer names the net of U8.10 (IO26)
- net OLED_RST: no longer names the net of U8.20 (CLK)
- net OLED_SCL: no longer names the net of U8.22 (SD1)
- net OLED_SDA: no longer names the net of U8.21 (SD0)
- net RX_USB: no longer names the net of U8.34 (RXD0)
- net TX_USB: no longer names the net of U8.35 (TXD0)
- no-connect marks 10 -> 16
Other:
- note removed: "UART DOWNLOAD"
- moved on the sheet: C32, C33, R43

Commit message: Add files via upload
Connections:
- net CAN_RX: now also U8.34 (RXD0); no longer U8.5 (IO34)
- net CAN_TX: now also U8.35 (TXD0); no longer U8.7 (IO32)
- no-connect marks 16 -> 17
Other:
- moved on the sheet: C32, C33, C34, C35, C36, C37, J6, R43, R44, R45, R46, R47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
