File: Master/ESP32_Master/PowerMonitor.kicad_sch (KiCad schematic)
At the start: 49 parts, among them U2 AMC1301 or AMC1302, U3 AMC1301, U5 OPA2197IDR, U6 ISL28022

Commit message: Add files via upload
Parts:
- R13: footprint Resistor_SMD:R_PSR500HTQFB0L10_Metric_Pad5.2x8.75mm_HandSolder -> Resistor_SMD:R_PSR500HTQFB0L10_Metric_Pad5.2x8.75mm_Hole
Connections:
- net Vin+: now reaches C19.2, R30.1, R32.1, U6.10 (Vin+)
- net Vin-: now reaches C20.2, R31.1, R32.2, U6.9 (Vin-)
- net BAT- renamed INP
- net CURRENT renamed INN
Other:
- moved on the sheet: C4
Changed lines of the file:
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@@
   (junction (at 301.625 107.95) (diameter 0) (color 0 0 0 0)
   )
-  (junction (at 133.35 178.435) (diameter 0) (color 0 0 0 0)
-  )
   (junction (at 134.62 173.355) (diameter 0) (color 0 0 0 0)
   )
@@
   (junction (at 298.45 178.435) (diameter 0) (color 0 0 0 0)
   )
-  (junction (at 133.35 187.325) (diameter 0) (color 0 0 0 0)
+  (junction (at 134.62 187.325) (diameter 0) (color 0 0 0 0)
   )
   (junction (at 361.95 102.87) (diameter 0) (color 0 0 0 0)
@@
   (junction (at 340.36 155.575) (diameter 0) (color 0 0 0 0)
   )
+  (junction (at 318.77 182.245) (diameter 0) (color 0 0 0 0)
+  )
   (junction (at 120.015 107.95) (diameter 0) (color 0 0 0 0)
   )
@@
   (junction (at 351.79 102.87) (diameter 0) (color 0 0 0 0)
   )
+  (junction (at 318.77 184.785) (diameter 0) (color 0 0 0 0)
+  )
   (junction (at 372.11 118.11) (diameter 0) (color 0 0 0 0)
+  )
+  (junction (at 134.62 178.435) (diameter 0) (color 0 0 0 0)
   )
   (junction (at 191.77 164.465) (diameter 0) (color 0 0 0 0)
@@
     (stroke (width 0) (type default))
   )
-  (wire (pts (xy 133.35 178.435) (xy 151.13 178.435))
-    (stroke (width 0) (type default))
-  )
   (wire (pts (xy 278.765 116.84) (xy 288.925 116.84))
     (stroke (width 0) (type default))
@@
     (stroke (width 0) (type default))
   )
-  (wire (pts (xy 133.35 183.515) (xy 133.35 187.325))
+  (wire (pts (xy 134.62 183.515) (xy 134.62 187.325))
     (stroke (width 0) (type default))
   )
@@
     (stroke (width 0) (type default))
   )
+  (wire (pts (xy 318.77 182.372) (xy 318.77 182.245))
+    (stroke (width 0) (type default))
+  )
   (wire (pts (xy 361.95 111.76) (xy 361.95 118.11))
     (stroke (width 0) (type default))
@@
     (stroke (width 0) (type default))
   )
+  (wire (pts (xy 318.77 182.245) (xy 330.2 182.245))
+    (stroke (width 0) (type default))
+  )
   (wire (pts (xy 191.77 164.465) (xy 205.74 164.465))
     (stroke (width 0) (type default))
@@
     (stroke (width 0) (type default))
   )
-  (wire (pts (xy 314.96 182.245) (xy 330.2 182.245))
+  (wire (pts (xy 314.96 182.245) (xy 318.77 182.245))
     (stroke (width 0) (type default))
   )
@@
     (stroke (width 0) (type default))
   )
-  (wire (pts (xy 133.35 178.435) (xy 133.35 180.975))
+  (wire (pts (xy 134.62 178.435) (xy 134.62 180.975))
     (stroke (width 0) (type default))
   )
@@
     (stroke (width 0) (type default))
   )
-  (wire (pts (xy 326.39 184.785) (xy 304.8 184.785))
-    (stroke (width 0) (type default))
-  )
   (wire (pts (xy 90.805 107.95) (xy 93.98 107.95))
     (stroke (width 0) (type default))
   )
-  (wire (pts (xy 125.73 178.435) (xy 133.35 178.435))
+  (wire (pts (xy 125.73 178.435) (xy 134.62 178.435))
     (stroke (width 0) (type default))
   )
@@
     (stroke (width 0) (type default))
   )
+  (wire (pts (xy 134.62 178.435) (xy 151.13 178.435))
+    (stroke (width 0) (type default))
+  )
   (wire (pts (xy 105.41 180.34) (xy 105.41 178.435))
     (stroke (width 0) (type default))
@@
     (stroke (width 0) (type default))
   )
+  (wire (pts (xy 318.77 184.912) (xy 318.77 184.785))
+    (stroke (width 0) (type default))
+  )
   (wire (pts (xy 120.015 116.84) (xy 123.825 116.84))
     (stroke (width 0) (type default))
@@
     (stroke (width 0) (type default))
   )
+  (wire (pts (xy 304.8 184.785) (xy 318.77 184.785))
+    (stroke (width 0) (type default))
+  )
   (wire (pts (xy 294.64 178.435) (xy 298.45 178.435))
     (stroke (width 0) (type default))
@@
     (stroke (width 0) (type default))
   )
-  (wire (pts (xy 151.13 187.325) (xy 133.35 187.325))
+  (wire (pts (xy 151.13 187.325) (xy 134.62 187.325))
     (stroke (width 0) (type default))
   )
@@
     (stroke (width 0) (type default))
   )
+  (wire (pts (xy 318.77 184.785) (xy 326.39 184.785))
+    (stroke (width 0) (type default))
+  )
   (wire (pts (xy 314.96 172.085) (xy 330.2 172.085))
     (stroke (width 0) (type default))
   )
-  (wire (pts (xy 125.73 187.325) (xy 133.35 187.325))
+  (wire (pts (xy 125.73 187.325) (xy 134.62 187.325))
     (stroke (width 0) (type default))
   )
@@
     (effects (font (size 1.27 1.27)) (justify left bottom))
   )
+  (label "INP" (at 95.25 178.435 0) (fields_autoplaced)
+    (effects (font (size 1.27 1.27)) (justify left bottom))
+  )
   (label "VBAT_SENSE" (at 330.835 111.76 0) (fields_autoplaced)
     (effects (font (size 1.27 1.27)) (justify left bottom))
@@
     (effects (font (size 1.27 1.27)) (justify left bottom))
   )
+  (label "INN" (at 95.25 187.325 0) (fields_autoplaced)
+    (effects (font (size 1.27 1.27)) (justify left bottom))
+  )
   (label "ISO+5V" (at 139.065 93.98 0) (fields_autoplaced)
     (effects (font (size 1.27 1.27)) (justify left bottom))
   )
+  (label "Vin-" (at 318.77 184.912 0) (fields_autoplaced)
+    (effects (font (size 1.27 1.27)) (justify left bottom))
+  )
+  (label "Vin+" (at 318.77 182.372 0) (fields_autoplaced)
+    (effects (font (size 1.27 1.27)) (justify left bottom))
+  )
   (hierarchical_label "ISO+5V" (shape input) (at 134.62 164.465 180) (fields_autoplaced)
     (effects (font (size 1.27 1.27)) (justify right))
@@
     (effects (font (size 1.27 1.27)) (justify left))
   )
-  (hierarchical_label "CURRENT" (shape input) (at 93.98 187.325 180) (fields_autoplaced)
-    (effects (font (size 1.27 1.27)) (justify right))
-  )
   (hierarchical_label "ISO+5V" (shape input) (at 135.255 93.98 180) (fields_autoplaced)
     (effects (font (size 1.27 1.27)) (justify right))
   )
-  (hierarchical_label "BAT-" (shape input) (at 93.98 178.435 180) (fields_autoplaced)
+  (hierarchical_label "INP" (shape input) (at 93.98 178.435 180) (fields_autoplaced)
     (effects (font (size 1.27 1.27)) (justify right))
   )
@@
       (effects (font (size 1.27 1.27)) hide)
     )
-    (property "Value" "GND" (at 315.087 180.2892 0)
+    (property "Value" "GND" (at 314.96 179.07 0)
       (effects (font (size 1.27 1.27)))
     )
@@
     )
   )
-  (symbol (lib_id "Device:C") (at 133.35 182.245 0) (unit 1)
-    (in_bom yes) (on_board yes) (dnp no)
-    (property "Reference" "C4" (at 133.985 180.34 0)
-      (effects (font (size 1.27 1.27)) (justify left))
-    )
-    (property "Value" "330pF/100V" (at 134.62 184.785 0)
-      (effects (font (size 1.27 1.27)) (justify left))
-    )
-    (property "Footprint" "Capacitor_SMD:C_0603_1608Metric" (at 134.3152 186.055 0)
-      (effects (font (size 1.27 1.27)) hide)
-    )
-    (property "Datasheet" "https://search.murata.co.jp/Ceramy/image/img/A01X/G101/ENG/GRM188R72A331KA01-01.pdf" (at 133.35 182.245 0)
-      (effects (font (size 1.27 1.27)) hide)
-    )
-    (property "MPN" "GRM188R72A331KA01D" (at 133.35 182.245 0)
-      (effects (font (size 1.27 1.27)) hide)
-    )
-    (property "Description" "330 pF ±10% 100V Ceramic Capacitor X7R 0603 (1608 Metric)" (at 133.35 182.245 0)
-      (effects (font (size 1.27 1.27)) hide)
-    )
-    (property "Link" "https://www.digikey.jp/en/products/detail/murata-electronics/GRM188R72A331KA01D/587128" (at 133.35 182.245 0)
+  (symbol (lib_id "Device:C") (at 134.62 182.245 0) (unit 1)
+    (in_bom yes) (on_board yes) (dnp no)
+    (property "Reference" "C4" (at 135.255 180.34 0)
+      (effects (font (size 1.27 1.27)) (justify left))
+    )
+    (property "Value" "330pF/100V" (at 135.89 184.785 0)
+      (effects (font (size 1.27 1.27)) (justify left))
+    )
+    (property "Footprint" "Capacitor_SMD:C_0603_1608Metric" (at 135.5852 186.055 0)
+      (effects (font (size 1.27 1.27)) hide)
+    )
+    (property "Datasheet" "https://search.murata.co.jp/Ceramy/image/img/A01X/G101/ENG/GRM188R72A331KA01-01.pdf" (at 134.62 182.245 0)
+      (effects (font (size 1.27 1.27)) hide)
+    )
+    (property "MPN" "GRM188R72A331KA01D" (at 134.62 182.245 0)
+      (effects (font (size 1.27 1.27)) hide)
+    )
+    (property "Description" "330 pF ±10% 100V Ceramic Capacitor X7R 0603 (1608 Metric)" (at 134.62 182.245 0)
+      (effects (font (size 1.27 1.27)) hide)
+    )
+    (property "Link" "https://www.digikey.jp/en/products/detail/murata-electronics/GRM188R72A331KA01D/587128" (at 134.62 182.245 0)
       (effects (font (size 1.27 1.27)) hide)
     )
@@
   (symbol (lib_id "Device:C") (at 248.92 183.515 0) (unit 1)
     (in_bom yes) (on_board yes) (dnp no)
-    (property "Reference" "C14" (at 251.841 182.3466 0)
-      (effects (font (size 1.27 1.27)) (justify left))
-    )
-    (property "Value" "2.2nF/16V" (at 251.841 184.658 0)
+    (property "Reference" "C14" (at 249.174 181.483 0)
+      (effects (font (size 1.27 1.27)) (justify left))
+    )
+    (property "Value" "2.2nF/16V" (at 249.301 185.42 0)
       (effects (font (size 1.27 1.27)) (justify left))
     )
@@
       (effects (font (size 1.27 1.27) (color 255 10 23 1)) (justify left top))
     )
-    (property "Footprint" "Resistor_SMD:R_PSR500HTQFB0L10_Metric_Pad5.2x8.75mm_HandSolder" (at 105.41 182.88 0)
-      (effects (font (size 1.27 1.27)) hide)
-    )
+    (property "Footprint" "Resistor_SMD:R_PSR500HTQFB0L10_Metric_Pad5.2x8.75mm_Hole" (at 105.41 182.88 0)
+      (effects (font (size 1.27 1.27)) hide)
+    )
