File: LTC6811_ESP32_V1p3/LTC6811.kicad_sch (KiCad schematic)
At the start: 61 parts, among them J13 B7B-XH-A, J14 B7B-XH-A, J15 PB MB, Q2 NSV1C201MZ4, U12 LTC6811HG-1

Commit message: Add files via upload
Parts:
- R58: value 100K -> 100R; Link https://www.digikey.jp/en/products/detail/yageo/RC0603JR-07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 -> https://www.digikey.jp/en/products/detail/yageo/RC0603FR-07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; MPN RC0603JR-07100KL -> RC0603FR-07100RL
- renumbered TP3 to TP4, TR2 to TR3, TR2 to TR4
Connections:
- net IMB: now also R58.2; no longer R58.1
- net IPB: now also R58.1; no longer R58.2
Changed lines of the file:
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@@
     (instances
       (project "LTC6811_ESP32_V1p3"
-        (path "/6a86ff6f-b159-4c4c-8a40-e732cc82e010/00000000-0000-0000-0000-00005ac18063"
+        (path "/6a86ff6f-b159-4c4c-8a40-e732cc82e010/0999518d-09c3-4a69-bd78-ff81b3ce8dd2"
           (reference "TP3") (unit 1)
         )
-        (path "/6a86ff6f-b159-4c4c-8a40-e732cc82e010/0999518d-09c3-4a69-bd78-ff81b3ce8dd2"
-          (reference "TP3") (unit 1)
-        )
       )
     )
@@
     )
   )
+  (symbol (lib_id "Device:R_Small") (at 213.995 118.745 90) (unit 1)
+    (in_bom yes) (on_board yes) (dnp no)
+    (property "Reference" "R58" (at 215.9 116.84 90)
+      (effects (font (size 1.27 1.27)) (justify left))
+    )
+    (property "Value" "100R" (at 216.535 120.65 90)
+      (effects (font (size 1.27 1.27)) (justify left))
+    )
+    (property "Footprint" "Resistor_SMD:R_0603_1608Metric" (at 213.995 120.523 90)
+      (effects (font (size 1.27 1.27)) hide)
+    )
+    (property "Datasheet" "https://www.yageo.com/upload/media/product/app/datasheet/rchip/pyu-rc_group_51_rohs_l.pdf" (at 213.995 118.745 0)
+      (effects (font (size 1.27 1.27)) hide)
+    )
+    (property "MPN" "RC0603FR-07100RL" (at 213.995 118.745 0)
+      (effects (font (size 1.27 1.27)) hide)
+    )
+    (property "Description" "100 Ohms ±1% 0.1W, 1/10W Chip Resistor 0603 (1608 Metric) Moisture Resistant Thick Film" (at 213.995 118.745 0)
+      (effects (font (size 1.27 1.27)) hide)
+    )
+    (property "Link" "https://www.digikey.jp/en/products/detail/yageo/RC0603FR-07100RL/726888?s=N4IgTCBcDaIEoGEAMA2JBmAYnAtEg7AIxJJwAyIAugL5A" (at 213.995 118.745 0)
+      (effects (font (size 1.27 1.27)) hide)
+    )
+    (pin "1")
+    (pin "2")
+    (instances
+      (project "LTC6811_ESP32_V1p3"
+        (path "/6a86ff6f-b159-4c4c-8a40-e732cc82e010/0999518d-09c3-4a69-bd78-ff81b3ce8dd2"
+          (reference "R58") (unit 1)
+        )
+      )
+      (project "LTC6811"
+        (path "/c4061cfa-a05d-44c7-ba89-bb211c8b143a"
+          (reference "R6") (unit 1)
+        )
+      )
+    )
+  )
   (symbol (lib_id "Connector:TestPoint") (at 304.165 156.845 270) (unit 1)
     (in_bom yes) (on_board yes) (dnp no)
-    (property "Reference" "TP3" (at 308.737 159.385 0)
+    (property "Reference" "TP4" (at 308.737 159.385 0)
       (effects (font (size 1.27 1.27)) (justify left) hide)
     )
@@
     (instances
       (project "LTC6811_ESP32_V1p3"
-        (path "/6a86ff6f-b159-4c4c-8a40-e732cc82e010/00000000-0000-0000-0000-00005ac18063"
-          (reference "TP3") (unit 1)
-        )
         (path "/6a86ff6f-b159-4c4c-8a40-e732cc82e010/0999518d-09c3-4a69-bd78-ff81b3ce8dd2"
           (reference "TP4") (unit 1)
@@
   (symbol (lib_id "ENNOID:HM2108NL") (at 316.23 51.435 180) (unit 1)
     (in_bom yes) (on_board yes) (dnp no)
-    (property "Reference" "TR2" (at 323.215 40.64 0)
+    (property "Reference" "TR4" (at 323.215 40.64 0)
       (effects (font (size 1.27 1.27)))
     )
@@
     (instances
       (project "LTC6811_ESP32_V1p3"
-        (path "/6a86ff6f-b159-4c4c-8a40-e732cc82e010/00000000-0000-0000-0000-00005ab72d4d"
-          (reference "TR2") (unit 1)
-        )
         (path "/6a86ff6f-b159-4c4c-8a40-e732cc82e010/0999518d-09c3-4a69-bd78-ff81b3ce8dd2"
           (reference "TR4") (unit 1)
@@
   (symbol (lib_id "ENNOID:HM2108NL") (at 316.23 66.675 180) (unit 1)
     (in_bom yes) (on_board yes) (dnp no)
-    (property "Reference" "TR2" (at 321.945 74.93 0)
+    (property "Reference" "TR3" (at 321.945 74.93 0)
       (effects (font (size 1.27 1.27)))
     )
@@
     (instances
       (project "LTC6811_ESP32_V1p3"
-        (path "/6a86ff6f-b159-4c4c-8a40-e732cc82e010/00000000-0000-0000-0000-00005ab72d4d"
-          (reference "TR2") (unit 1)
-        )
         (path "/6a86ff6f-b159-4c4c-8a40-e732cc82e010/0999518d-09c3-4a69-bd78-ff81b3ce8dd2"
           (reference "TR3") (unit 1)
@@
         )
       )
-    )
-  )
-  (symbol (lib_id "Device:R_Small") (at 213.995 118.745 270) (unit 1)
-    (in_bom yes) (on_board yes) (dnp no)
-    (property "Reference" "R58" (at 209.55 116.84 90)
-      (effects (font (size 1.27 1.27)) (justify left))
-    )
-    (property "Value" "100K" (at 214.63 116.84 90)
-      (effects (font (size 1.27 1.27)) (justify left))
-    )
-    (property "Footprint" "Resistor_SMD:R_0603_1608Metric" (at 213.995 116.967 90)
-      (effects (font (size 1.27 1.27)) hide)
-    )
-    (property "Datasheet" "https://www.yageo.com/upload/media/product/app/datasheet/rchip/pyu-rc_group_51_rohs_l.pdf" (at 213.995 118.745 0)
-      (effects (font (size 1.27 1.27)) hide)
-    )
-    (property "MPN" "RC0603JR-07100KL" (at 213.995 118.745 0)
-      (effects (font (size 1.27 1.27)) hide)
-    )
-    (property "Description" "100 kOhms ±5% 0.1W, 1/10W Chip Resistor 0603 (1608 Metric) Moisture Resistant Thick Film" (at 213.995 118.745 0)
-      (effects (font (size 1.27 1.27)) hide)
-    )
-    (property "Link" "https://www.digikey.jp/en/products/detail/yageo/RC0603JR-07100KL/726698?s=N4IgTCBcDaIEoGEAMA2JBmAUnAtEg7AIxJIDSAMiALoC%2BQA" (at 213.995 118.745 0)
-      (effects (font (size 1.27 1.27)) hide)
-    )
-    (pin "1")
-    (pin "2")
-    (instances
-      (project "LTC6811_ESP32_V1p3"
-        (path "/6a86ff6f-b159-4c4c-8a40-e732cc82e010/0999518d-09c3-4a69-bd78-ff81b3ce8dd2"
-          (reference "R58") (unit 1)
-        )
-      )
-      (project "LTC6811"
-        (path "/c4061cfa-a05d-44c7-ba89-bb211c8b143a"
-          (reference "R60") (unit 1)
-        )
-      )

Commit message: change page setting A3 for print
change page setting A3 for print
Other:
- moved on the sheet: C22, C46, C47, C48, C49, C50, C51, C52, C53, C54, C55, C56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
