File: LTC6811_ESP32_V1p3/MCU.kicad_sch (KiCad schematic)
At the start: 17 parts, among them J5 UART /NC, J6 JTAG /NC, U8 ESP32-DevKitC V4, U9 LTC6820

Commit message: Optimize signal transmission lines.
Connections:
- net CAN_RX is gone; now on net RX_USB: J5.2 (Pin_2), U8.34 (RXD0)
- net CAN_TX is gone; now on net TX_USB: J5.3 (Pin_3), U8.35 (TXD0)
- net MTCK: now also J6.3 (Pin_3); no longer J6.4 (Pin_4)
- net MTDO: now also J6.4 (Pin_4); no longer J6.3 (Pin_3)
- net RX_USB: no longer U8.16 (SD2)
- net TX_USB: no longer U8.17 (SD3)
- no-connect marks 8 -> 10
Changed lines of the file:
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@@
   (junction (at 146.685 79.375) (diameter 0) (color 0 0 0 0)
   )
+  (no_connect (at 59.055 161.925))
   (no_connect (at 59.055 167.005))
   (no_connect (at 59.055 128.905))
@@
   (no_connect (at 102.235 154.305))
   (no_connect (at 29.845 59.055))
+  (no_connect (at 59.055 164.465))
   (no_connect (at 102.235 151.765))
   (wire (pts (xy 102.235 164.465) (xy 111.76 164.465))
@@
     (stroke (width 0) (type default))
   )
-  (wire (pts (xy 48.26 161.925) (xy 59.055 161.925))
-    (stroke (width 0) (type default))
-  )
   (wire (pts (xy 106.045 83.185) (xy 106.045 93.345))
     (stroke (width 0) (type default))
@@
     (stroke (width 0) (type default))
   )
-  (wire (pts (xy 48.26 164.465) (xy 59.055 164.465))
-    (stroke (width 0) (type default))
-  )
   (wire (pts (xy 127 131.445) (xy 135.89 131.445))
     (stroke (width 0) (type default))
@@
     (effects (font (size 1.27 1.27)) (justify right bottom))
   )
-  (label "CAN_RX" (at 127.635 131.445 0) (fields_autoplaced)
-    (effects (font (size 1.27 1.27)) (justify left bottom))
-  )
   (label "MTCK" (at 51.435 159.385 0) (fields_autoplaced)
     (effects (font (size 1.27 1.27)) (justify left bottom))
   )
-  (label "MTCK" (at 130.175 162.56 0) (fields_autoplaced)
+  (label "MTCK" (at 130.175 160.02 0) (fields_autoplaced)
     (effects (font (size 1.27 1.27)) (justify left bottom))
   )
@@
     (effects (font (size 1.27 1.27)) (justify left bottom))
   )
-  (label "MTDO" (at 130.175 160.02 0) (fields_autoplaced)
+  (label "MTDO" (at 130.175 162.56 0) (fields_autoplaced)
     (effects (font (size 1.27 1.27)) (justify left bottom))
   )
@@
     (effects (font (size 1.27 1.27)) (justify left bottom))
   )
-  (label "CAN_TX" (at 127.635 133.985 0) (fields_autoplaced)
-    (effects (font (size 1.27 1.27)) (justify left bottom))
-  )
   (label "MOSI" (at 106.045 126.365 0) (fields_autoplaced)
     (effects (font (size 1.27 1.27)) (justify left bottom))
@@
     (effects (font (size 1.27 1.27)) (justify left bottom))
   )
+  (label "TX_USB" (at 128.27 133.985 0) (fields_autoplaced)
+    (effects (font (size 1.27 1.27)) (justify left bottom))
+  )
   (label "MTDI" (at 130.175 157.48 0) (fields_autoplaced)
     (effects (font (size 1.27 1.27)) (justify left bottom))
   )
+  (label "RX_USB" (at 128.27 131.445 0) (fields_autoplaced)
+    (effects (font (size 1.27 1.27)) (justify left bottom))
+  )
   (label "MTMS" (at 130.175 154.94 0) (fields_autoplaced)
     (effects (font (size 1.27 1.27)) (justify left bottom))
@@
     (effects (font (size 1.27 1.27)) (justify left))
   )
-  (hierarchical_label "CAN_RX" (shape input) (at 111.76 133.985 0) (fields_autoplaced)
-    (effects (font (size 1.27 1.27)) (justify left))
-  )
-  (hierarchical_label "CAN_TX" (shape input) (at 111.76 131.445 0) (fields_autoplaced)
-    (effects (font (size 1.27 1.27)) (justify left))
-  )
   (hierarchical_label "PA" (shape input) (at 23.495 64.135 180) (fields_autoplaced)
     (effects (font (size 1.27 1.27)) (justify right))
@@
     (effects (font (size 1.27 1.27)) (justify right))
   )
-  (hierarchical_label "RX_USB" (shape input) (at 48.26 161.925 180) (fields_autoplaced)
-    (effects (font (size 1.27 1.27)) (justify right))
+  (hierarchical_label "RX_USB" (shape input) (at 111.76 133.985 0) (fields_autoplaced)
+    (effects (font (size 1.27 1.27)) (justify left))
   )
   (hierarchical_label "LED0" (shape input) (at 48.26 146.685 180) (fields_autoplaced)
@@
     (effects (font (size 1.27 1.27)) (justify left))
   )
-  (hierarchical_label "TX_USB" (shape input) (at 48.26 164.465 180) (fields_autoplaced)
-    (effects (font (size 1.27 1.27)) (justify right))
+  (hierarchical_label "TX_USB" (shape input) (at 111.76 131.445 0) (fields_autoplaced)
+    (effects (font (size 1.27 1.27)) (justify left))
   )
   (symbol (lib_id "Device:R_Small") (at 94.615 50.165 180) (unit 1)
