File: LTC6811_ESP32_V1p3/PowerMonitor.kicad_sch (KiCad schematic)
At the start: 51 parts, among them U2 AMC1301 or AMC1302, U3 AMC1301, U5 OPA2197IDR, U6 ISL28022

Commit message: Add files via upload
Parts:
- renumbered C15 to C11, C62 to C12, C9 to C14, C65 to C15, C10 to C16, C68 to C17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
