File: LTC6811_ESP32_V1p3/PowerSupply.kicad_sch (KiCad schematic)
At the start: 26 parts, among them J15 PB MB, U1 TPS76350, U4 SN6501DBV, U7 LMR51420XDDCR

Commit message: Optimize signal transmission lines.
Connections:
- net +12V: now also J15.1 (Pin_1); no longer J15.2 (Pin_2)
- net GND: now also J15.2 (Pin_2); no longer J15.1 (Pin_1)
Other:
- moved on the sheet: J15
Changed lines of the file:
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@@
     )
   )
-  (symbol (lib_id "Connector_Generic:Conn_01x02") (at 51.435 61.595 180) (unit 1)
+  (symbol (lib_id "Connector_Generic:Conn_01x02") (at 51.435 59.055 0) (mirror y) (unit 1)
     (in_bom yes) (on_board yes) (dnp no)
-    (property "Reference" "J15" (at 49.403 61.3918 0)
+    (property "Reference" "J15" (at 49.403 59.2582 0)
       (effects (font (size 1.27 1.27)) (justify left))
     )
-    (property "Value" "PB MB" (at 49.403 59.0804 0)
+    (property "Value" "PB MB" (at 49.403 61.5696 0)
       (effects (font (size 1.27 1.27)) (justify left))
     )
-    (property "Footprint" "Connector_JST:JST_VH_B2P-VH-B_1x02_P3.96mm_Vertical" (at 51.435 61.595 0)
+    (property "Footprint" "Connector_JST:JST_VH_B2P-VH-B_1x02_P3.96mm_Vertical" (at 51.435 59.055 0)
       (effects (font (size 1.27 1.27)) hide)
     )
-    (property "Datasheet" "https://www.jst-mfg.com/product/pdf/eng/eVH.pdf" (at 51.435 61.595 0)
+    (property "Datasheet" "https://www.jst-mfg.com/product/pdf/eng/eVH.pdf" (at 51.435 59.055 0)
       (effects (font (size 1.27 1.27)) hide)
     )
-    (property "MPN" "B2P-VH" (at 51.435 61.595 0)
+    (property "MPN" "B2P-VH" (at 51.435 59.055 0)
       (effects (font (size 1.27 1.27)) hide)
     )
-    (property "Link" "https://www.digikey.jp/en/products/detail/jst-sales-america-inc/B2P-VH/926547" (at 51.435 61.595 0)
+    (property "Link" "https://www.digikey.jp/en/products/detail/jst-sales-america-inc/B2P-VH/926547" (at 51.435 59.055 0)
       (effects (font (size 1.27 1.27)) hide)
     )
-    (property "Description" "Connector Header Through Hole 2 position 0.156\" (3.96mm)" (at 51.435 61.595 0)
+    (property "Description" "Connector Header Through Hole 2 position 0.156\" (3.96mm)" (at 51.435 59.055 0)
       (effects (font (size 1.27 1.27)) hide)
     )

Commit message: Add files via upload
Parts:
- renumbered C3 to C2, C3 to C25, J15 to J1, R65 to R37
