File: LTC6811_ESP32_V1p3/USB.kicad_sch (KiCad schematic)
At the start: 11 parts, among them J8 SERIAL /NC, U10 CP2104

Commit message: Optimize signal transmission lines.
Parts:
- removed J8: SERIAL /NC, Connector_PinHeader_2.54mm:PinHeader_1x04_P2.54mm_Vertical, symbol Connector_Generic:Conn_01x04
- R49, R50: value 240R -> 0; Link https://www.digikey.jp/en/products/detail/yageo/RC0603FR-07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 -> https://www.digikey.jp/en/products/detail/yageo/RC0603JR-07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; MPN RC0603FR-07240RL -> RC0603JR-070RL
Connections:
- net VDD is gone; now on net +3V3: C39.1, R51.1, U10.5 (VIO), U10.6 (VDD)

Commit message: Add files via upload
Parts:
- renumbered C39 to C38, C40 to C39, C41 to C40, C42 to C41, D8 to D7
