File: LTC6811_ESP32_V1p3/cell.kicad_sch (KiCad schematic)
At the start: 6 parts, among them Q3 TSM2323

Commit message: kicad v8対応
kicad v8対応
Parts:
- renumbered C59 to C60, D13 to D14, Q3 to Q4, R68 to R71, R69 to R72, R70 to R73
