File: Slaves/ESP32_Slaves_V0/ESP32_Slaves_V0.kicad_pcb (KiCad board)
At the start: 2 copper layers, 168.3 x 81.7 mm, 147 parts, among them J1 B7B-XH-A, J2 B7B-XH-A, J3 PB MB, J4 PB MA, J6 Hole /NC, J7 Hole /NC, J8 Hole /NC, Q1 TSM2323, Q10 TSM2323, Q11 TSM2323, Q12 TSM2323, Q13 NSV1C201MZ4, Q2 TSM2323, Q3 TSM2323, Q4 TSM2323, Q5 TSM2323, Q6 TSM2323, Q7 TSM2323, Q8 TSM2323, Q9 TSM2323, U1 LTC6811HG-1

Commit message: Add files via upload
Parts:
- moved TH5 109.4 mm to (240.9, 132.5), turned to -90 degrees
- moved TH4 107.7 mm to (238.7, 132.5), turned to -90 degrees
- moved D14 107.4 mm to (80.1, 95.4), turned to 90 degrees
- moved TH3 106.0 mm to (236.5, 132.5), turned to -90 degrees
- moved R45 105.7 mm to (245.6, 125.8), turned to -90 degrees
- moved C25 105.2 mm to (240.8, 129.0), turned to -90 degrees
- moved TH2 104.5 mm to (234.3, 132.5), turned to -90 degrees
- moved C16 104.3 mm to (244.0, 125.8), turned to -90 degrees
- moved TH1 104.2 mm to (232.3, 133.4), turned to -90 degrees
- moved C24 103.5 mm to (238.7, 129.0), turned to -90 degrees
- moved C15 102.9 mm to (242.4, 125.8), turned to -90 degrees
- moved D13 102.5 mm to (82.5, 95.4), turned to 90 degrees
- moved C23 102.3 mm to (237.1, 129.0), turned to -90 degrees
- moved R50 101.6 mm to (240.8, 125.8), turned to 90 degrees
- moved R52 100.7 mm to (102.2, 64.4), turned to -90 degrees
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Routing:
- net /cell1/C+: track 0.00 -> 147.7 mm
- net /cell6/C+: track 0.00 -> 146.8 mm
- net /cell2/C+: track 0.00 -> 145.7 mm
- net /cell3/C+: track 0.00 -> 143.7 mm
- net /cell7/C+: track 0.00 -> 141.9 mm
- net /cell4/C+: track 0.00 -> 139.1 mm
- net /cell8/C+: track 0.00 -> 138.2 mm
- net /cell5/C+: track 0.00 -> 135.5 mm
- net /cell10/C-: track 0.00 -> 134.7 mm
- net /cell10/C+: track 0.00 -> 129.8 mm
- net /cell11/C+: track 1.20 -> 112.9 mm
- net /cell12/C+: track 0.00 -> 92.9 mm
- net /BAT+: track 0.00 -> 39.3 mm
Other:
- board size 168.3 x 81.7 mm -> 64.9 x 99.9 mm

Commit message: Add files via upload
Parts:
- added J10: PACK-, Connector_JST:JST_VH_B2P-VH-B_1x02_P3.96mm_Vertical, F.Cu at (119.7, 43.8)
- added J5: Hole /NC, MountingHole:MountingHole_3.2mm_M3_ISO7380_Pad, F.Cu at (104.0, 44.1)
- added J9: BAT+, Connector_JST:JST_VH_B2P-VH-B_1x02_P3.96mm_Vertical, F.Cu at (160.6, 99.0)
- R47, R48, R49, R50, R51: value 100K -> 10K
- TH1, TH4, TH5: value 100K NTC -> 10K NTC
- TH2, TH3: value 100K NTC -> 10K NTC; footprint Resistor_THT:R_Axial_DIN0204_L3.6mm_D1.6mm_P1.90mm_Vertical -> Resistor_SMD:R_0603_1608Metric
- moved R50 132.0 mm to (109.5, 111.5), turned to 180 degrees
- moved R49 130.2 mm to (109.5, 109.4), turned to 180 degrees
- moved TH5 130.0 mm to (112.3, 113.5), turned to 90 degrees
- moved TH1 129.2 mm to (120.8, 68.0), turned to 90 degrees
- moved R48 128.9 mm to (109.5, 107.2), turned to 180 degrees
- moved R47 127.0 mm to (109.5, 105.3), turned to 180 degrees
- moved TH4 126.3 mm to (114.5, 109.4)
- moved R51 125.8 mm to (109.5, 103.5), turned to 0 degrees
- moved C23 125.4 mm to (113.6, 107.2), turned to 0 degrees
- moved C25 124.7 mm to (117.4, 111.5), turned to 0 degrees
- moved J6 124.1 mm to (160.8, 44.1)
- moved C22 123.6 mm to (113.6, 105.3), turned to 0 degrees
- moved C24 122.9 mm to (117.4, 109.4), turned to 0 degrees
- moved C26 122.5 mm to (113.6, 103.5), turned to 0 degrees
- moved C16 121.6 mm to (123.3, 110.9)
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Routing:
- net /cell12/C+: track 92.9 -> 187.3 mm
- net /cell11/C+: track 112.9 -> 186.0 mm
- net /T3: track 0.00 -> 65.2 mm, vias 0 -> 1
- net /T2: track 0.00 -> 53.3 mm, vias 0 -> 1
- net /T1: track 0.00 -> 51.7 mm, vias 0 -> 1
- net /cell10/C+: track 129.8 -> 181.3 mm
- net /cell10/C-: track 134.7 -> 182.9 mm
- net /cell12/C: track 0.00 -> 40.8 mm
- net /cell12/S: track 0.00 -> 39.4 mm
- net /BAT+: track 39.3 -> 0.00 mm
- net /cell11/C: track 0.00 -> 39.0 mm
- net /cell5/C+: track 135.5 -> 171.5 mm
- net /cell11/S: track 0.00 -> 35.5 mm
- net /cell8/C+: track 138.2 -> 172.5 mm
- net /cell10/S: track 0.00 -> 34.0 mm
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- added copper zone on F.Cu, net GND_PACK
Other:
- board size 64.9 x 99.9 mm -> 65.9 x 99.9 mm

Commit message: Add files via upload
Parts:
- C1, C10, C11, C12, C13, C14, C15, C16, C17, C18, C19, C2, C20, C21, C22, C23, C24, C25, C26, C3, C4, C5, C6, C7, C8, C9: footprint Capacitor_SMD:C_0603_1608Metric -> Library:C_0603_1608Metric
- D1, D10, D11, D12, D2, D3, D4, D5, D6, D7, D8, D9: footprint Diode_SMD:D_SOD-323_HandSoldering -> Library:D_SOD-323_HandSoldering
- D13, D14: footprint Diode_SMD:D_SOD-123 -> Library:D_SOD-123
- D15: footprint Diode_SMD:D_SOD-123F -> Library:D_SOD-123F
- D16: footprint LED_SMD:LED_0603_1608Metric -> Library:LED_0603_1608Metric
- F1, F10, F11, F12, F13, F14, F2, F3, F4, F5, F6, F8, F9: footprint Fuse:Fuse_0805_2012Metric -> Library:Fuse_0805_2012Metric
- FB1, R11, R12, R14, R15, R17, R18, R2, R20, R21, R23, R24, R26, R27, R29, R3, R30, R32, R33, R35, R36, R37, R38, R39, R40, R41, R42, R43, R44, R45, R46, R47, R48, R49, R5, R50, R51, R6, R8, R9, TH1, TH2, TH3: footprint Resistor_SMD:R_0603_1608Metric -> Library:R_0603_1608Metric
- J1, J2: footprint Connector_JST:JST_XH_B7B-XH-A_1x07_P2.50mm_Vertical_BAT_6S -> Library:JST_XH_B7B-XH-A_1x07_P2.50mm_Vertical_BAT_6S
- J10, J3, J4, J9: footprint Connector_JST:JST_VH_B2P-VH-B_1x02_P3.96mm_Vertical -> Library:JST_VH_B2P-VH-B_1x02_P3.96mm_Vertical
- J5, J6, J7, J8: footprint MountingHole:MountingHole_3.2mm_M3_ISO7380_Pad -> Library:MountingHole_3.2mm_M3_ISO7380_Pad
- LOGO1: footprint Symbol:teTra-LOGO -> Library:teTra-LOGO
- Q1, Q10, Q11, Q12, Q2, Q3, Q4, Q5, Q6, Q7, Q8, Q9: footprint Package_TO_SOT_SMD:SOT-23 -> Library:SOT-23
- Q13: footprint Package_TO_SOT_SMD:SOT-223 -> Library:SOT-223
- R1, R10, R13, R16, R19, R22, R25, R28, R31, R34, R4, R52, R53, R54, R55, R56, R57, R58, R59, R60, R61, R62, R63, R7: footprint Resistor_SMD:R_2512_6332Metric -> Library:R_2512_6332Metric
- TH4, TH5: footprint Resistor_THT:R_Axial_DIN0204_L3.6mm_D1.6mm_P1.90mm_Vertical -> Library:R_Axial_DIN0204_L3.6mm_D1.6mm_P1.90mm_Vertical
- TR1: footprint Transformer_SMD:HM2102NL_PUL -> Library:HM2102NL_PUL
- U1: footprint Package_SO:TSSOP-48_6.1x12.5mm_P0.5mm -> Library:TSSOP-48_6.1x12.5mm_P0.5mm
- moved LOGO1 98.9 mm to (138.7, 42.8), turned to 180 degrees
- moved R38 26.7 mm to (147.1, 101.8), turned to 180 degrees
- moved R39 25.5 mm to (147.1, 100.2), turned to 180 degrees
- moved C17 21.4 mm to (144.0, 100.2), turned to 180 degrees
- moved R37 20.3 mm to (117.7, 117.8), turned to 180 degrees
- moved D16 16.3 mm to (120.9, 117.8), turned to 0 degrees
- moved C18 14.9 mm to (137.2, 121.0), turned to -90 degrees
- moved Q13 13.8 mm to (130.0, 120.2), turned to 0 degrees
- moved D15 6.77 mm to (149.9, 100.5)
- moved C19 6.55 mm to (120.9, 122.5), turned to 180 degrees
- moved J9 4.45 mm to (161.7, 94.7), turned to -90 degrees
- moved C20 4.40 mm to (120.9, 121.0), turned to 180 degrees
- moved R44 3.08 mm to (128.0, 114.9)
- moved R43 3.08 mm to (129.5, 114.9)
- moved D14 2.91 mm to (154.7, 100.2)
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Routing:
- net GND_PACK: track 2.97 -> 224.5 mm, vias 3 -> 177
- net Net-(C18-Pad1): track 0.00 -> 39.0 mm
- net /BAT+: track 0.00 -> 33.4 mm
- net /Vref2: track 5.63 -> 30.9 mm
- net /T3: track 65.2 -> 86.4 mm, vias 1 -> 2
- net /T2: track 53.3 -> 71.7 mm, vias 1 -> 2
- net Net-(U1-V+): track 0.00 -> 16.5 mm
- net /C2_G: track 0.00 -> 16.1 mm
- net /Vreg: track 15.8 -> 28.7 mm, vias 0 -> 2
- net /cell10/C+: track 181.3 -> 170.6 mm, vias 0 -> 44
- net /cell11/C+: track 186.0 -> 175.5 mm, vias 0 -> 44
- net /cell8/C+: track 172.5 -> 163.7 mm, vias 0 -> 40
- net /cell6/C+: track 171.5 -> 163.0 mm, vias 0 -> 36
- net /cell7/C+: track 168.0 -> 160.3 mm, vias 0 -> 36
- net Net-(J3-Pin_2): track 0.00 -> 7.61 mm
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- added copper zone on F.Cu, net /Vreg
- added copper zone on B.Cu, net /cell1/C+
- added copper zone on F.Cu, net /cell1/C+
- added copper zone on B.Cu, net /cell10/C+
- added copper zone on F.Cu, net /cell10/C+
- added copper zone on B.Cu, net /cell10/C-
- added copper zone on F.Cu, net /cell10/C-
- added copper zone on B.Cu, net /cell11/C+
- added copper zone on F.Cu, net /cell11/C+
- added copper zone on B.Cu, net /cell2/C+
- added copper zone on F.Cu, net /cell2/C+
- added copper zone on B.Cu, net /cell3/C+
- added copper zone on F.Cu, net /cell3/C+
- added copper zone on B.Cu, net /cell4/C+
- added copper zone on F.Cu, net /cell4/C+
- added copper zone on B.Cu, net /cell5/C+
- added copper zone on F.Cu, net /cell5/C+
- added copper zone on B.Cu, net /cell6/C+
- added copper zone on F.Cu, net /cell6/C+
- added copper zone on B.Cu, net /cell7/C+
- added copper zone on F.Cu, net /cell7/C+
- added copper zone on B.Cu, net /cell8/C+
- added copper zone on F.Cu, net /cell8/C+
- added copper zone on B.Cu, net GND_PACK
- added copper zone on F.Cu, net Net-(C18-Pad1)
- added copper zone on B.Cu, net Net-(Q1-D)
- added copper zone on F.Cu, net Net-(Q1-D)
- added copper zone on B.Cu, net Net-(Q10-D)
- added copper zone on F.Cu, net Net-(Q10-D)
- added copper zone on B.Cu, net Net-(Q11-D)
- added copper zone on F.Cu, net Net-(Q11-D)
- added copper zone on B.Cu, net Net-(Q12-D)
- added copper zone on F.Cu, net Net-(Q12-D)
- added copper zone on B.Cu, net Net-(Q2-D)
- added copper zone on F.Cu, net Net-(Q2-D)
- added copper zone on B.Cu, net Net-(Q3-D)
- added copper zone on F.Cu, net Net-(Q3-D)
- added copper zone on B.Cu, net Net-(Q4-D)
- added copper zone on F.Cu, net Net-(Q4-D)
- added copper zone on B.Cu, net Net-(Q5-D)
- added copper zone on F.Cu, net Net-(Q5-D)
- added copper zone on B.Cu, net Net-(Q6-D)
- added copper zone on F.Cu, net Net-(Q6-D)
- added copper zone on B.Cu, net Net-(Q7-D)
- added copper zone on F.Cu, net Net-(Q7-D)
- added copper zone on B.Cu, net Net-(Q8-D)
- added copper zone on F.Cu, net Net-(Q8-D)
- added copper zone on B.Cu, net Net-(Q9-D)
- added copper zone on F.Cu, net Net-(Q9-D)
- added copper zone on B.Cu, net Net-(R1-Pad1)
- added copper zone on F.Cu, net Net-(R1-Pad1)
- added copper zone on B.Cu, net Net-(R10-Pad1)
- added copper zone on F.Cu, net Net-(R10-Pad1)
- added copper zone on B.Cu, net Net-(R13-Pad1)
- added copper zone on F.Cu, net Net-(R13-Pad1)
- added copper zone on B.Cu, net Net-(R16-Pad1)
- added copper zone on F.Cu, net Net-(R16-Pad1)
- added copper zone on B.Cu, net Net-(R19-Pad1)
- added copper zone on F.Cu, net Net-(R19-Pad1)
- added copper zone on B.Cu, net Net-(R22-Pad1)
- added copper zone on F.Cu, net Net-(R22-Pad1)
- added copper zone on B.Cu, net Net-(R25-Pad1)
- added copper zone on F.Cu, net Net-(R25-Pad1)
- added copper zone on B.Cu, net Net-(R28-Pad1)
- added copper zone on F.Cu, net Net-(R28-Pad1)
- added copper zone on B.Cu, net Net-(R31-Pad1)
- added copper zone on F.Cu, net Net-(R31-Pad1)
- added copper zone on B.Cu, net Net-(R34-Pad1)
- added copper zone on F.Cu, net Net-(R34-Pad1)
- added copper zone on B.Cu, net Net-(R4-Pad1)
- added copper zone on F.Cu, net Net-(R4-Pad1)
- added copper zone on B.Cu, net Net-(R54-Pad2)
- added copper zone on F.Cu, net Net-(R54-Pad2)
Other:
- board text added: "2024/06/14"
- board text added: "ESP32_Slaves_V0 2024/06/14"
- board text added: "Slaves_V0"
- board text removed: "2024/02/26"
- board text removed: "LTC6811_Slaves_V1p2 2024/02/26"
- board text removed: "Slaves_V1P2"
