File: LTC6811_ESP32_V2/CAN.kicad_sch (KiCad schematic)
At the start: 6 parts, among them U10 ISO1050DUBR

Commit message: Add files via upload
Parts:
- C33, C34, C35, C36: symbol Device:C -> Library:C
- D5: symbol Power_Protection:SZNUP2105L -> Library:SZNUP2105L
- U10: symbol ENNOID:ISO1050DUBR -> Library:ISO1050DUBR
Changed lines of the file:
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@@
 	)
 	(symbol
-		(lib_id "ENNOID:ISO1050DUBR")
+		(lib_id "Library:ISO1050DUBR")
 		(at 187.452 138.938 0)
 		(unit 1)
@@
 	)
 	(symbol
-		(lib_id "power:GND")
+		(lib_id "Library:GND")
 		(at 173.482 145.288 0)
 		(unit 1)
@@
 	)
 	(symbol
-		(lib_id "Device:C")
+		(lib_id "Library:C")
 		(at 140.462 138.938 0)
 		(unit 1)
@@
 	)
 	(symbol
-		(lib_id "power:GND")
+		(lib_id "Library:GND")
 		(at 140.462 142.113 0)
 		(unit 1)
@@
 	)
 	(symbol
-		(lib_id "Device:C")
+		(lib_id "Library:C")
 		(at 129.032 138.938 0)
 		(unit 1)
@@
 	)
 	(symbol
-		(lib_id "power:GND")
+		(lib_id "Library:GND")
 		(at 129.032 142.113 0)
 		(unit 1)
@@
 	)
 	(symbol
-		(lib_id "Device:C")
+		(lib_id "Library:C")
 		(at 222.377 126.238 180)
 		(unit 1)
@@
 	)
 	(symbol
-		(lib_id "Device:C")
+		(lib_id "Library:C")
 		(at 213.487 126.238 0)
 		(unit 1)
@@
 	)
 	(symbol
-		(lib_id "Power_Protection:SZNUP2105L")
+		(lib_id "Library:SZNUP2105L")
 		(at 223.012 149.098 0)
 		(unit 1)
@@
 	)
 	(symbol
-		(lib_id "power:+3V3")
+		(lib_id "Library:+3V3")
 		(at 173.482 132.588 0)
 		(mirror y)
@@
 	)
 	(symbol
-		(lib_id "power:+3V3")
+		(lib_id "Library:+3V3")
 		(at 129.032 135.763 0)
 		(mirror y)
@@
 	)
 	(symbol
-		(lib_id "power:+3V3")
+		(lib_id "Library:+3V3")
 		(at 140.462 135.763 0)
 		(mirror y)
