File: LTC6811_ESP32_V2/LTC6811_ESP32_V2.kicad_pcb (KiCad board)
At the start: 2 copper layers, 360 x 55 mm, 568 parts, among them J1 Hole /NC, J10 B7B-XH-A, J11 B7B-XH-A, J12 B7B-XH-A, J13 B7B-XH-A, J14 B7B-XH-A, J15 B7B-XH-A, J16 B7B-XH-A, J17 B7B-XH-A, J18 B2P-VH-B, J2 Hole /NC, J3 Hole /NC, J4 Hole /NC, J5 CAN /NC, J6 Molex 5569, J7 B2P-VH-B, J8 JTAG /NC, J9 B2P-VH-B, Q1 NSV1C201MZ4, Q10 TSM2323, Q11 TSM2323, Q12 TSM2323, Q13 TSM2323, Q14 NSV1C201MZ4, Q15 TSM2323, Q16 TSM2323, Q17 TSM2323, Q18 TSM2323, Q19 TSM2323, Q2 TSM2323, Q20 TSM2323, Q21 TSM2323, Q22 TSM2323, Q23 TSM2323, Q24 TSM2323, Q25 TSM2323, Q26 TSM2323, Q27 NSV1C201MZ4, Q28 TSM2323, Q29 TSM2323, Q3 TSM2323, Q30 TSM2323, Q31 TSM2323, Q32 TSM2323, Q33 TSM2323, Q34 TSM2323, Q35 TSM2323, Q36 TSM2323, Q37 TSM2323, Q38 TSM2323, Q39 TSM2323, Q4 TSM2323, Q40 NSV1C201MZ4, Q41 TSM2323, Q42 TSM2323, Q43 TSM2323, Q44 TSM2323, Q45 TSM2323, Q46 TSM2323, Q47 TSM2323, Q48 TSM2323, Q49 TSM2323, Q5 TSM2323, Q50 TSM2323, Q51 TSM2323, Q52 TSM2323, Q6 TSM2323, Q7 TSM2323, Q8 TSM2323, Q9 TSM2323, U10 ISO1050DUBR, U11 LTC6811HG-1, U12 LTC6811HG-1, U13 LTC6811HG-1, U14 LTC6811HG-1, U6 LMR51420XDDCR, U8 ESP32-DevKitC V4, U9 LTC6820

Commit message: Add files via upload
Parts:
- removed C118, C120, C121, C68, C69, C92, C94, C95: 1uF/25V, Capacitor_SMD:C_0603_1608Metric
- removed C122, C123: 100pF/100V, Capacitor_SMD:C_0603_1608Metric
- removed R144, R195: 1.2K, Resistor_SMD:R_0603_1608Metric
- removed R148, R199: 100K, Resistor_SMD:R_0603_1608Metric
- removed R149, R200: 806R, Resistor_SMD:R_0603_1608Metric
- removed R151, R202: 100R, Resistor_SMD:R_0603_1608Metric
- added C24: 10nF/100V, Library:C_0402_1005Metric, F.Cu at (54.0, 150.7)
- added C26: 10nF/100V, Library:C_0402_1005Metric, F.Cu at (77.5, 161.6)
- added C46: 10nF/100V, Library:C_0402_1005Metric, F.Cu at (-134.0, 566.2)
- added C47: 10nF/100V, Library:C_0402_1005Metric, F.Cu at (116.9, 175.8)
- added C48: 10nF/100V, Library:C_0402_1005Metric, F.Cu at (241.1, 470.3)
- added C49: 10nF/100V, Library:C_0402_1005Metric, F.Cu at (116.9, 178.3)
- added C50: 10nF/100V, Library:C_0402_1005Metric, F.Cu at (77.0, 160.0)
- added C72: 10nF/100V, Library:C_0402_1005Metric, F.Cu at (241.1, 472.8)
- added C73: 10nF/100V, Library:C_0402_1005Metric, F.Cu at (53.5, 152.2)
- added C74: 10nF/100V, Library:C_0402_1005Metric, F.Cu at (34.1, 151.7)
- added C75: 10nF/100V, Library:C_0402_1005Metric, F.Cu at (184.0, 176.1)
- added C76: 10nF/100V, Library:C_0402_1005Metric, F.Cu at (184.0, 178.6)
- added R1: 49.9R, Library:R_0402_1005Metric, F.Cu at (54.5, 149.2)
- added R101: 1K, Library:R_0603_1608Metric, F.Cu at (289.6, 401.2)
- added R2: 49.9R, Library:R_0402_1005Metric, F.Cu at (174.0, 208.5)
- added R23: 49.9R, Library:R_0402_1005Metric, F.Cu at (-166.2, 586.8)
- added R24: 49.9R, Library:R_0402_1005Metric, F.Cu at (202.6, 476.6)
- added R25: 49.9R, Library:R_0402_1005Metric, F.Cu at (54.5, 153.2)
- added R26: 49.9R, Library:R_0402_1005Metric, F.Cu at (218.5, 212.3)
- added R27: 49.9R, Library:R_0402_1005Metric, F.Cu at (-134.0, 568.7)
- added R28: 49.9R, Library:R_0402_1005Metric, F.Cu at (241.1, 475.3)
- added R29: 49.9R, Library:R_0402_1005Metric, F.Cu at (76.5, 158.5)
- added R32: 49.9R, Library:R_0402_1005Metric, F.Cu at (76.5, 162.5)
- added R50: 49.9R, Library:R_0402_1005Metric, F.Cu at (-134.0, 571.2)
- added R51: 49.9R, Library:R_0402_1005Metric, F.Cu at (-134.0, 573.7)
- added R52: 49.9R, Library:R_0402_1005Metric, F.Cu at (241.1, 477.8)
- added R53: 49.9R, Library:R_0402_1005Metric, F.Cu at (241.1, 480.4)
- added R54: 1K, Library:R_0603_1608Metric, F.Cu at (-115.0, 584.3)
- added TR1: HM2108NL, Library:HM2108NL, F.Cu at (43.7, 151.2)
- C1, C10, C103, C104, C105, C106, C107, C108, C109, C11, C110, C111, C112, C113, C114, C115, C116, C117, C119, C12, C129, C13, C130, C131, C132, C133, C134, C135, C136, C137, C138, C139, C14, C140, C15, C16, C17, C18, C19, C2, C20, C21, C22, C27, C28, C3, C31, C32, C33, C34, C35, C36, C37, C38, C39, C4, C41, C5, C51, C52, C53, C54, C55, C56, C57, C58, C59, C6, C60, C61, C62, C63, C64, C65, C67, C7, C77, C78, C79, C8, C80, C81, C82, C83, C84, C85, C86, C87, C88, C89, C9, C90, C91, C93: footprint Capacitor_SMD:C_0603_1608Metric -> Library:C_0603_1608Metric
- C23, C25: footprint Capacitor_SMD:C_0805_2012Metric -> Library:C_0805_2012Metric
- C29, C30: footprint Capacitor_SMD:C_0603_1608Metric -> Library:C_0402_1005Metric
- C40, C42, C43, C66: value 1uF/25V -> 4.7uF/16V; footprint Capacitor_SMD:C_0603_1608Metric -> Library:C_0603_1608Metric
- C44, C45, C70, C71, C96, C97: value 100pF/100V -> 10nF/100V; footprint Capacitor_SMD:C_0603_1608Metric -> Library:C_0402_1005Metric
- D10, D11, D12, D13, D14, D15, D16, D17, D18, D19, D20, D21, D26, D27, D28, D29, D30, D31, D32, D33, D34, D35, D36, D37, D42, D43, D44, D45, D46, D47, D48, D49, D50, D51, D52, D53, D58, D59, D60, D61, D62, D63, D64, D65, D66, D67, D68, D69: footprint Diode_SMD:D_SOD-323_HandSoldering -> Library:D_SOD-323_HandSoldering
- D22, D23, D38, D39, D54, D55, D6, D7: footprint Diode_SMD:D_SOD-123 -> Library:D_SOD-123
- D24, D40, D56, D8: footprint Diode_SMD:D_SOD-123F -> Library:D_SOD-123F
- D25, D4, D41, D57, D9: footprint LED_SMD:LED_0603_1608Metric -> Library:LED_0603_1608Metric
- D5, Q10, Q11, Q12, Q13, Q15, Q16, Q17, Q18, Q19, Q2, Q20, Q21, Q22, Q23, Q24, Q25, Q26, Q28, Q29, Q3, Q30, Q31, Q32, Q33, Q34, Q35, Q36, Q37, Q38, Q39, Q4, Q41, Q42, Q43, Q44, Q45, Q46, Q47, Q48, Q49, Q5, Q50, Q51, Q52, Q6, Q7, Q8, Q9: footprint Package_TO_SOT_SMD:SOT-23 -> Library:SOT-23
- F1, F10, F11, F12, F13, F14, F15, F16, F17, F18, F19, F2, F20, F21, F22, F23, F24, F25, F26, F27, F28, F29, F3, F30, F31, F32, F33, F34, F35, F36, F37, F38, F39, F4, F40, F41, F42, F43, F44, F45, F46, F47, F48, F49, F5, F50, F51, F52, F6, F7, F8, F9: footprint Fuse:Fuse_0805_2012Metric -> Library:Fuse_0805_2012Metric
- FB1, FB2, FB3, FB4, R10, R107, R108, R11, R110, R111, R113, R114, R116, R117, R119, R12, R120, R122, R123, R125, R126, R128, R129, R13, R131, R132, R134, R135, R137, R138, R14, R140, R141, R142, R143, R145, R146, R147, R15, R150, R158, R159, R16, R161, R162, R164, R165, R167, R168, R17, R170, R171, R173, R174, R176, R177, R179, R18, R180, R182, R183, R185, R186, R188, R189, R19, R191, R192, R193, R194, R196, R197, R198, R20, R201, R209, R21, R210, R212, R213, R215, R216, R218, R219, R22, R221, R222, R224, R225, R227, R228, R230, R231, R233, R234, R236, R237, R239, R240, R242, R243, R3, R30, R31, R33, R34, R39, R4, R40, R41, R43, R44, R45, R48, R5, R56, R57, R59, R6, R60, R62, R63, R65, R66, R68, R69, R7, R71, R72, R74, R75, R77, R78, R8, R80, R81, R83, R84, R86, R87, R89, R9, R90, R91, R92, R94, R95, R96, R99, TH1, TH11, TH16, TH6: footprint Resistor_SMD:R_0603_1608Metric -> Library:R_0603_1608Metric
- J1, J2, J3, J4: footprint MountingHole:MountingHole_3.2mm_M3_ISO7380_Pad -> Library:MountingHole_3.2mm_M3_ISO7380_Pad
- J10, J11, J12, J13, J14, J15, J16, J17: footprint Connector_JST:JST_XH_B7B-XH-A_1x07_P2.50mm_Vertical_BAT_6S -> Library:JST_XH_B7B-XH-A_1x07_P2.50mm_Vertical_BAT_6S
- J18, J7, J9: footprint Connector_JST:JST_VH_B2P-VH-B_1x02_P3.96mm_Vertical -> Library:JST_VH_B2P-VH-B_1x02_P3.96mm_Vertical
- J5, J8: footprint Connector_PinHeader_2.54mm:PinHeader_1x04_P2.54mm_Vertical -> Library:PinHeader_1x04_P2.54mm_Vertical
- J6: footprint Connector_Molex:Molex_Mini-Fit_Jr_5569-04A2_2x02_P4.20mm_Horizontal -> Library:Molex_Mini-Fit_Jr_5569-04A2_2x02_P4.20mm_Horizontal
- L1: footprint Inductor_SMD:L_Bourns_SRP5030T -> Library:L_Bourns_SRP5030T
- LOGO1, LOGO2: footprint Symbol:teTra-LOGO -> Library:teTra-LOGO
- Q1, Q14, Q27, Q40: footprint Package_TO_SOT_SMD:SOT-223 -> Library:SOT-223
- R100: value 100R -> 1K; footprint Resistor_SMD:R_0603_1608Metric -> Library:R_0603_1608Metric
- R106, R109, R112, R115, R118, R121, R124, R127, R130, R133, R136, R139, R157, R160, R163, R166, R169, R172, R175, R178, R181, R184, R187, R190, R208, R211, R214, R217, R220, R223, R226, R229, R232, R235, R238, R241, R55, R58, R61, R64, R67, R70, R73, R76, R79, R82, R85, R88: footprint Resistor_SMD:R_2512_6332Metric -> Library:R_2512_6332Metric
- R35, R47, R98: value 806R -> 1K; footprint Resistor_SMD:R_0603_1608Metric -> Library:R_0603_1608Metric
- R36, R37: value 51R -> 49.9R; footprint Resistor_SMD:R_0603_1608Metric -> Library:R_0402_1005Metric
- R38, R42, R93: value 1.2K -> 1K; footprint Resistor_SMD:R_0603_1608Metric -> Library:R_0603_1608Metric
- R46: value 100K -> 49.9R; footprint Resistor_SMD:R_0603_1608Metric -> Library:R_0402_1005Metric
- R49: value 100R -> 49.9R; footprint Resistor_SMD:R_0603_1608Metric -> Library:R_0402_1005Metric
- R97: value 100K -> 1K; footprint Resistor_SMD:R_0603_1608Metric -> Library:R_0603_1608Metric
- TH10, TH12, TH13, TH14, TH15, TH17, TH18, TH19, TH2, TH20, TH3, TH4, TH5, TH7, TH8, TH9: footprint Resistor_THT:R_Axial_DIN0204_L3.6mm_D1.6mm_P1.90mm_Vertical -> Library:R_Axial_DIN0204_L3.6mm_D1.6mm_P1.90mm_Vertical
- TP10, TP4, TP6, TP8: value TestPoint -> Vref2; footprint TestPoint:TestPoint_Pad_D1.0mm -> Library:TestPoint_Pad_D1.0mm
- TP2: footprint TestPoint:TestPoint_Pad_D1.0mm -> Library:TestPoint_Pad_D1.0mm
- TP3, TP5, TP7, TP9: value TestPoint -> Vreg; footprint TestPoint:TestPoint_Pad_D1.0mm -> Library:TestPoint_Pad_D1.0mm
- TR2: footprint Transformer_SMD:HM2108NL -> Library:HM2108NL
- TR3, TR4, TR5, TR6: value HM2102NL -> HM2108NL; footprint Transformer_SMD:HM2102NL_PUL -> Library:HM2108NL
- U10: footprint Package_SO:SOP-8_6.62x9.15mm_P2.54mm -> Library:SOP-8_6.62x9.15mm_P2.54mm
- U11, U12, U13, U14: footprint Package_SO:TSSOP-48_6.1x12.5mm_P0.5mm -> Library:TSSOP-48_6.1x12.5mm_P0.5mm
- U6: footprint Package_TO_SOT_SMD:SOT-23-6_Handsoldering -> Library:SOT-23-6_Handsoldering
- U8: footprint RF_Module:ESP32-DevKitc V4_DIP-38_27.9mm×48.2mm -> Library:ESP32-DevKitc V4_DIP-38_27.9mm×48.2mm
- U9: footprint Package_SO:MSOP-16_3x4mm_P0.5mm -> Library:MSOP-16_3x4mm_P0.5mm
- moved C43 489.7 mm to (-149.5, 629.8), turned to -90 degrees
- moved TH12 452.8 mm to (-167.4, 569.7)
- moved C109 369.1 mm to (-162.3, 576.2)
- moved R14 369.1 mm to (-154.1, 591.7)
- moved R176 369.1 mm to (-162.3, 578.7)
- moved R177 369.1 mm to (-162.3, 581.2)
- moved D48 369.1 mm to (-157.7, 576.4)
- moved Q34 369.1 mm to (-157.8, 580.3)
- moved R175 369.1 mm to (-160.0, 572.5)
- moved C103 351.5 mm to (-127.4, 604.7)
- moved C108 351.5 mm to (-127.4, 590.3)
- moved C11 351.5 mm to (-173.7, 571.1)
- moved C110 351.5 mm to (-149.6, 590.3)
- moved C111 351.5 mm to (-138.5, 604.7)
- moved C112 351.5 mm to (-149.6, 604.7)
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Connections:
- net /Slaves/LTC6811_4/MA renamed Net-(J9-Pin_1)
- net /Slaves/LTC6811_4/PA renamed Net-(J9-Pin_2)
- C42 pad 1: /Slaves/LTC6811_1/Vreg -> /Slaves/LTC6811_2/Vreg
- C43 pad 1: /Slaves/LTC6811_1/Vreg -> /Slaves/LTC6811_3/Vreg
- C66 pad 1: /Slaves/LTC6811_2/Vreg -> /Slaves/LTC6811_4/Vreg
- J7 pad 1: /Slaves/LTC6811_1/PB -> Net-(J7-Pin_1)
- J7 pad 2: /Slaves/LTC6811_1/MB -> Net-(J7-Pin_2)
- R100 pad 1: /Slaves/LTC6811_2/IPA -> Net-(U13-ICMP)
- R100 pad 2: /Slaves/LTC6811_2/IMA -> GND_PACK
- R35 pad 1: Net-(U9-ICMP) -> GND
- R35 pad 2: GND -> Net-(U9-ICMP)
- R38 pad 1: Net-(U9-IBIAS) -> Net-(U9-ICMP)
- R38 pad 2: Net-(U9-ICMP) -> Net-(U9-IBIAS)
- R46 pad 1: /Slaves/LTC6811_1/IMB -> Net-(C70-Pad1)
- R46 pad 2: /Slaves/LTC6811_1/IPB -> /Slaves/LTC6811_2/IPA
- R47 pad 1: Net-(U11-ICMP) -> Net-(U12-IBIAS)
- R47 pad 2: GND_PACK -> Net-(U12-ICMP)
- R49 pad 1: /Slaves/LTC6811_1/IPA -> /Slaves/LTC6811_2/IMA
- R49 pad 2: /Slaves/LTC6811_1/IMA -> Net-(C70-Pad1)
- R93 pad 1: Net-(U12-IBIAS) -> Net-(U14-IBIAS)
- R93 pad 2: Net-(U12-ICMP) -> Net-(U14-ICMP)
- R97 pad 1: /Slaves/LTC6811_2/IMB -> Net-(U11-ICMP)
- R97 pad 2: /Slaves/LTC6811_2/IPB -> GND_PACK
- TH12 pad 1: /Slaves/LTC6811_1/T3 -> /Slaves/LTC6811_3/T2
- TH13 pad 1: /Slaves/LTC6811_2/T3 -> /Slaves/LTC6811_3/T3
- TH17 pad 1: /Slaves/LTC6811_3/T3 -> /Slaves/LTC6811_4/T2
- TH3 pad 1: /Slaves/LTC6811_2/T2 -> /Slaves/LTC6811_1/T3
- TH7 pad 1: /Slaves/LTC6811_3/T2 -> /Slaves/LTC6811_2/T2
- TH8 pad 1: /Slaves/LTC6811_4/T2 -> /Slaves/LTC6811_2/T3
- TR3 pad 1: /Slaves/LTC6811_1/MA -> /Slaves/LTC6811_2/IPB
- TR3 pad 2: unconnected-(TR3-Pad2) -> Net-(C45-Pad1)
- TR3 pad 3: /Slaves/LTC6811_1/PA -> /Slaves/LTC6811_2/IMB
- TR3 pad 4: /Slaves/LTC6811_1/MB -> /Slaves/LTC6811_1/IMA
- TR3 pad 5: unconnected-(TR3-Pad5) -> Net-(C26-Pad1)
- TR3 pad 6: /Slaves/LTC6811_1/PB -> /Slaves/LTC6811_1/IPA
- TR4 pad 1: /Slaves/LTC6811_2/MA -> /Slaves/LTC6811_3/IPB
- TR4 pad 2: unconnected-(TR4-Pad2) -> Net-(C49-Pad1)
- TR4 pad 3: /Slaves/LTC6811_2/PA -> /Slaves/LTC6811_3/IMB
- TR4 pad 4: /Slaves/LTC6811_1/MA -> /Slaves/LTC6811_2/IMA
- TR4 pad 5: unconnected-(TR4-Pad5) -> Net-(C47-Pad1)
- TR4 pad 6: /Slaves/LTC6811_1/PA -> /Slaves/LTC6811_2/IPA
- TR5 pad 1: /Slaves/LTC6811_3/MA -> /Slaves/LTC6811_4/IPB
- TR5 pad 2: unconnected-(TR5-Pad2) -> Net-(C76-Pad1)
- TR5 pad 3: /Slaves/LTC6811_3/PA -> /Slaves/LTC6811_4/IMB
- TR5 pad 4: /Slaves/LTC6811_2/MA -> /Slaves/LTC6811_3/IMA
- TR5 pad 5: unconnected-(TR5-Pad5) -> Net-(C75-Pad1)
- TR5 pad 6: /Slaves/LTC6811_2/PA -> /Slaves/LTC6811_3/IPA
- TR6 pad 2: unconnected-(TR6-Pad2) -> Net-(C97-Pad1)
- TR6 pad 4: /Slaves/LTC6811_3/MA -> /Slaves/LTC6811_4/IMA
- TR6 pad 5: unconnected-(TR6-Pad5) -> Net-(C96-Pad1)
- TR6 pad 6: /Slaves/LTC6811_3/PA -> /Slaves/LTC6811_4/IPA
Routing:
- net /Slaves/LTC6811_1/T1: track 0.00 -> 98.7 mm
- net /Slaves/LTC6811_1/Vreg: track 0.00 -> 37.3 mm, vias 0 -> 2
- net /Slaves/LTC6811_1/cell1/S: track 0.00 -> 35.7 mm
- net /Slaves/LTC6811_1/Vref2: track 0.00 -> 33.0 mm
- net /Slaves/LTC6811_1/cell1/C: track 0.00 -> 28.2 mm
- net /Slaves/LTC6811_1/cell12/C: track 0.00 -> 26.6 mm
- net /Slaves/LTC6811_1/cell12/S: track 0.00 -> 25.9 mm
- net /Slaves/LTC6811_1/cell11/C: track 0.00 -> 25.5 mm
- net /Slaves/LTC6811_1/cell2/S: track 0.00 -> 25.5 mm
- net /Slaves/LTC6811_1/cell2/C: track 0.00 -> 24.6 mm
- net /Slaves/LTC6811_1/T5: track 0.00 -> 23.6 mm
- net /Slaves/LTC6811_1/DRIVE: track 0.00 -> 23.4 mm, vias 0 -> 2
- net /Slaves/LTC6811_1/cell11/S: track 0.00 -> 22.4 mm
- net /Slaves/LTC6811_1/T4: track 0.00 -> 22.3 mm
- net /Slaves/LTC6811_1/BAT+: track 0.00 -> 22.2 mm
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Other:
- board size 360 x 55 mm -> 360 x 50 mm

Commit message: Add files via upload
Parts:
- C1, C10, C103, C104, C105, C106, C107, C108, C109, C11, C110, C111, C112, C113, C114, C115, C116, C117, C119, C12, C129, C13, C130, C131, C132, C133, C134, C135, C136, C137, C138, C139, C14, C140, C15, C16, C17, C18, C19, C2, C20, C21, C22, C27, C28, C3, C31, C32, C33, C34, C35, C36, C37, C38, C39, C4, C40, C41, C42, C43, C5, C51, C52, C53, C54, C55, C56, C57, C58, C59, C6, C60, C61, C62, C63, C64, C65, C66, C67, C7, C77, C78, C79, C8, C80, C81, C82, C83, C84, C85, C86, C87, C88, C89, C9, C90, C91, C93: footprint Library:C_0603_1608Metric -> Capacitor_SMD:C_0603_1608Metric
- C23, C25: footprint Library:C_0805_2012Metric -> Capacitor_SMD:C_0805_2012Metric
- C24, C26, C29, C30, C44, C45, C46, C47, C48, C49, C50, C70, C71, C72, C73, C74, C75, C76, C96, C97: footprint Library:C_0402_1005Metric -> Capacitor_SMD:C_0603_1608Metric
- D10, D11, D12, D13, D14, D15, D16, D17, D18, D19, D20, D21, D26, D27, D28, D29, D30, D31, D32, D33, D34, D35, D36, D37, D42, D43, D44, D45, D46, D47, D48, D49, D50, D51, D52, D53, D58, D59, D60, D61, D62, D63, D64, D65, D66, D67, D68, D69: footprint Library:D_SOD-323_HandSoldering -> Diode_SMD:D_SOD-323_HandSoldering
- D22, D23, D38, D39, D54, D55, D6, D7: footprint Library:D_SOD-123 -> Diode_SMD:D_SOD-123
- D24, D40, D56, D8: footprint Library:D_SOD-123F -> Diode_SMD:D_SOD-123F
- D25, D4, D41, D57, D9: footprint Library:LED_0603_1608Metric -> LED_SMD:LED_0603_1608Metric
- D5, Q10, Q11, Q12, Q13, Q15, Q16, Q17, Q18, Q19, Q2, Q20, Q21, Q22, Q23, Q24, Q25, Q26, Q28, Q29, Q3, Q30, Q31, Q32, Q33, Q34, Q35, Q36, Q37, Q38, Q39, Q4, Q41, Q42, Q43, Q44, Q45, Q46, Q47, Q48, Q49, Q5, Q50, Q51, Q52, Q6, Q7, Q8, Q9: footprint Library:SOT-23 -> Package_TO_SOT_SMD:SOT-23
- F1, F10, F11, F12, F13, F14, F15, F16, F17, F18, F19, F2, F20, F21, F22, F23, F24, F25, F26, F27, F28, F29, F3, F30, F31, F32, F33, F34, F35, F36, F37, F38, F39, F4, F40, F41, F42, F43, F44, F45, F46, F47, F48, F49, F5, F50, F51, F52, F6, F7, F8, F9: footprint Library:Fuse_0805_2012Metric -> Fuse:Fuse_0805_2012Metric
- FB1, FB2, FB3, FB4, R10, R100, R101, R107, R108, R11, R110, R111, R113, R114, R116, R117, R119, R12, R120, R122, R123, R125, R126, R128, R129, R13, R131, R132, R134, R135, R137, R138, R14, R140, R141, R142, R143, R145, R146, R147, R15, R150, R158, R159, R16, R161, R162, R164, R165, R167, R168, R17, R170, R171, R173, R174, R176, R177, R179, R18, R180, R182, R183, R185, R186, R188, R189, R19, R191, R192, R193, R194, R196, R197, R198, R20, R201, R209, R21, R210, R212, R213, R215, R216, R218, R219, R22, R221, R222, R224, R225, R227, R228, R230, R231, R233, R234, R236, R237, R239, R240, R242, R243, R3, R30, R31, R33, R34, R35, R38, R39, R4, R40, R41, R42, R43, R44, R45, R47, R48, R5, R54, R56, R57, R59, R6, R60, R62, R63, R65, R66, R68, R69, R7, R71, R72, R74, R75, R77, R78, R8, R80, R81, R83, R84, R86, R87, R89, R9, R90, R91, R92, R93, R94, R95, R96, R97, R98, R99, TH1, TH11, TH16, TH6: footprint Library:R_0603_1608Metric -> Resistor_SMD:R_0603_1608Metric
- J1, J2, J3, J4: footprint Library:MountingHole_3.2mm_M3_ISO7380_Pad -> MountingHole:MountingHole_3.2mm_M3_ISO7380_Pad
- J10, J11, J12, J13, J14, J15, J16, J17: footprint Library:JST_XH_B7B-XH-A_1x07_P2.50mm_Vertical_BAT_6S -> Connector_JST:JST_XH_B7B-XH-A_1x07_P2.50mm_Vertical_BAT_6S
- J18, J7, J9: footprint Library:JST_VH_B2P-VH-B_1x02_P3.96mm_Vertical -> Connector_JST:JST_VH_B2P-VH-B_1x02_P3.96mm_Vertical
- J5, J8: footprint Library:PinHeader_1x04_P2.54mm_Vertical -> Connector_PinHeader_2.54mm:PinHeader_1x04_P2.54mm_Vertical
- J6: footprint Library:Molex_Mini-Fit_Jr_5569-04A2_2x02_P4.20mm_Horizontal -> Connector_Molex:Molex_Mini-Fit_Jr_5569-04A2_2x02_P4.20mm_Horizontal
- L1: footprint Library:L_Bourns_SRP5030T -> Inductor_SMD:L_Bourns_SRP5030T
- LOGO1, LOGO2: footprint Library:teTra-LOGO -> Symbol:teTra-LOGO
- Q1, Q14, Q27, Q40: footprint Library:SOT-223 -> Package_TO_SOT_SMD:SOT-223
- R1, R2, R23, R24, R25, R26, R27, R28, R29, R32, R36, R37, R46, R49, R50, R51, R52, R53: footprint Library:R_0402_1005Metric -> Resistor_SMD:R_0603_1608Metric
- R106, R109, R112, R115, R118, R121, R124, R127, R130, R133, R136, R139, R157, R160, R163, R166, R169, R172, R175, R178, R181, R184, R187, R190, R208, R211, R214, R217, R220, R223, R226, R229, R232, R235, R238, R241, R55, R58, R61, R64, R67, R70, R73, R76, R79, R82, R85, R88: footprint Library:R_2512_6332Metric -> Resistor_SMD:R_2512_6332Metric
- TH10, TH12, TH13, TH14, TH15, TH17, TH18, TH19, TH2, TH20, TH3, TH4, TH5, TH7, TH8, TH9: footprint Library:R_Axial_DIN0204_L3.6mm_D1.6mm_P1.90mm_Vertical -> Resistor_THT:R_Axial_DIN0204_L3.6mm_D1.6mm_P1.90mm_Vertical
- TP10, TP2, TP3, TP4, TP5, TP6, TP7, TP8, TP9: footprint Library:TestPoint_Pad_D1.0mm -> TestPoint:TestPoint_Pad_D1.0mm
- TR1, TR2, TR3, TR4, TR5, TR6: footprint Library:HM2108NL -> Transformer_SMD:HM2108NL
- U10: footprint Library:SOP-8_6.62x9.15mm_P2.54mm -> Package_SO:SOP-8_6.62x9.15mm_P2.54mm
- U11, U12, U13, U14: footprint Library:TSSOP-48_6.1x12.5mm_P0.5mm -> Package_SO:TSSOP-48_6.1x12.5mm_P0.5mm
- U6: footprint Library:SOT-23-6_Handsoldering -> Package_TO_SOT_SMD:SOT-23-6_Handsoldering
- U8: footprint Library:ESP32-DevKitc V4_DIP-38_27.9mm×48.2mm -> RF_Module:ESP32-DevKitc V4_DIP-38_27.9mm×48.2mm
- U9: footprint Library:MSOP-16_3x4mm_P0.5mm -> Package_SO:MSOP-16_3x4mm_P0.5mm
- moved C11 652.6 mm to (210.3, 43.4)
- moved C12 652.6 mm to (239.4, 41.0)
- moved C13 652.6 mm to (239.4, 43.5)
- moved C14 652.6 mm to (239.4, 46.0)
- moved C15 652.6 mm to (239.4, 48.5)
- moved C93 652.6 mm to (191.2, 75.4)
- moved D40 652.6 mm to (201.8, 92.5)
- moved FB3 652.6 mm to (195.2, 80.4)
- moved R100 652.6 mm to (268.9, 59.1)
- moved R13 652.6 mm to (210.3, 45.9)
- moved R14 652.6 mm to (229.9, 64.0)
- moved R142 652.6 mm to (195.2, 82.9)
- moved R145 652.6 mm to (228.9, 101.3)
- moved R146 652.6 mm to (228.9, 103.8)
- moved R147 652.6 mm to (228.9, 106.3)
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Connections:
- TR1 pad 1: /Slaves/LTC6811_1/IMB -> /Slaves/LTC6811_1/IPA
- TR1 pad 3: /Slaves/LTC6811_1/IPB -> /Slaves/LTC6811_1/IMA
- TR1 pad 4: Net-(J7-Pin_1) -> Net-(J7-Pin_2)
- TR1 pad 6: Net-(J7-Pin_2) -> Net-(J7-Pin_1)
- TR3 pad 1: /Slaves/LTC6811_2/IPB -> /Slaves/LTC6811_2/IPA
- TR3 pad 3: /Slaves/LTC6811_2/IMB -> /Slaves/LTC6811_2/IMA
- TR3 pad 4: /Slaves/LTC6811_1/IMA -> /Slaves/LTC6811_1/IMB
- TR3 pad 6: /Slaves/LTC6811_1/IPA -> /Slaves/LTC6811_1/IPB
- TR4 pad 1: /Slaves/LTC6811_3/IPB -> /Slaves/LTC6811_3/IPA
- TR4 pad 3: /Slaves/LTC6811_3/IMB -> /Slaves/LTC6811_3/IMA
- TR4 pad 4: /Slaves/LTC6811_2/IMA -> /Slaves/LTC6811_2/IMB
- TR4 pad 6: /Slaves/LTC6811_2/IPA -> /Slaves/LTC6811_2/IPB
- TR5 pad 1: /Slaves/LTC6811_4/IPB -> /Slaves/LTC6811_4/IPA
- TR5 pad 3: /Slaves/LTC6811_4/IMB -> /Slaves/LTC6811_4/IMA
- TR5 pad 4: /Slaves/LTC6811_3/IMA -> /Slaves/LTC6811_3/IMB
- TR5 pad 6: /Slaves/LTC6811_3/IPA -> /Slaves/LTC6811_3/IPB
- TR6 pad 4: /Slaves/LTC6811_4/IMA -> /Slaves/LTC6811_4/IMB
- TR6 pad 6: /Slaves/LTC6811_4/IPA -> /Slaves/LTC6811_4/IPB
Routing:
- net /Slaves/LTC6811_1/T1: track 98.7 -> 34.7 mm
- net /Slaves/LTC6811_1/cell1/S: track 35.7 -> 60.2 mm
- net /Slaves/LTC6811_1/Vreg: track 37.3 -> 19.4 mm
- net Net-(J7-Pin_2): track 14.6 -> 0.00 mm
- net /Slaves/LTC6811_1/T2: track 21.5 -> 35.1 mm
- net /Slaves/LTC6811_1/Vref2: track 33.0 -> 44.4 mm
- net /Slaves/LTC6811_1/T5: track 23.6 -> 33.2 mm
- net /Slaves/LTC6811_1/BAT+: track 22.2 -> 13.0 mm
- net Net-(U11-Vref1): track 5.88 -> 14.1 mm
- net Net-(U11-WDT): track 5.25 -> 13.2 mm
- net Net-(U11-DTEN): track 5.44 -> 13.1 mm
- net Net-(J7-Pin_1): track 7.57 -> 0.00 mm
- net /Slaves/LTC6811_1/IMB: track 18.5 -> 25.5 mm
- net Net-(C41-Pad1): track 11.0 -> 4.69 mm
- net Net-(U11-ISOMD): track 5.63 -> 10.3 mm
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
Commit message: Add files via upload
Parts:
- C74: value 10nF/100V -> 10nF/100V NC
- moved C20 504.1 mm to (42.4, 176.7)
- moved C21 504.1 mm to (42.4, 179.2)
- moved C23 504.1 mm to (46.6, 190.5)
- moved C25 504.1 mm to (46.6, 193.5)
- moved D4 504.1 mm to (56.7, 196.9)
- moved L1 504.1 mm to (52.9, 189.7)
- moved R30 504.1 mm to (42.4, 186.7)
- moved R31 504.1 mm to (42.4, 189.2)
- moved R33 504.1 mm to (42.4, 194.3)
- moved TP2 504.1 mm to (61.4, 180.0)
- moved U6 504.1 mm to (51.8, 195.5)
- moved C33 489.2 mm to (37.7, 134.0)
- moved C34 489.2 mm to (37.7, 136.5)
- moved C35 489.2 mm to (37.7, 139.0)
- moved C36 489.2 mm to (37.7, 141.5)
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Routing:
- net /Slaves/LTC6811_1/T1: track 34.7 -> 97.4 mm
- net /Slaves/LTC6811_2/cell1/C: track 0.00 -> 26.3 mm
- net /Slaves/LTC6811_1/cell1/S: track 60.2 -> 35.2 mm, vias 0 -> 2
- net /Slaves/LTC6811_2/cell2/S: track 0.00 -> 24.2 mm
- net /Slaves/LTC6811_2/cell3/S: track 0.00 -> 21.3 mm
- net /Slaves/LTC6811_2/cell4/S: track 0.00 -> 18.2 mm
- net /Slaves/LTC6811_2/cell2/C: track 0.00 -> 17.9 mm
- net /Slaves/LTC6811_2/cell4/C: track 0.00 -> 16.7 mm
- net /Slaves/LTC6811_1/C6: track 0.00 -> 15.2 mm
- net /Slaves/LTC6811_2/cell5/S: track 0.00 -> 14.8 mm
- net /Slaves/LTC6811_2/cell3/C: track 0.00 -> 14.8 mm
- net /Slaves/LTC6811_2/cell5/C: track 0.00 -> 13.6 mm
- net /Slaves/LTC6811_1/cell12/C+: track 3.62 -> 15.7 mm
- net /Slaves/LTC6811_2/cell6/C: track 0.00 -> 12.0 mm
- net /Slaves/LTC6811_1/BAT+: track 13.0 -> 24.7 mm
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Other:
- board size 360 x 50 mm -> 320 x 55 mm
