File: LTC6811_ESP32_V2/PowerSupply.kicad_sch (KiCad schematic)
At the start: 12 parts, among them J6 Molex 5569, U6 LMR51420XDDCR

Commit message: Add files via upload
Parts:
- C20, C21, C? (x2): symbol Device:C -> Library:C
- D4: symbol Device:LED -> Library:LED
- J6: symbol Connector_Generic:Conn_01x04 -> Library:Conn_01x04
- L1: symbol Device:L -> Library:L
- R30, R33, R?: symbol Device:R_Small -> Library:R_Small
- TP2: symbol Connector:TestPoint -> Library:TestPoint
- U6: symbol Regulator_Switching:LMR51420 -> Library:LMR51420
Changed lines of the file:
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@@
 	)
 	(symbol
-		(lib_id "Device:L")
+		(lib_id "Library:L")
 		(at 193.04 106.68 90)
 		(unit 1)
@@
 	)
 	(symbol
-		(lib_id "power:GND")
+		(lib_id "Library:GND")
 		(at 208.915 116.84 0)
 		(unit 1)
@@
 	)
 	(symbol
-		(lib_id "power:GND")
+		(lib_id "Library:GND")
 		(at 143.51 111.76 0)
 		(unit 1)
@@
 	)
 	(symbol
-		(lib_id "Connector:TestPoint")
+		(lib_id "Library:TestPoint")
 		(at 237.49 154.305 270)
 		(unit 1)
@@
 	)
 	(symbol
-		(lib_id "power:GND")
+		(lib_id "Library:GND")
 		(at 238.76 122.555 0)
 		(unit 1)
@@
 	)
 	(symbol
-		(lib_id "Device:C")
+		(lib_id "Library:C")
 		(at 220.345 109.22 0)
 		(unit 1)
@@
 	)
 	(symbol
-		(lib_id "Device:LED")
+		(lib_id "Library:LED")
 		(at 238.76 116.205 270)
 		(unit 1)
@@
 	)
 	(symbol
-		(lib_id "Device:R_Small")
+		(lib_id "Library:R_Small")
 		(at 199.39 114.3 0)
 		(unit 1)
@@
 	)
 	(symbol
-		(lib_id "power:+3V3")
+		(lib_id "Library:+3V3")
 		(at 220.345 106.68 0)
 		(mirror y)
@@
 	)
 	(symbol
-		(lib_id "Connector_Generic:Conn_01x04")
+		(lib_id "Library:Conn_01x04")
 		(at 129.54 104.14 180)
 		(unit 1)
@@
 	)
 	(symbol
-		(lib_id "Device:C")
+		(lib_id "Library:C")
 		(at 150.495 106.68 0)
 		(unit 1)
@@
 	)
 	(symbol
-		(lib_id "Device:C")
+		(lib_id "Library:C")
 		(at 208.915 109.22 0)
 		(unit 1)
@@
 	)
 	(symbol
-		(lib_id "power:+3V3")
+		(lib_id "Library:+3V3")
 		(at 238.76 106.045 0)
 		(mirror y)
@@
 	)
 	(symbol
-		(lib_id "Device:R_Small")
+		(lib_id "Library:R_Small")
 		(at 238.76 109.22 180)
 		(unit 1)
@@
 	)
 	(symbol
-		(lib_id "Device:C")
+		(lib_id "Library:C")
 		(at 182.245 103.505 180)
 		(unit 1)
@@
 	)
 	(symbol
-		(lib_id "Device:R_Small")
+		(lib_id "Library:R_Small")
 		(at 199.39 109.22 180)
 		(unit 1)
@@
 	)
 	(symbol
-		(lib_id "Regulator_Switching:LMR51420")
+		(lib_id "Library:LMR51420")
 		(at 165.1 106.68 0)
 		(unit 1)

Commit message: Add files via upload
Parts:
- TP2: value TestPoint -> 3V3
Changed lines of the file:
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@@
 			)
 		)
-		(property "Value" "TestPoint"
+		(property "Value" "3V3"
 			(at 242.57 154.305 90)
 			(effects
@@
 				)
 				(justify left)
+				(hide yes)
 			)
 		)
