File: LTC6811_ESP32_V2/LTC6811.kicad_sch (KiCad schematic)
At the start: 59 parts, among them J16 B7B-XH-A, J17 B7B-XH-A, Q40 NSV1C201MZ4, U14 LTC6811HG-1

Commit message: Add files via upload
Parts:
- removed C118, C120, C121: 1uF/25V, Capacitor_SMD:C_0603_1608Metric, symbol Device:C
- removed C122, C123: 100pF/100V, Capacitor_SMD:C_0603_1608Metric, symbol Device:C
- removed R195: 1.2K, Resistor_SMD:R_0603_1608Metric, symbol Device:R_Small
- removed R199: 100K, Resistor_SMD:R_0603_1608Metric, symbol Device:R_Small
- removed R200: 806R, Resistor_SMD:R_0603_1608Metric, symbol Device:R_Small
- removed R202: 100R, Resistor_SMD:R_0603_1608Metric, symbol Device:R_Small
- removed TR6: HM2102NL, Transformer_SMD:HM2102NL_PUL, symbol Transformer:HM2102NL
- added C48, C72: 10nF/100V, Capacitor_SMD:C_0402_1005Metric, symbol Library:C
- added C66: 4.7uF/16V, Capacitor_SMD:C_0603_1608Metric, symbol Library:C
- added R101, R93: 1K, Resistor_SMD:R_0603_1608Metric, symbol Library:R_Small
- added R24, R28, R52, R53: 49.9R, Resistor_SMD:R_0402_1005Metric, symbol Library:R_Small
- C115, C116, C117, C119: symbol Device:C -> Library:C
- C16: renamed from C1; symbol Device:C -> Library:C
- C17: renamed from C2; symbol LTC6811-rescue:C-Device -> Library:C-Device
- C18: renamed from C3; symbol LTC6811-rescue:C-Device -> Library:C-Device
- C19: renamed from C4; symbol LTC6811-rescue:C-Device -> Library:C-Device
- C22: renamed from C5; symbol LTC6811-rescue:C-Device -> Library:C-Device
- D54, D55: symbol Diode:1N4148W -> Library:1N4148W
- D56: symbol Diode:BZT52Bxx -> Library:BZT52Bxx
- D57: symbol Device:LED -> Library:LED
- F40, F41, F42, F43, F44, F45, F46, F47, F48, F49, F50, F51, F52: symbol Device:Fuse -> Library:Fuse
- FB4: symbol LTC6811-rescue:Ferrite_Bead-Device -> Library:Ferrite_Bead-Device
- J16, J17: symbol Connector_Generic:Conn_01x07_BAT_6S -> Library:Conn_01x07_BAT_6S
- Q40: symbol Device:Q_NPN_BCEC -> Library:Q_NPN_BCEC
- R18: renamed from R3; symbol Device:R_Small -> Library:R_Small
- R19: renamed from R4; symbol Device:R -> Library:R
- R193, R194, R196, R197, R198, R201: symbol Device:R_Small -> Library:R_Small
- R20: renamed from R5; symbol Device:R -> Library:R
- R21: renamed from R6; symbol Device:R -> Library:R
- R22: renamed from R7; symbol Device:R -> Library:R
- TH16: renamed from TH1; symbol Device:Thermistor -> Library:Thermistor
- TH17: renamed from TH2; symbol Device:Thermistor -> Library:Thermistor
- TH18: renamed from TH12; symbol Device:Thermistor -> Library:Thermistor
- TH19: renamed from TH4; symbol Device:Thermistor -> Library:Thermistor
- TH20: renamed from TH5; symbol Device:Thermistor -> Library:Thermistor
- TP10: value TestPoint -> Vref2; symbol Connector:TestPoint -> Library:TestPoint
- TP9: value TestPoint -> Vreg; symbol Connector:TestPoint -> Library:TestPoint
- U14: symbol ENNOID:LTC6811-1 -> Library:LTC6811-1
Connections:
- net GND_PACK: now also C48.2, C66.2, C72.2, R101.2
- net IMA: now also R53.1
- net IMB: now also R28.1
- net IPA: now also R52.2
- net IPB: now also R24.2
- net Vreg: now also C66.1
- net at U14.45 (IBIAS): now also R93.1
- net at U14.46 (ICMP): now also R101.1, R93.2
- new net: C72.1, R52.1, R53.2
- new net: C48.1, R24.1, R28.2
- no-connect marks 4 -> 2
Other:
- note removed: "12V"

Commit message: Add files via upload
Parts:
- C48, C72: footprint Capacitor_SMD:C_0402_1005Metric -> Capacitor_SMD:C_0603_1608Metric; Link https://www.digikey.jp/en/products/detail/kemet/C0402C103K1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 -> https://www.digikey.jp/en/products/detail/kemet/C0603X103K1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; MPN C0402C103K1RACAUTO -> C0603X103K1RAC3316
- R24, R28, R52, R53: footprint Resistor_SMD:R_0402_1005Metric -> Resistor_SMD:R_0603_1608Metric; Link https://www.digikey.jp/en/products/detail/yageo/RC0402FR-07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 -> https://www.digikey.jp/en/products/detail/panasonic-electro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; MPN RC0402FR-0749R9L -> ERJ-3EKF49R9V
Changed lines of the file:
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@@
 			)
 		)
-		(property "Footprint" "Capacitor_SMD:C_0402_1005Metric"
+		(property "Footprint" "Capacitor_SMD:C_0603_1608Metric"
 			(at 242.2652 133.35 0)
 			(effects
@@
 			)
 		)
-		(property "Datasheet" "https://content.kemet.com/datasheets/KEM_C1023_X7R_AUTO_SMD.pdf"
+		(property "Datasheet" "https://content.kemet.com/datasheets/KEM_X7R_FT_VW_AUDI.pdf"
 			(at 241.3 129.54 0)
 			(effects
@@
 			)
 		)
-		(property "Description" "10000 pF ±10% 100V Ceramic Capacitor X7R 0402 (1005 Metric)"
+		(property "Description" "10000 pF ±10% 100V Ceramic Capacitor X7R 0603 (1608 Metric)"
 			(at 241.3 129.54 0)
 			(effects
@@
 			)
 		)
-		(property "MPN" "C0402C103K1RACAUTO"
+		(property "MPN" "C0603X103K1RAC3316"
 			(at 241.3 129.54 0)
 			(effects
@@
 			)
 		)
-		(property "Link" "https://www.digikey.jp/en/products/detail/kemet/C0402C103K1RACAUTO/19200876"
+		(property "Link" "https://www.digikey.jp/en/products/detail/kemet/C0603X103K1RAC3316/10315782"
 			(at 241.3 129.54 0)
 			(effects
@@
 			)
 		)
-		(property "Footprint" "Capacitor_SMD:C_0402_1005Metric"
+		(property "Footprint" "Capacitor_SMD:C_0603_1608Metric"
 			(at 242.2652 119.38 0)
 			(effects
@@
 			)
 		)
-		(property "Datasheet" "https://content.kemet.com/datasheets/KEM_C1023_X7R_AUTO_SMD.pdf"
+		(property "Datasheet" "https://content.kemet.com/datasheets/KEM_X7R_FT_VW_AUDI.pdf"
 			(at 241.3 115.57 0)
 			(effects
@@
 			)
 		)
-		(property "Description" "10000 pF ±10% 100V Ceramic Capacitor X7R 0402 (1005 Metric)"
+		(property "Description" "10000 pF ±10% 100V Ceramic Capacitor X7R 0603 (1608 Metric)"
 			(at 241.3 115.57 0)
 			(effects
@@
 			)
 		)
-		(property "MPN" "C0402C103K1RACAUTO"
+		(property "MPN" "C0603X103K1RAC3316"
 			(at 241.3 115.57 0)
 			(effects
@@
 			)
 		)
-		(property "Link" "https://www.digikey.jp/en/products/detail/kemet/C0402C103K1RACAUTO/19200876"
+		(property "Link" "https://www.digikey.jp/en/products/detail/kemet/C0603X103K1RAC3316/10315782"
 			(at 241.3 115.57 0)
 			(effects
@@
 			)
 		)
-		(property "Footprint" "Resistor_SMD:R_0402_1005Metric"
+		(property "Footprint" "Resistor_SMD:R_0603_1608Metric"
 			(at 227.33 130.81 0)
 			(effects
@@
 			)
 		)
-		(property "Datasheet" "https://www.yageo.com/upload/media/product/products/datasheet/rchip/PYu-RC_Group_51_RoHS_L_12.pdf"
+		(property "Datasheet" "https://industrial.panasonic.com/cdbs/www-data/pdf/RDA0000/AOA0000C304.pdf"
 			(at 227.33 130.81 0)
 			(effects
@@
 			)
 		)
-		(property "Description" "49.9 Ohms ±1% 0.063W, 1/16W Chip Resistor 0402 (1005 Metric) Moisture Resistant Thick Film"
+		(property "Description" "49.9 Ohms ±1% 0.1W, 1/10W Chip Resistor 0603 (1608 Metric) Automotive AEC-Q200 Thick Film"
 			(at 227.33 130.81 0)
 			(effects
@@
 			)
 		)
-		(property "Link" "https://www.digikey.jp/en/products/detail/yageo/RC0402FR-0749R9L/726621"
+		(property "Link" "https://www.digikey.jp/en/products/detail/panasonic-electronic-components/ERJ-3EKF49R9V/196378"
 			(at 227.33 130.81 0)
 			(effects
@@
 			)
 		)
-		(property "MPN" "RC0402FR-0749R9L"
+		(property "MPN" "ERJ-3EKF49R9V"
 			(at 227.33 130.81 0)
 			(effects
@@
 			)
 		)
-		(property "Footprint" "Resistor_SMD:R_0402_1005Metric"
+		(property "Footprint" "Resistor_SMD:R_0603_1608Metric"
 			(at 228.6 114.3 0)
 			(effects
@@
 			)
 		)
-		(property "Datasheet" "https://www.yageo.com/upload/media/product/products/datasheet/rchip/PYu-RC_Group_51_RoHS_L_12.pdf"
+		(property "Datasheet" "https://industrial.panasonic.com/cdbs/www-data/pdf/RDA0000/AOA0000C304.pdf"
 			(at 228.6 114.3 0)
 			(effects
@@
 			)
 		)
-		(property "Description" "49.9 Ohms ±1% 0.063W, 1/16W Chip Resistor 0402 (1005 Metric) Moisture Resistant Thick Film"
+		(property "Description" "49.9 Ohms ±1% 0.1W, 1/10W Chip Resistor 0603 (1608 Metric) Automotive AEC-Q200 Thick Film"
 			(at 228.6 114.3 0)
 			(effects
@@
 			)
 		)
-		(property "Link" "https://www.digikey.jp/en/products/detail/yageo/RC0402FR-0749R9L/726621"
+		(property "Link" "https://www.digikey.jp/en/products/detail/panasonic-electronic-components/ERJ-3EKF49R9V/196378"
 			(at 228.6 114.3 0)
 			(effects
@@
 			)
 		)
-		(property "MPN" "RC0402FR-0749R9L"
+		(property "MPN" "ERJ-3EKF49R9V"
 			(at 228.6 114.3 0)
 			(effects
@@
 			)
 		)
-		(property "Footprint" "Resistor_SMD:R_0402_1005Metric"
+		(property "Footprint" "Resistor_SMD:R_0603_1608Metric"
 			(at 227.33 125.73 0)
 			(effects
@@
 			)
 		)
-		(property "Datasheet" "https://www.yageo.com/upload/media/product/products/datasheet/rchip/PYu-RC_Group_51_RoHS_L_12.pdf"
+		(property "Datasheet" "https://industrial.panasonic.com/cdbs/www-data/pdf/RDA0000/AOA0000C304.pdf"
 			(at 227.33 125.73 0)
 			(effects
@@
 			)
 		)
-		(property "Description" "49.9 Ohms ±1% 0.063W, 1/16W Chip Resistor 0402 (1005 Metric) Moisture Resistant Thick Film"
+		(property "Description" "49.9 Ohms ±1% 0.1W, 1/10W Chip Resistor 0603 (1608 Metric) Automotive AEC-Q200 Thick Film"
 			(at 227.33 125.73 0)
 			(effects
@@
 			)
 		)
-		(property "Link" "https://www.digikey.jp/en/products/detail/yageo/RC0402FR-0749R9L/726621"
+		(property "Link" "https://www.digikey.jp/en/products/detail/panasonic-electronic-components/ERJ-3EKF49R9V/196378"
 			(at 227.33 125.73 0)
 			(effects
@@
 			)
 		)
-		(property "MPN" "RC0402FR-0749R9L"
+		(property "MPN" "ERJ-3EKF49R9V"
 			(at 227.33 125.73 0)
 			(effects
@@
 			)
 		)
-		(property "Footprint" "Resistor_SMD:R_0402_1005Metric"
+		(property "Footprint" "Resistor_SMD:R_0603_1608Metric"
 			(at 228.6 109.22 0)
 			(effects
@@
 			)
 		)
-		(property "Datasheet" "https://www.yageo.com/upload/media/product/products/datasheet/rchip/PYu-RC_Group_51_RoHS_L_12.pdf"
+		(property "Datasheet" "https://industrial.panasonic.com/cdbs/www-data/pdf/RDA0000/AOA0000C304.pdf"
 			(at 228.6 109.22 0)
 			(effects
@@
 			)
 		)
-		(property "Description" "49.9 Ohms ±1% 0.063W, 1/16W Chip Resistor 0402 (1005 Metric) Moisture Resistant Thick Film"
+		(property "Description" "49.9 Ohms ±1% 0.1W, 1/10W Chip Resistor 0603 (1608 Metric) Automotive AEC-Q200 Thick Film"
 			(at 228.6 109.22 0)
 			(effects
@@
 			)
 		)
-		(property "Link" "https://www.digikey.jp/en/products/detail/yageo/RC0402FR-0749R9L/726621"
+		(property "Link" "https://www.digikey.jp/en/products/detail/panasonic-electronic-components/ERJ-3EKF49R9V/196378"
 			(at 228.6 109.22 0)
 			(effects
@@
 			)
 		)
-		(property "MPN" "RC0402FR-0749R9L"
+		(property "MPN" "ERJ-3EKF49R9V"
 			(at 228.6 109.22 0)
 			(effects

Commit message: Add files via upload
Parts:
- removed R18: 100K, Resistor_SMD:R_0603_1608Metric, symbol Library:R_Small
- added R18: 10K, Resistor_SMD:R_0603_1608Metric, symbol Library:R
Connections:
- net T1: now also R18.1
- net Vref2: now also R18.2
Changed lines of the file:
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@@
 	(wire
 		(pts
-			(xy 322.58 198.12) (xy 322.58 203.2)
-		)
-		(stroke
-			(width 0)
-			(type default)
-		)
-	)
-	(wire
-		(pts
 			(xy 76.2 67.31) (xy 88.9 67.31)
 		)
@@
 	(wire
 		(pts
+			(xy 322.58 184.15) (xy 322.58 191.77)
+		)
+		(stroke
+			(width 0)
+			(type default)
+		)
+	)
+	(wire
+		(pts
 			(xy 209.55 152.4) (xy 215.9 152.4)
 		)
@@
 	(wire
 		(pts
-			(xy 322.58 184.15) (xy 322.58 193.04)
-		)
-		(stroke
-			(width 0)
-			(type default)
-		)
-	)
-	(wire
-		(pts
 			(xy 140.97 128.27) (xy 144.78 128.27)
 		)
@@
 	(wire
 		(pts
+			(xy 322.58 199.39) (xy 322.58 203.2)
+		)
+		(stroke
+			(width 0)
+			(type default)
+		)
+	)
+	(wire
+		(pts
 			(xy 121.92 229.87) (xy 144.78 229.87)
 		)
@@
 	)
 	(symbol
+		(lib_id "Library:R")
+		(at 322.58 195.58 180)
+		(unit 1)
+		(exclude_from_sim no)
+		(in_bom yes)
+		(on_board yes)
+		(dnp no)
+		(property "Reference" "R18"
+			(at 320.04 196.85 0)
+			(effects
+				(font
+					(size 1.27 1.27)
+				)
+				(justify left)
+			)
+		)
+		(property "Value" "10K"
+			(at 320.04 194.31 0)
+			(effects
+				(font
+					(size 1.27 1.27)
+				)
+				(justify left)
+			)
+		)
+		(property "Footprint" "Resistor_SMD:R_0603_1608Metric"
+			(at 324.358 195.58 90)
+			(effects
+				(font
+					(size 1.27 1.27)
+				)
+				(hide yes)
+			)
+		)
+		(property "Datasheet" "https://www.seielect.com/catalog/sei-rmcf_rmcp.pdf"
+			(at 322.58 195.58 0)
+			(effects
+				(font
+					(size 1.27 1.27)
+				)
+				(hide yes)
+			)
+		)
+		(property "Description" "10 kOhms ±5% 0.1W, 1/10W Chip Resistor 0603 (1608 Metric) Automotive AEC-Q200 Thick Film"
+			(at 322.58 195.58 0)
+			(effects
+				(font
+					(size 1.27 1.27)
+				)
+				(hide yes)
+			)
+		)
+		(property "MPN" "RMCF0603JT10K0"
+			(at 322.58 195.58 0)
+			(effects
+				(font
+					(size 1.27 1.27)
+				)
+				(hide yes)
+			)
+		)
+		(property "Link" "https://www.digikey.jp/en/products/detail/stackpole-electronics-inc/RMCF0603JT10K0/1758104"
+			(at 322.58 195.58 0)
+			(effects
+				(font
+					(size 1.27 1.27)
+				)
+				(hide yes)
+			)
+		)
+		(pin "1"
+		)
+		(pin "2"
+		)
+		(instances
+			(project "LTC6811_ESP32_V2"
+				(path "/6a86ff6f-b159-4c4c-8a40-e732cc82e010/6b51f869-3fd5-42f9-b3ca-66a1d105433e/30216584-ee65-4156-92ea-2fa17f75418d"
+					(reference "R18")
+					(unit 1)
+				)
+				(path "/6a86ff6f-b159-4c4c-8a40-e732cc82e010/6b51f869-3fd5-42f9-b3ca-66a1d105433e/4e3577f7-fcc6-43dd-b7cf-8d175ec4d9f0"
+					(reference "R8")
+					(unit 1)
+				)
+				(path "/6a86ff6f-b159-4c4c-8a40-e732cc82e010/6b51f869-3fd5-42f9-b3ca-66a1d105433e/78d47b54-c839-4ab7-a5b0-c9844eec1512"
+					(reference "R13")
+					(unit 1)
+				)
+				(path "/6a86ff6f-b159-4c4c-8a40-e732cc82e010/6b51f869-3fd5-42f9-b3ca-66a1d105433e/fc3c799d-b983-4472-9d9d-934d3bacd380"
+					(reference "R3")
+					(unit 1)
+				)
+			)
+		)
+	)
+	(symbol
 		(lib_id "Library:LTC6811-1")
 		(at 196.85 144.78 0)
@@
 					(unit 1)
 				)
-			)
-		)
-	)
-	(symbol
-		(lib_id "Library:R_Small")
-		(at 322.58 195.58 0)
-		(unit 1)
-		(exclude_from_sim no)
-		(in_bom yes)
-		(on_board yes)
-		(dnp no)
-		(property "Reference" "R18"
-			(at 325.12 194.31 0)
-			(effects
-				(font
-					(size 1.27 1.27)
-				)
-				(justify left)
-			)
-		)
-		(property "Value" "100K"
-			(at 325.12 196.85 0)
-			(effects
-				(font
-					(size 1.27 1.27)
-				)
-				(justify left)
-			)
-		)
-		(property "Footprint" "Resistor_SMD:R_0603_1608Metric"
-			(at 320.802 195.58 90)
-			(effects
-				(font
-					(size 1.27 1.27)
-				)
-				(hide yes)
-			)
-		)
-		(property "Datasheet" "https://www.yageo.com/upload/media/product/app/datasheet/rchip/pyu-rc_group_51_rohs_l.pdf"
-			(at 322.58 195.58 0)
-			(effects
-				(font
-					(size 1.27 1.27)
-				)
-				(hide yes)
-			)
-		)
-		(property "Description" "100 kOhms ±5% 0.1W, 1/10W Chip Resistor 0603 (1608 Metric) Moisture Resistant Thick Film"
-			(at 322.58 195.58 0)
-			(effects
-				(font
-					(size 1.27 1.27)
-				)
-				(hide yes)
-			)
-		)
-		(property "MPN" "RC0603JR-07100KL"
-			(at 322.58 195.58 0)
-			(effects
-				(font
-					(size 1.27 1.27)
-				)
-				(hide yes)
-			)
-		)
-		(property "Link" "https://www.digikey.jp/en/products/detail/yageo/RC0603JR-07100KL/726698?s=N4IgTCBcDaIEoGEAMA2JBmAUnAtEg7AIxJIDSAMiALoC%2BQA"
-			(at 322.58 195.58 0)
-			(effects
-				(font
-					(size 1.27 1.27)
-				)
-				(hide yes)
-			)
-		)
-		(pin "1"
-		)
-		(pin "2"
-		)
-		(instances
-			(project "LTC6811_ESP32_V2"
-				(path "/6a86ff6f-b159-4c4c-8a40-e732cc82e010/6b51f869-3fd5-42f9-b3ca-66a1d105433e/30216584-ee65-4156-92ea-2fa17f75418d"
-					(reference "R18")
-					(unit 1)
-				)
-				(path "/6a86ff6f-b159-4c4c-8a40-e732cc82e010/6b51f869-3fd5-42f9-b3ca-66a1d105433e/4e3577f7-fcc6-43dd-b7cf-8d175ec4d9f0"
-					(reference "R8")
-					(unit 1)
-				)
-				(path "/6a86ff6f-b159-4c4c-8a40-e732cc82e010/6b51f869-3fd5-42f9-b3ca-66a1d105433e/78d47b54-c839-4ab7-a5b0-c9844eec1512"
-					(reference "R13")
-					(unit 1)
-				)
-				(path "/6a86ff6f-b159-4c4c-8a40-e732cc82e010/6b51f869-3fd5-42f9-b3ca-66a1d105433e/fc3c799d-b983-4472-9d9d-934d3bacd380"
-					(reference "R3")
-					(unit 1)
-				)
