File: LTC6811_ESP32_V2/Slaves.kicad_sch (KiCad schematic)
At the start: 3 parts, among them J7 B2P-VH-B, J9 B2P-VH-B

Commit message: Add files via upload
Parts:
- added C26, C45, C47, C49, C73, C74, C75, C76, C96, C97: 10nF/100V, Capacitor_SMD:C_0402_1005Metric, symbol Library:C
- added TR1, TR3, TR4, TR5, TR6: HM2108NL, Transformer_SMD:HM2108NL, symbol Library:HM2108NL
- J7, J9: symbol Connector_Generic:Conn_01x02 -> Library:Conn_01x02
- LOGO2: symbol Graphic:Logo_Tetra -> Library:Logo_Tetra
Connections:
- net LTC6811_1/MB: no longer names the net of J7.2 (Pin_2)
- net LTC6811_1/MB: now also TR1.6
- net LTC6811_1/PB: no longer names the net of J7.1 (Pin_1)
- net LTC6811_1/PB: now also TR1.4
- net LTC6811_4/MA: no longer names the net of J9.1 (Pin_1)
- net LTC6811_4/MA: now also TR6.1
- net LTC6811_4/PA: no longer names the net of J9.2 (Pin_2)
- net LTC6811_4/PA: now also TR6.3
- new net: C73.2, TR1.2
- new net: C74.1, TR1.5
- new net: C76.1, TR5.2
- new net: C75.1, TR5.5
- new net: C96.1, TR6.5
- new net: C97.1, TR6.2
- new net: C26.1, TR3.5
- new net: C45.1, TR3.2
- new net: C49.1, TR4.2
- new net: C47.1, TR4.5
- new net GND_PACK: C26.2, C45.2, C47.2, C49.2, C73.1, C74.2, C75.2, C76.2, C96.2, C97.2
- new net LTC6811_1/IMA: TR3.4
- new net LTC6811_1/IMB: TR1.1
- new net LTC6811_1/IPA: TR3.6
- new net LTC6811_1/IPB: TR1.3
- new net LTC6811_2/IMA: TR4.4
- new net LTC6811_2/IMB: TR3.3
- new net LTC6811_2/IPA: TR4.6
- new net LTC6811_2/IPB: TR3.1
- new net LTC6811_3/IMA: TR5.4
- new net LTC6811_3/IMB: TR4.3
- new net LTC6811_3/IPA: TR5.6
- new net LTC6811_3/IPB: TR4.1
- new net LTC6811_4/IMA: TR6.4
- new net LTC6811_4/IMB: TR5.3
- new net LTC6811_4/IPA: TR6.6
- new net LTC6811_4/IPB: TR5.1
Other:
- sheet LTC6811_1 ports: added IMA, IMB, IPA, IPB; removed MA, MB, PA, PB
- sheet LTC6811_2 ports: added IMA, IMB, IPA, IPB; removed MA, MB, PA, PB
- sheet LTC6811_3 ports: added IMA, IMB, IPA, IPB; removed MA, MB, PA, PB
- sheet LTC6811_4 ports: added IMA, IMB, IPA, IPB; removed MA, MB, PA, PB
- moved on the sheet: J7, J9

Commit message: Add files via upload
Connections:
- net LTC6811_1/IMA: now also TR1.3; no longer TR3.4
- net LTC6811_1/IMB: now also TR3.4; no longer TR1.1
- net LTC6811_1/IPA: now also TR1.1; no longer TR3.6
- net LTC6811_1/IPB: now also TR3.6; no longer TR1.3
- net LTC6811_2/IMA: now also TR3.3; no longer TR4.4
- net LTC6811_2/IMB: now also TR4.4; no longer TR3.3
- net LTC6811_2/IPA: now also TR3.1; no longer TR4.6
- net LTC6811_2/IPB: now also TR4.6; no longer TR3.1
- net LTC6811_3/IMA: now also TR4.3; no longer TR5.4
- net LTC6811_3/IMB: now also TR5.4; no longer TR4.3
- net LTC6811_3/IPA: now also TR4.1; no longer TR5.6
- net LTC6811_3/IPB: now also TR5.6; no longer TR4.1
- net LTC6811_4/IMA: now also TR5.3; no longer TR6.4
- net LTC6811_4/IMB: now also TR6.4; no longer TR5.3
- net LTC6811_4/IPA: now also TR5.1; no longer TR6.6
- net LTC6811_4/IPB: now also TR6.6; no longer TR5.1
- net at TR1.4: now also J7.2 (Pin_2); no longer J7.1 (Pin_1)
- net at TR1.6: now also J7.1 (Pin_1); no longer J7.2 (Pin_2)
Other:
- note added: "TO Master"
- note added: "TO Slaves"
Changed lines of the file:
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@@
+		)
+	)
+	(text "TO Master"
+		(exclude_from_sim no)
+		(at 23.114 74.93 0)
+		(effects
+			(font
+				(size 1.27 1.27)
+			)
+		)
+	)
+	(text "TO Slaves"
+		(exclude_from_sim no)
+		(at 277.114 75.438 0)
+		(effects
+			(font
+				(size 1.27 1.27)
+			)
 		)
 	)
@@
 	(symbol
 		(lib_id "Library:HM2108NL")
-		(at 53.34 81.28 0)
+		(at 53.34 83.82 0)
+		(mirror x)
 		(unit 1)
 		(exclude_from_sim no)
@@
 		(dnp no)
 		(property "Reference" "TR1"
-			(at 47.752 93.472 0)
+			(at 47.752 71.628 0)
 			(effects
 				(font
@@
 		)
 		(property "Value" "HM2108NL"
-			(at 48.006 90.678 0)
+			(at 48.006 74.422 0)
 			(effects
 				(font
@@
 		)
 		(property "Footprint" "Transformer_SMD:HM2108NL"
-			(at 54.61 83.82 0)
+			(at 54.61 81.28 0)
 			(effects
 				(font
@@
 		)
 		(property "Datasheet" "https://productfinder.pulseelectronics.com/api/open/part-attachments/datasheet/HM2108NL"
-			(at 54.61 83.82 0)
+			(at 54.61 81.28 0)
 			(effects
 				(font
@@
 		)
 		(property "Description" "135µH Pulse Transformer Surface Mount"
-			(at 53.34 81.28 0)
+			(at 53.34 83.82 0)
 			(effects
 				(font
@@
 		)
 		(property "MPN" "HM2108NL"
-			(at 53.34 81.28 0)
+			(at 53.34 83.82 0)
 			(effects
 				(font
@@
 		)
 		(property "Link" "https://www.digikey.jp/en/products/detail/pulse-electronics/HM2108NL/7914611"
-			(at 53.34 81.28 0)
+			(at 53.34 83.82 0)
 			(effects
 				(font
@@
 		)
 		(pin "IPA" input
+			(at 223.52 77.47 180)
+			(effects
+				(font
+					(size 1.27 1.27)
+				)
+				(justify left)
+			)
+		)
+		(pin "IMB" input
+			(at 238.76 87.63 0)
+			(effects
+				(font
+					(size 1.27 1.27)
+				)
+				(justify right)
+			)
+		)
+		(pin "IMA" input
+			(at 223.52 87.63 180)
+			(effects
+				(font
+					(size 1.27 1.27)
+				)
+				(justify left)
+			)
+		)
+		(pin "IPB" input
 			(at 238.76 77.47 0)
 			(effects
@@
 				)
 				(justify right)
-			)
-		)
-		(pin "IMB" input
-			(at 223.52 87.63 180)
-			(effects
-				(font
-					(size 1.27 1.27)
-				)
-				(justify left)
-			)
-		)
-		(pin "IMA" input
-			(at 238.76 87.63 0)
-			(effects
-				(font
-					(size 1.27 1.27)
-				)
-				(justify right)
-			)
-		)
-		(pin "IPB" input
-			(at 223.52 77.47 180)
-			(effects
-				(font
-					(size 1.27 1.27)
-				)
-				(justify left)
 			)
 		)
@@
 		)
 		(pin "IPA" input
+			(at 120.65 77.47 180)
+			(effects
+				(font
+					(size 1.27 1.27)
+				)
+				(justify left)
+			)
+		)
+		(pin "IMB" input
+			(at 137.16 87.63 0)
+			(effects
+				(font
+					(size 1.27 1.27)
+				)
+				(justify right)
+			)
+		)
+		(pin "IMA" input
+			(at 120.65 87.63 180)
+			(effects
+				(font
+					(size 1.27 1.27)
+				)
+				(justify left)
+			)
+		)
+		(pin "IPB" input
 			(at 137.16 77.47 0)
 			(effects
@@
 				)
 				(justify right)
-			)
-		)
-		(pin "IMB" input
-			(at 120.65 87.63 180)
-			(effects
-				(font
-					(size 1.27 1.27)
-				)
-				(justify left)
-			)
-		)
-		(pin "IMA" input
-			(at 137.16 87.63 0)
-			(effects
-				(font
-					(size 1.27 1.27)
-				)
-				(justify right)
-			)
-		)
-		(pin "IPB" input
-			(at 120.65 77.47 180)
-			(effects
-				(font
-					(size 1.27 1.27)
-				)
-				(justify left)
 			)
 		)
@@
 		)
 		(pin "IPA" input
+			(at 171.45 77.47 180)
+			(effects
+				(font
+					(size 1.27 1.27)
+				)
+				(justify left)
+			)
+		)
+		(pin "IMB" input
+			(at 184.15 87.63 0)
+			(effects
+				(font
+					(size 1.27 1.27)
+				)
+				(justify right)
+			)
+		)
+		(pin "IMA" input
+			(at 171.45 87.63 180)
+			(effects
+				(font
+					(size 1.27 1.27)
+				)
+				(justify left)
+			)
+		)
+		(pin "IPB" input
 			(at 184.15 77.47 0)
 			(effects
@@
 				)
 				(justify right)
-			)
-		)
-		(pin "IMB" input
-			(at 171.45 87.63 180)
-			(effects
-				(font
-					(size 1.27 1.27)
-				)
-				(justify left)
-			)
-		)
-		(pin "IMA" input
-			(at 184.15 87.63 0)
-			(effects
-				(font
-					(size 1.27 1.27)
-				)
-				(justify right)
-			)
-		)
-		(pin "IPB" input
-			(at 171.45 77.47 180)
-			(effects
-				(font
-					(size 1.27 1.27)
-				)
-				(justify left)
 			)
 		)
@@
 		)
 		(pin "IPB" input
+			(at 86.36 77.47 0)
+			(effects
+				(font
+					(size 1.27 1.27)
+				)
+				(justify right)
+			)
+		)
+		(pin "IMA" input
+			(at 67.31 87.63 180)
+			(effects
+				(font
+					(size 1.27 1.27)
+				)
+				(justify left)
+			)
+		)
+		(pin "IPA" input
 			(at 67.31 77.47 180)
 			(effects
@@
 			)
 		)
-		(pin "IMA" input
+		(pin "IMB" input
 			(at 86.36 87.63 0)
 			(effects
@@
 			)
 		)
-		(pin "IPA" input
-			(at 86.36 77.47 0)
-			(effects
-				(font
-					(size 1.27 1.27)
-				)
-				(justify right)
-			)
-		)
-		(pin "IMB" input
-			(at 67.31 87.63 180)
-			(effects
-				(font
-					(size 1.27 1.27)
-				)
-				(justify left)
-			)
-		)

Commit message: Add files via upload
Parts:
- C26, C45, C47, C49, C73, C75, C76, C96, C97: footprint Capacitor_SMD:C_0402_1005Metric -> Capacitor_SMD:C_0603_1608Metric; Link https://www.digikey.jp/en/products/detail/kemet/C0402C103K1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 -> https://www.digikey.jp/en/products/detail/kemet/C0603X103K1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; MPN C0402C103K1RACAUTO -> C0603X103K1RAC3316
- C74: value 10nF/100V -> 10nF/100V NC; footprint Capacitor_SMD:C_0402_1005Metric -> Capacitor_SMD:C_0603_1608Metric; Link https://www.digikey.jp/en/products/detail/kemet/C0402C103K1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 -> https://www.digikey.jp/en/products/detail/kemet/C0603X103K1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; MPN C0402C103K1RACAUTO -> C0603X103K1RAC3316

Commit message: Add files via upload
Parts:
- removed C74: 10nF/100V NC, Capacitor_SMD:C_0603_1608Metric, symbol Library:C
- removed C97: 10nF/100V, Capacitor_SMD:C_0603_1608Metric, symbol Library:C
Connections:
- no-connect marks 0 -> 2

Commit message: Add files via upload
Parts:
- removed C73: 10nF/100V, Capacitor_SMD:C_0603_1608Metric, symbol Library:C
- removed J7: B2P-VH-B, Connector_JST:JST_VH_B2P-VH-B_1x02_P3.96mm_Vertical, symbol Library:Conn_01x02
- removed TR1: HM2108NL, Transformer_SMD:HM2108NL, symbol Library:HM2108NL
Connections:
- net LTC6811_4/IMB: now also TR6.6; no longer TR6.4
- net LTC6811_4/IPB: now also TR6.4; no longer TR6.6
- net at TR6.1: now also J9.2 (Pin_2); no longer J9.1 (Pin_1)
- net at TR6.3: now also J9.1 (Pin_1); no longer J9.2 (Pin_2)
- no-connect marks 2 -> 1

Commit message: Add two positioning holes.
Connections:
- net MB: now reaches J9.2 (Pin_2), TR6.1
- net PB: now reaches J9.1 (Pin_1), TR6.3
Changed lines of the file:
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@@
+		)
+	)
+	(label "MB"
+		(at 269.24 87.63 0)
+		(fields_autoplaced yes)
+		(effects
+			(font
+				(size 1.27 1.27)
+			)
+			(justify left bottom)
+		)
+	)
+	(label "PB"
+		(at 269.24 77.47 0)
+		(fields_autoplaced yes)
+		(effects
+			(font
+				(size 1.27 1.27)
+			)
+			(justify left bottom)
 		)
 	)
