File: LTC6811_ESP32_V3/CAN.kicad_sch (KiCad schematic)
At the start: 6 parts, among them U10 ISO1050DUBR

Commit message: Update BOM
Parts:
- C33, C35: Link https://www.digikey.jp/en/products/detail/nextgen-component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 -> https://www.digikey.jp/en/products/detail/samsung-electro-m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; MPN 0603B105K250XD -> CL10B105KA8NNNC
Changed lines of the file:
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@@
 			)
 		)
-		(property "Datasheet" "https://mm.digikey.com/Volume0/opasdata/d220001/medias/docus/4562/0603B105K250XD.pdf"
+		(property "Datasheet" "https://mm.digikey.com/Volume0/opasdata/d220001/medias/docus/3644/CL10B105KA8NNNC_spec.pdf"
 			(at 129.032 138.938 0)
 			(effects
@@
 			)
 		)
-		(property "MPN" "0603B105K250XD"
-			(at 129.032 138.938 0)
-			(effects
-				(font
-					(size 1.27 1.27)
-				)
-				(hide yes)
-			)
-		)
-		(property "Link" "https://www.digikey.jp/en/products/detail/nextgen-components/0603B105K250XD/14670931"
+		(property "MPN" "CL10B105KA8NNNC"
+			(at 129.032 138.938 0)
+			(effects
+				(font
+					(size 1.27 1.27)
+				)
+				(hide yes)
+			)
+		)
+		(property "Link" "https://www.digikey.jp/en/products/detail/samsung-electro-mechanics/CL10B105KA8NNNC/3886842"
 			(at 129.032 138.938 0)
 			(effects
@@
 			)
 		)
-		(property "Datasheet" "https://mm.digikey.com/Volume0/opasdata/d220001/medias/docus/4562/0603B105K250XD.pdf"
+		(property "Datasheet" "https://mm.digikey.com/Volume0/opasdata/d220001/medias/docus/3644/CL10B105KA8NNNC_spec.pdf"
 			(at 213.487 126.238 0)
 			(effects
@@
 			)
 		)
-		(property "MPN" "0603B105K250XD"
-			(at 213.487 126.238 0)
-			(effects
-				(font
-					(size 1.27 1.27)
-				)
-				(hide yes)
-			)
-		)
-		(property "Link" "https://www.digikey.jp/en/products/detail/nextgen-components/0603B105K250XD/14670931"
-			(at 213.487 126.238 0)
-			(effects
+		(property "MPN" "CL10B105KA8NNNC"
+			(at 213.487 126.238 0)
+			(effects
+				(font
+					(size 1.27 1.27)
+				)
+				(hide yes)
+			)
+		)
+		(property "Link" "https://www.digikey.jp/en/products/detail/samsung-electro-mechanics/CL10B105KA8NNNC/3886842"
+			(at 213.487 126.238 0)
+			(effects
