File: LTC6811_ESP32_V3/LTC6811.kicad_sch (KiCad schematic)
At the start: 52 parts, among them J16 B7B-XH-A, J17 B7B-XH-A, Q40 NSV1C201MZ4, U14 LTC6811HG-1

Commit message: Update BOM
Parts:
- removed TH16: 100K NTC SMD, Resistor_SMD:R_0603_1608Metric, symbol Library:Thermistor
- added TH1: 10K NTC SMD, Library:R_0603_1608Metric, symbol Device:Thermistor
- C116, C117: Link https://www.digikey.jp/en/products/detail/nextgen-component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 -> https://www.digikey.jp/en/products/detail/samsung-electro-m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; MPN 0603B105K250XD -> CL10B105KA8NNNC
- C66: Link (none) -> https://www.digikey.jp/en/products/detail/samsung-electro-m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; 购买链接 https://www.digikey.jp/en/products/detail/samsung-electro-m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 -> (none)
- R101, R93: Link (none) -> https://www.digikey.jp/en/products/detail/yageo/RC0603FR-07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; MPN (none) -> RC0603FR-071KL
- R18, R19, R20, R21, R22: Link https://www.digikey.jp/en/products/detail/stackpole-electro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 -> https://www.digikey.jp/en/products/detail/yageo/RC0603FR-07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; MPN RMCF0603JT10K0 -> RC0603FR-0710KL
Connections:
- net GND_PACK: now also TH1.2
- net T1: now also TH1.1
