File: LTC6811_ESP32_V3/MCU.kicad_sch (KiCad schematic)
At the start: 30 parts, among them J21 B2P-VH-B, SW1 SW_DIP_x08, U1 MCP23S17_SP, U8 ESP32-DevKitC V4, U9 LTC6820

Commit message: Update BOM
Parts:
- C31: Link https://www.digikey.jp/en/products/detail/nextgen-component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 -> https://www.digikey.jp/en/products/detail/samsung-electro-m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; MPN 0603B105K250XD -> CL10B105KA8NNNC
- J21: Link https://www.digikey.jp/en/products/detail/molex/0705430001/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 -> https://www.digikey.jp/en/products/detail/jst-sales-america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; MPN 70543-0001 -> B2P-VH
- R102, R103, R104, R105, R144, R148, R149, R151, R34: Link https://www.digikey.jp/en/products/detail/stackpole-electro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 -> https://www.digikey.jp/en/products/detail/yageo/RC0603FR-07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; MPN RMCF0603JT10K0 -> RC0603FR-0710KL
- R35, R38: Link (none) -> https://www.digikey.jp/en/products/detail/yageo/RC0603FR-07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; MPN (none) -> RC0603FR-071KL
- SW1: Link (none) -> https://www.digikey.jp/en/products/detail/cts-electrocompon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; MPN (none) -> 208-8
- U1: Link (none) -> https://www.digikey.jp/en/products/detail/microchip-technol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; MPN (none) -> MCP23S17-E/SP
