File: LTC6811_ESP32_V5/Slaves/LTC6811.kicad_sch (KiCad schematic)
At the start: 52 parts, among them J16 B7B-XH-A, J17 B7B-XH-A, Q40 NSV1C201MZ4, U14 LTC6811HG-1

Commit message: Add files via upload
Parts:
- C11: renamed from C16; footprint Capacitor_SMD:C_0603_1608Metric -> Library:C_0603_1608Metric
- C12: renamed from C17; footprint Capacitor_SMD:C_0603_1608Metric -> Library:C_0603_1608Metric; symbol Library:C-Device -> Library:C_Small
- C13: renamed from C18; footprint Capacitor_SMD:C_0603_1608Metric -> Library:C_0603_1608Metric; symbol Library:C-Device -> Library:C_Small
- C14: renamed from C19; footprint Capacitor_SMD:C_0603_1608Metric -> Library:C_0603_1608Metric; symbol Library:C-Device -> Library:C_Small
- C15: renamed from C22; footprint Capacitor_SMD:C_0603_1608Metric -> Library:C_0603_1608Metric; symbol Library:C-Device -> Library:C_Small
- C43: renamed from C66; footprint Capacitor_SMD:C_0603_1608Metric -> Library:C_0603_1608Metric
- C89: renamed from C115; footprint Capacitor_SMD:C_0603_1608Metric -> Library:C_0603_1608Metric
- C90: renamed from C116; footprint Capacitor_SMD:C_0603_1608Metric -> Library:C_0603_1608Metric
- C91: renamed from C117; footprint Capacitor_SMD:C_0603_1608Metric -> Library:C_0603_1608Metric
- C93: renamed from C119; footprint Capacitor_SMD:C_0603_1608Metric -> Library:C_0603_1608Metric
- D38: renamed from D54; footprint Diode_SMD:D_SOD-123 -> Library:D_SOD-123
- D39: renamed from D55; footprint Diode_SMD:D_SOD-123 -> Library:D_SOD-123
- D40: renamed from D56; footprint Diode_SMD:D_SOD-123F -> Library:D_SOD-123F
- D41: renamed from D57; footprint LED_SMD:LED_0603_1608Metric -> Library:LED_0603_1608Metric
- F27: renamed from F40; footprint Fuse:Fuse_0805_2012Metric -> Library:Fuse_0805_2012Metric
- F28: renamed from F41; footprint Fuse:Fuse_0805_2012Metric -> Library:Fuse_0805_2012Metric
- F29: renamed from F42; footprint Fuse:Fuse_0805_2012Metric -> Library:Fuse_0805_2012Metric
- F30: renamed from F43; footprint Fuse:Fuse_0805_2012Metric -> Library:Fuse_0805_2012Metric
- F31: renamed from F44; footprint Fuse:Fuse_0805_2012Metric -> Library:Fuse_0805_2012Metric
- F32: renamed from F45; footprint Fuse:Fuse_0805_2012Metric -> Library:Fuse_0805_2012Metric
- F33: renamed from F46; footprint Fuse:Fuse_0805_2012Metric -> Library:Fuse_0805_2012Metric
- F34: renamed from F47; footprint Fuse:Fuse_0805_2012Metric -> Library:Fuse_0805_2012Metric
- F35: renamed from F48; footprint Fuse:Fuse_0805_2012Metric -> Library:Fuse_0805_2012Metric
- F36: renamed from F49; footprint Fuse:Fuse_0805_2012Metric -> Library:Fuse_0805_2012Metric
- F37: renamed from F50; footprint Fuse:Fuse_0805_2012Metric -> Library:Fuse_0805_2012Metric
- F38: renamed from F51; footprint Fuse:Fuse_0805_2012Metric -> Library:Fuse_0805_2012Metric
- F39: renamed from F52; footprint Fuse:Fuse_0805_2012Metric -> Library:Fuse_0805_2012Metric
- FB3: renamed from FB4; footprint Resistor_SMD:R_0603_1608Metric -> Library:R_0603_1608Metric
- J14: renamed from J16; footprint Connector_JST:JST_XH_B7B-XH-A_1x07_P2.50mm_Vertical_BAT_6S -> Library:JST_XH_B7B-XH-A_1x07_P2.50mm_Vertical_BAT_6S
- J15: renamed from J17; footprint Connector_JST:JST_XH_B7B-XH-A_1x07_P2.50mm_Vertical_BAT_6S -> Library:JST_XH_B7B-XH-A_1x07_P2.50mm_Vertical_BAT_6S
- Q27: renamed from Q40; footprint Package_TO_SOT_SMD:SOT-223 -> Library:SOT-223
- R100: renamed from R101; footprint Resistor_SMD:R_0603_1608Metric -> Library:R_0603_1608Metric
- R13: renamed from R18; footprint Resistor_SMD:R_0603_1608Metric -> Library:R_0603_1608Metric
- R14: renamed from R19; footprint Resistor_SMD:R_0603_1608Metric -> Library:R_0603_1608Metric
- R142: renamed from R193; footprint Resistor_SMD:R_0603_1608Metric -> Library:R_0603_1608Metric
- R143: renamed from R194; footprint Resistor_SMD:R_0603_1608Metric -> Library:R_0603_1608Metric
- R145: renamed from R196; footprint Resistor_SMD:R_0603_1608Metric -> Library:R_0603_1608Metric
- R146: renamed from R197; footprint Resistor_SMD:R_0603_1608Metric -> Library:R_0603_1608Metric
- R147: renamed from R198; footprint Resistor_SMD:R_0603_1608Metric -> Library:R_0603_1608Metric
- R15: renamed from R20; footprint Resistor_SMD:R_0603_1608Metric -> Library:R_0603_1608Metric
- R150: renamed from R201; footprint Resistor_SMD:R_0603_1608Metric -> Library:R_0603_1608Metric
- R16: renamed from R21; footprint Resistor_SMD:R_0603_1608Metric -> Library:R_0603_1608Metric
- R17: renamed from R22; footprint Resistor_SMD:R_0603_1608Metric -> Library:R_0603_1608Metric
- R54: renamed from R93; footprint Resistor_SMD:R_0603_1608Metric -> Library:R_0603_1608Metric
- TH11: renamed from TH16; symbol Library:Thermistor -> Library:Thermistor_NTC_small
- TH12: renamed from TH17; footprint Resistor_THT:R_Axial_DIN0204_L3.6mm_D1.6mm_P1.90mm_Vertical -> Library:R_Axial_DIN0204_L3.6mm_D1.6mm_P1.90mm_Vertical; symbol Library:Thermistor -> Library:Thermistor_NTC_small
- TH13: renamed from TH18; footprint Resistor_THT:R_Axial_DIN0204_L3.6mm_D1.6mm_P1.90mm_Vertical -> Library:R_Axial_DIN0204_L3.6mm_D1.6mm_P1.90mm_Vertical; symbol Library:Thermistor -> Library:Thermistor_NTC_small
- TH14: renamed from TH19; footprint Resistor_THT:R_Axial_DIN0204_L3.6mm_D1.6mm_P1.90mm_Vertical -> Library:R_Axial_DIN0204_L3.6mm_D1.6mm_P1.90mm_Vertical; symbol Library:Thermistor -> Library:Thermistor_NTC_small
- TH15: renamed from TH20; footprint Resistor_THT:R_Axial_DIN0204_L3.6mm_D1.6mm_P1.90mm_Vertical -> Library:R_Axial_DIN0204_L3.6mm_D1.6mm_P1.90mm_Vertical; symbol Library:Thermistor -> Library:Thermistor_NTC_small
- TP7: renamed from TP9; footprint TestPoint:TestPoint_Pad_D1.0mm -> Library:TestPoint_Pad_D1.0mm; now left out of the parts list
- TP8: renamed from TP10; footprint TestPoint:TestPoint_Pad_D1.0mm -> Library:TestPoint_Pad_D1.0mm; now left out of the parts list
- U13: renamed from U14; footprint Package_SO:TSSOP-48_6.1x12.5mm_P0.5mm -> Library:TSSOP-48_6.1x12.5mm_P0.5mm
Other:
- moved on the sheet: C11, C12, C13, C14, C15, C43, C89, C90, C91, C93, D38, D39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
