File: LTC6811_ESP32_V5/Slaves/cell.kicad_sch (KiCad schematic)
At the start: 6 parts, among them Q48 TSM2323

Commit message: Add files via upload
Parts:
- C110: renamed from C136; footprint Capacitor_SMD:C_0603_1608Metric -> Library:C_0603_1608Metric
- D49: renamed from D65; footprint Diode_SMD:D_SOD-323_HandSoldering -> Library:D_SOD-323_HandSoldering
- Q35: renamed from Q48; footprint Package_TO_SOT_SMD:SOT-23 -> Library:SOT-23
- R178: renamed from R229; footprint Resistor_SMD:R_2512_6332Metric -> Library:R_2512_6332Metric
- R179: renamed from R230; footprint Resistor_SMD:R_0603_1608Metric -> Library:R_0603_1608Metric
- R180: renamed from R231; footprint Resistor_SMD:R_0603_1608Metric -> Library:R_0603_1608Metric
Other:
- moved on the sheet: C110, D49, Q35, R178, R179, R180
