File: LTC6811_ESP32_V5/Main/CAN.kicad_sch (KiCad schematic)
At the start: 7 parts, among them U2 MCP2562T-E/SN

Commit message: Add files via upload
Parts:
- added JP4: SolderJumper_2_Open, Jumper:SolderJumper-2_P1.3mm_Open_TrianglePad1.0x1.5mm, symbol Jumper:SolderJumper_2_Open
Connections:
- net CAN_H: now also JP4.1 (A); no longer R153.2
- new net: JP4.2 (B), R153.2
Other:
- moved on the sheet: C21, C47, C48, C49, R152, R153, U2
