File: LTC6811_ESP32_V5/Main/LTC6811.kicad_sch (KiCad schematic)
At the start: 52 parts, among them J16 B7B-XH-A, J17 B7B-XH-A, Q40 NSV1C201MZ4, U14 LTC6811HG-1

Commit message: Add files via upload
Parts:
- renumbered C22 to C10, C66 to C42, C16 to C6, C115 to C63, C116 to C64, C117 to C65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

Commit message: Add files via upload
Other:
- moved on the sheet: C10, C42, C6, C63, C64, C65, C67, C7, C8, C9, D22, D23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
