File: LTC6811_ESP32_V5/Main/LTC6811_ESP32_V5_Main.kicad_pcb (KiCad board)
At the start: 2 copper layers, 200 x 55 mm, 325 parts, among them J10 B7B-XH-A, J11 B7B-XH-A, J12 B7B-XH-A, J13 B7B-XH-A, J18 Hole /NC, J19 Hole /NC, J21 Hole /NC, J23 CAN, J3 Hole /NC, J4 Hole /NC, J5 CAN, J6 B2P-VH-B, J7 Hole /NC, Q1 NSV1C201MZ4, Q10 TSM2323, Q11 TSM2323, Q12 TSM2323, Q13 TSM2323, Q14 NSV1C201MZ4, Q15 TSM2323, Q16 TSM2323, Q17 TSM2323, Q18 TSM2323, Q19 TSM2323, Q2 TSM2323, Q20 TSM2323, Q21 TSM2323, Q22 TSM2323, Q23 TSM2323, Q24 TSM2323, Q25 TSM2323, Q26 TSM2323, Q3 TSM2323, Q4 TSM2323, Q5 TSM2323, Q6 TSM2323, Q7 TSM2323, Q8 TSM2323, Q9 TSM2323, SW1 SW_DIP_x08, U1 MCP23017T-E/SO, U11 LTC6811HG-1, U12 LTC6811HG-1, U2 MCP2562T-E/SN, U3 BD33FC0FP-E2, U4 BD50FC0FP-E2, U8 ESP32-DevKitC V4, U9 LTC6820

Commit message: Add files via upload
Parts:
- added JP4: SolderJumper_2_Open, Jumper:SolderJumper-2_P1.3mm_Open_TrianglePad1.0x1.5mm, F.Cu at (47.5, 129.2)
Connections:
- R153 pad 2: /CAN/CAN_H -> Net-(JP4-B)
Changed lines of the file:
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@@
 	(net 275 "/PowerSupply/+12V")
 	(net 276 "Net-(C29-Pad2)")
+	(net 277 "Net-(JP4-B)")
 	(footprint "RF_Module:ESP32-DevKitc V4_DIP-38_27.9mm×48.2mm"
 		(layer "F.Cu")
@@
 			(layers "F.Cu" "F.Paste" "F.Mask")
 			(roundrect_rratio 0.25)
-			(net 53 "/CAN/CAN_H")
+			(net 277 "Net-(JP4-B)")
 			(pintype "passive")
 		)
@@
 			)
 		)
+	)
+	(footprint "Jumper:SolderJumper-2_P1.3mm_Open_TrianglePad1.0x1.5mm"
+		(layer "F.Cu")
+		(at 47.475 129.2)
+		(descr "SMD Solder Jumper, 1x1.5mm Triangular Pads, 0.3mm gap, open")
+		(tags "solder jumper open")
+		(property "Reference" "JP4"
+			(at 0 -1.8 0)
+			(layer "F.SilkS")
+			(effects
+				(font
+					(size 1 1)
+					(thickness 0.15)
+				)
+			)
+		)
+		(property "Value" "SolderJumper_2_Open"
+			(at 0 1.9 0)
+			(layer "F.Fab")
+			(effects
+				(font
+					(size 1 1)
+					(thickness 0.15)
+				)
+			)
+		)
+		(property "Footprint" "Jumper:SolderJumper-2_P1.3mm_Open_TrianglePad1.0x1.5mm"
+			(at 0 0 0)
+			(unlocked yes)
+			(layer "F.Fab")
+			(hide yes)
+			(effects
+				(font
+					(size 1.27 1.27)
+					(thickness 0.15)
+				)
+			)
+		)
+		(property "Datasheet" ""
+			(at 0 0 0)
+			(unlocked yes)
+			(layer "F.Fab")
+			(hide yes)
+			(effects
+				(font
+					(size 1.27 1.27)
+					(thickness 0.15)
+				)
+			)
+		)
+		(property "Description" "Solder Jumper, 2-pole, open"
+			(at 0 0 0)
+			(unlocked yes)
+			(layer "F.Fab")
+			(hide yes)
+			(effects
+				(font
+					(size 1.27 1.27)
+					(thickness 0.15)
+				)
+			)
+		)
+		(property ki_fp_filters "SolderJumper*Open*")
+		(sheetname "CAN")
+		(sheetfile "CAN.kicad_sch")
+		(zone_connect 1)
+		(attr exclude_from_pos_files exclude_from_bom)
+		(fp_line
+			(start -1.4 -1)
+			(end 1.4 -1)
+			(stroke
+				(width 0.12)
+				(type solid)
+			)
+			(layer "F.SilkS")
+		)
+		(fp_line
+			(start -1.4 1)
+			(end -1.4 -1)
+			(stroke
+				(width 0.12)
+				(type solid)
+			)
+			(layer "F.SilkS")
+		)
+		(fp_line
+			(start 1.4 -1)
+			(end 1.4 1)
+			(stroke
+				(width 0.12)
+				(type solid)
+			)
+			(layer "F.SilkS")
+		)
+		(fp_line
+			(start 1.4 1)
+			(end -1.4 1)
+			(stroke
+				(width 0.12)
+				(type solid)
+			)
+			(layer "F.SilkS")
+		)
+		(fp_line
+			(start -1.65 -1.25)
+			(end -1.65 1.25)
+			(stroke
+				(width 0.05)
+				(type solid)
+			)
+			(layer "F.CrtYd")
+		)
+		(fp_line
+			(start -1.65 -1.25)
+			(end 1.65 -1.25)
+			(stroke
+				(width 0.05)
+				(type solid)
+			)
+			(layer "F.CrtYd")
+		)
+		(fp_line
+			(start 1.65 1.25)
+			(end -1.65 1.25)
+			(stroke
+				(width 0.05)
+				(type solid)
+			)
+			(layer "F.CrtYd")
+		)
+		(fp_line
+			(start 1.65 1.25)
+			(end 1.65 -1.25)
+			(stroke
+				(width 0.05)
+				(type solid)
+			)
+			(layer "F.CrtYd")
+		)
+		(pad "1" smd custom
+			(at -0.725 0)
+			(size 0.3 0.3)
+			(layers "F.Cu" "F.Mask")
+			(net 53 "/CAN/CAN_H")
+			(pinfunction "A")
+			(pintype "passive")
+			(zone_connect 2)
+			(thermal_bridge_angle 45)
+			(options
+				(clearance outline)
+				(anchor rect)
+			)
+			(primitives
+				(gr_poly
+					(pts
+						(xy 1 0) (xy 0.5 0.75) (xy -0.5 0.75) (xy -0.5 -0.75) (xy 0.5 -0.75)
+					)
+					(width 0)
+					(fill yes)
+				)
+			)
+		)
+		(pad "2" smd custom
+			(at 0.725 0)
+			(size 0.3 0.3)
+			(layers "F.Cu" "F.Mask")
+			(net 277 "Net-(JP4-B)")
+			(pinfunction "B")
+			(pintype "passive")
+			(zone_connect 2)
+			(thermal_bridge_angle 45)
+			(options
+				(clearance outline)
+				(anchor rect)
+			)
+			(primitives
+				(gr_poly
+					(pts
+						(xy 0.5 0.75) (xy -0.65 0.75) (xy -0.15 0) (xy -0.65 -0.75) (xy 0.5 -0.75)
+					)
+					(width 0)
+					(fill yes)
+				)
+			)
+		)
