File: LTC6811_ESP32_V5/Main/LTC6811_ESP32_V5_Main.kicad_sch (KiCad schematic)
At the start: 13 parts, among them J1 Hole /NC, J18 Hole /NC, J19 Hole /NC, J2 Hole /NC, J20 Hole /NC, J21 Hole /NC, J23 CAN, J3 Hole /NC, J4 Hole /NC, J5 CAN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

Commit message: Add files via upload
Parts:
- removed J1, J2, J20, J8: Hole /NC, MountingHole:MountingHole_3.2mm_M3_ISO7380, symbol Mechanical:MountingHole
