File: LTC6811_ESP32_V5/Master/CAN.kicad_sch (KiCad schematic)
At the start: 7 parts, among them U2 MCP2562T-E/SN

Commit message: Add files via upload
Parts:
- C47, C49: value 0.1uF/50V -> 100nF/100V; Link https://www.digikey.jp/en/products/detail/samsung-electro-mechanics/CL10B104KB8NNWC/3887593 -> https://www.digikey.jp/en/products/detail/samsung-electro-mechanics/CL10B104KC8NNNC/5961291?s=N4IgTCBcDaIMIBkCMAGAQqgLAaTgDgDki4QBdAXyA; MPN CL10B104KB8NNWC -> CL10B104KC8NNNC
- JP4: now left out of the parts list
Changed lines of the file:
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@@
 			)
 		)
-		(property "Value" "0.1uF/50V"
+		(property "Value" "100nF/100V"
 			(at 132.08 67.945 0)
 			(effects
@@
 			)
 		)
-		(property "Datasheet" "https://mm.digikey.com/Volume0/opasdata/d220001/medias/docus/658/CL10B104KB8NNWC_Spec.pdf"
+		(property "Datasheet" "https://www.digikey.jp/en/products/detail/samsung-electro-mechanics/CL10B104KC8NNNC/5961291?s=N4IgTCBcDaIMIBkCMAGAQqgLAaTgDgDki4AdEkAXQF8g"
 			(at 132.08 65.405 0)
 			(effects
@@
 			)
 		)
-		(property "Description" "0.1 µF ±10% 50V Ceramic Capacitor X7R 0603 (1608 Metric)"
+		(property "Description" "0.1 µF ±10% 100V Ceramic Capacitor X7R 0603 (1608 Metric)"
 			(at 132.08 65.405 0)
 			(effects
@@
 			)
 		)
-		(property "MPN" "CL10B104KB8NNWC"
+		(property "MPN" "CL10B104KC8NNNC"
 			(at 132.08 65.405 0)
 			(effects
@@
 			)
 		)
-		(property "Link" "https://www.digikey.jp/en/products/detail/samsung-electro-mechanics/CL10B104KB8NNWC/3887593"
+		(property "Link" "https://www.digikey.jp/en/products/detail/samsung-electro-mechanics/CL10B104KC8NNNC/5961291?s=N4IgTCBcDaIMIBkCMAGAQqgLAaTgDgDki4QBdAXyA"
 			(at 132.08 65.405 0)
 			(effects
@@
 		(unit 1)
 		(exclude_from_sim yes)
-		(in_bom yes)
+		(in_bom no)
 		(on_board yes)
 		(dnp no)
@@
 			)
 		)
-		(property "Value" "0.1uF/50V"
+		(property "Value" "100nF/100V"
 			(at 89.535 89.535 0)
 			(effects
@@
 			)
 		)
-		(property "Datasheet" "https://mm.digikey.com/Volume0/opasdata/d220001/medias/docus/658/CL10B104KB8NNWC_Spec.pdf"
+		(property "Datasheet" "https://www.digikey.jp/en/products/detail/samsung-electro-mechanics/CL10B104KC8NNNC/5961291?s=N4IgTCBcDaIMIBkCMAGAQqgLAaTgDgDki4AdEkAXQF8g"
 			(at 89.535 86.995 0)
 			(effects
@@
 			)
 		)
-		(property "Description" "0.1 µF ±10% 50V Ceramic Capacitor X7R 0603 (1608 Metric)"
+		(property "Description" "0.1 µF ±10% 100V Ceramic Capacitor X7R 0603 (1608 Metric)"
 			(at 89.535 86.995 0)
 			(effects
@@
 			)
 		)
-		(property "MPN" "CL10B104KB8NNWC"
+		(property "MPN" "CL10B104KC8NNNC"
 			(at 89.535 86.995 0)
 			(effects
@@
 			)
 		)
-		(property "Link" "https://www.digikey.jp/en/products/detail/samsung-electro-mechanics/CL10B104KB8NNWC/3887593"
+		(property "Link" "https://www.digikey.jp/en/products/detail/samsung-electro-mechanics/CL10B104KC8NNNC/5961291?s=N4IgTCBcDaIMIBkCMAGAQqgLAaTgDgDki4QBdAXyA"
 			(at 89.535 86.995 0)
 			(effects
