File: LTC6811_ESP32_V5/Master/LTC6811_ESP32_Master_V5.kicad_pcb (KiCad board)
At the start: 2 copper layers, 200 x 55 mm, 325 parts, among them J10 B7B-XH-A, J11 B7B-XH-A, J12 B7B-XH-A, J13 B7B-XH-A, J18 Hole /NC, J19 Hole /NC, J21 Hole /NC, J23 CAN, J3 Hole /NC, J4 Hole /NC, J5 CAN, J6 B2P-VH-B, J7 Hole /NC, Q1 NSV1C201MZ4, Q10 TSM2323, Q11 TSM2323, Q12 TSM2323, Q13 TSM2323, Q14 NSV1C201MZ4, Q15 TSM2323, Q16 TSM2323, Q17 TSM2323, Q18 TSM2323, Q19 TSM2323, Q2 TSM2323, Q20 TSM2323, Q21 TSM2323, Q22 TSM2323, Q23 TSM2323, Q24 TSM2323, Q25 TSM2323, Q26 TSM2323, Q3 TSM2323, Q4 TSM2323, Q5 TSM2323, Q6 TSM2323, Q7 TSM2323, Q8 TSM2323, Q9 TSM2323, SW1 SW_DIP_x08, U1 MCP23017T-E/SO, U11 LTC6811HG-1, U12 LTC6811HG-1, U2 MCP2562T-E/SN, U3 BD33FC0FP-E2, U4 BD50FC0FP-E2, U8 ESP32-DevKitC V4, U9 LTC6820

Commit message: Add files via upload
Parts:
- C47, C49: value 0.1uF/50V -> 100nF/100V
Other:
- board text added: "BMS_ESP32 2024/09/12 LTC6811_Master_V5"
- board text removed: "BMS_Master 2024/09/12 LTC6811_ESP32_V5"
- board text removed: "BMS_Master LTC6811_ESP32_V5 2024/09/12"
Changed lines of the file:
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@@
 		(sheetname "LTC6811_1")
 		(sheetfile "LTC6811.kicad_sch")
-		(attr exclude_from_pos_files)
+		(attr exclude_from_pos_files exclude_from_bom)
 		(fp_circle
 			(center 0 0)
@@
 			(at 0 -1.448 0)
 			(layer "F.SilkS")
+			(hide yes)
 			(effects
 				(font
@@
 		)
 		(property "Value" "Vref2"
-			(at 0 1.55 0)
-			(layer "F.Fab")
+			(at 0.05 -1.75 0)
+			(layer "F.SilkS")
 			(effects
 				(font
@@
 		(sheetname "LTC6811_1")
 		(sheetfile "LTC6811.kicad_sch")
-		(attr exclude_from_pos_files)
+		(attr exclude_from_pos_files exclude_from_bom)
 		(fp_circle
 			(center 0 0)
@@
 		(property ki_fp_filters "MountingHole*")
 		(sheetname "根目录")
-		(sheetfile "LTC6811_ESP32_V5_Main.kicad_sch")
+		(sheetfile "LTC6811_ESP32_Master_V5.kicad_sch")
 		(attr exclude_from_pos_files exclude_from_bom)
 		(fp_circle
@@
 		(sheetname "PowerSupply")
 		(sheetfile "PowerSupply.kicad_sch")
-		(attr exclude_from_pos_files)
+		(attr exclude_from_pos_files exclude_from_bom)
 		(fp_circle
 			(center 0 0)
@@
 		)
 		(sheetname "根目录")
-		(sheetfile "LTC6811_ESP32_V5_Main.kicad_sch")
+		(sheetfile "LTC6811_ESP32_Master_V5.kicad_sch")
 		(attr smd exclude_from_bom)
 		(fp_poly
@@
 		(sheetname "PowerSupply")
 		(sheetfile "PowerSupply.kicad_sch")
-		(attr exclude_from_pos_files)
+		(attr exclude_from_pos_files exclude_from_bom)
 		(fp_circle
 			(center 0 0)
@@
 		(sheetname "LTC6811_2")
 		(sheetfile "LTC6811.kicad_sch")
-		(attr exclude_from_pos_files)
+		(attr exclude_from_pos_files exclude_from_bom)
 		(fp_circle
 			(center 0 0)
@@
 		(property ki_fp_filters "MountingHole*")
 		(sheetname "根目录")
-		(sheetfile "LTC6811_ESP32_V5_Main.kicad_sch")
+		(sheetfile "LTC6811_ESP32_Master_V5.kicad_sch")
 		(attr exclude_from_pos_files exclude_from_bom)
 		(fp_circle
@@
 		(property ki_fp_filters "MountingHole*")
 		(sheetname "根目录")
-		(sheetfile "LTC6811_ESP32_V5_Main.kicad_sch")
+		(sheetfile "LTC6811_ESP32_Master_V5.kicad_sch")
 		(attr exclude_from_pos_files exclude_from_bom)
 		(fp_circle
@@
 		(sheetname "LTC6811_2")
 		(sheetfile "LTC6811.kicad_sch")
-		(attr exclude_from_pos_files)
+		(attr exclude_from_pos_files exclude_from_bom)
 		(fp_circle
 			(center 0 0)
@@
 		(sheetfile "CAN.kicad_sch")
 		(zone_connect 1)
-		(attr exclude_from_pos_files)
+		(attr exclude_from_pos_files exclude_from_bom)
 		(fp_line
 			(start -0.7 -1)
@@
 		(property ki_fp_filters "MountingHole*")
 		(sheetname "根目录")
-		(sheetfile "LTC6811_ESP32_V5_Main.kicad_sch")
+		(sheetfile "LTC6811_ESP32_Master_V5.kicad_sch")
 		(attr exclude_from_pos_files exclude_from_bom)
 		(fp_circle
@@
 		(property ki_fp_filters "MountingHole*")
 		(sheetname "根目录")
-		(sheetfile "LTC6811_ESP32_V5_Main.kicad_sch")
+		(sheetfile "LTC6811_ESP32_Master_V5.kicad_sch")
 		(attr exclude_from_pos_files exclude_from_bom)
 		(fp_circle
@@
 		(property ki_fp_filters "Connector*:*_1x??_*")
 		(sheetname "根目录")
-		(sheetfile "LTC6811_ESP32_V5_Main.kicad_sch")
+		(sheetfile "LTC6811_ESP32_Master_V5.kicad_sch")
 		(zone_connect 2)
 		(attr through_hole)
@@
 		(property ki_fp_filters "MountingHole*")
 		(sheetname "根目录")
-		(sheetfile "LTC6811_ESP32_V5_Main.kicad_sch")
+		(sheetfile "LTC6811_ESP32_Master_V5.kicad_sch")
 		(attr exclude_from_pos_files exclude_from_bom)
 		(fp_circle
@@
 			)
 		)
-		(property "Value" "0.1uF/50V"
+		(property "Value" "100nF/100V"
 			(at 0 1.43 0)
 			(layer "F.Fab")
@@
 			)
 		)
-		(property "Datasheet" "https://mm.digikey.com/Volume0/opasdata/d220001/medias/docus/658/CL10B104KB8NNWC_Spec.pdf"
+		(property "Datasheet" "https://www.digikey.jp/en/products/detail/samsung-electro-mechanics/CL10B104KC8NNNC/5961291?s=N4IgTCBcDaIMIBkCMAGAQqgLAaTgDgDki4AdEkAXQF8g"
 			(at 0 0 180)
 			(unlocked yes)
@@
 			)
 		)
-		(property "Description" "0.1 µF ±10% 50V Ceramic Capacitor X7R 0603 (1608 Metric)"
+		(property "Description" "0.1 µF ±10% 100V Ceramic Capacitor X7R 0603 (1608 Metric)"
 			(at 0 0 180)
 			(unlocked yes)
@@
 			)
 		)
-		(property "MPN" "CL10B104KB8NNWC"
+		(property "MPN" "CL10B104KC8NNNC"
 			(at 0 0 180)
 			(unlocked yes)
@@
 			)
 		)
-		(property "Link" "https://www.digikey.jp/en/products/detail/samsung-electro-mechanics/CL10B104KB8NNWC/3887593"
+		(property "Link" "https://www.digikey.jp/en/products/detail/samsung-electro-mechanics/CL10B104KC8NNNC/5961291?s=N4IgTCBcDaIMIBkCMAGAQqgLAaTgDgDki4QBdAXyA"
 			(at 0 0 180)
 			(unlocked yes)
@@
 		(property ki_fp_filters "Connector*:*_1x??_*")
 		(sheetname "根目录")
-		(sheetfile "LTC6811_ESP32_V5_Main.kicad_sch")
+		(sheetfile "LTC6811_ESP32_Master_V5.kicad_sch")
 		(zone_connect 2)
 		(attr through_hole)
@@
 			)
 		)
-		(property "Value" "0.1uF/50V"
+		(property "Value" "100nF/100V"
 			(at 0 1.43 90)
 			(layer "F.Fab")
@@
 			)
 		)
-		(property "Datasheet" "https://mm.digikey.com/Volume0/opasdata/d220001/medias/docus/658/CL10B104KB8NNWC_Spec.pdf"
+		(property "Datasheet" "https://www.digikey.jp/en/products/detail/samsung-electro-mechanics/CL10B104KC8NNNC/5961291?s=N4IgTCBcDaIMIBkCMAGAQqgLAaTgDgDki4AdEkAXQF8g"
 			(at 0 0 90)
 			(unlocked yes)
@@
 			)
 		)
-		(property "Description" "0.1 µF ±10% 50V Ceramic Capacitor X7R 0603 (1608 Metric)"
+		(property "Description" "0.1 µF ±10% 100V Ceramic Capacitor X7R 0603 (1608 Metric)"
 			(at 0 0 90)
 			(unlocked yes)
@@
 			)
 		)
-		(property "MPN" "CL10B104KB8NNWC"
+		(property "MPN" "CL10B104KC8NNNC"
 			(at 0 0 90)
 			(unlocked yes)
@@
 			)
 		)
-		(property "Link" "https://www.digikey.jp/en/products/detail/samsung-electro-mechanics/CL10B104KB8NNWC/3887593"
+		(property "Link" "https://www.digikey.jp/en/products/detail/samsung-electro-mechanics/CL10B104KC8NNNC/5961291?s=N4IgTCBcDaIMIBkCMAGAQqgLAaTgDgDki4QBdAXyA"
 			(at 0 0 90)
 			(unlocked yes)
@@
 		(layer "F.Fab")
 	)
-	(gr_text "BMS_Master\nLTC6811_ESP32_V5\n2024/09/12"
-		(at 85.7 135.941928 0)
+	(gr_text "BMS_ESP32\n2024/09/12\nLTC6811_Master_V5\n"
+		(at 87.65 136.65 -0)
 		(layer "B.SilkS")
 		(effects
 			(font
-				(size 0.8 0.8)
-				(thickness 0.12)
+				(size 1 1)
+				(thickness 0.15)
 			)
 			(justify left bottom mirror)
@@
 		)
 	)
-	(gr_text "BMS_Master\n2024/09/12\nLTC6811_ESP32_V5\n"
+	(gr_text "BMS_ESP32\n2024/09/12\nLTC6811_Master_V5\n"
 		(at 97.7 161.6 0)
 		(layer "F.SilkS")
